Commit message: p2os_urdf added correct version of pioneer 3dx model in correct directory

File: p2os/p2os_urdf/correct/pioneer3dx.xacro (robot description, xacro)
@@ -7,5 +7,5 @@
 <!-- Chassis -->
 	<link name="base_link">
-		<inertial>
+		<intertial>
 			<mass value="3.5"/>
 			<origin xyz="-0.025 0 -0.223"/>
@@ -15,7 +15,7 @@
 		</inertial>
 		<visual name="base_visual">
-			<origin xyz="-0.045 0 0.148" rpy="0 0 0"/>
+			<origin xyz="0 0 0.318" rpy="0 0 0"/>
 			<geometry name="pioneer_geom">
-				<mesh filename="package://p2os_urdf/meshes/p3dx_meshes/chassis.stl"/>
+				<mesh filename="package://p2os_urdf/correct/pioneer3dx_meshes/chassis.stl"/>
 			</geometry>
 			<material name="ChassisRed">
@@ -38,9 +38,9 @@
 				 iyy="1" iyz="0"
  				izz="1"/>
-		</inertial>
+			</inertial>
 		<visual name="base_visual">
-			<origin xyz="-0.045 0 0.234" rpy="0 0 0"/>
+			<origin xyz="0 0 0.236" rpy="0 0 0"/>
 			<geometry name="pioneer_geom">
-				<mesh filename="package://p2os_urdf/meshes/p3dx_meshes/top.stl"/>
+				<mesh filename="package://p2os_urdf/correct/pioneer3dx_meshes/top.stl"/>
 			</geometry>
 			<material name="TopBlack">
@@ -64,7 +64,7 @@
   	 	</inertial>
 	<visual name="base_visual">
-		<origin xyz="-0.185 0 0.055" rpy="0 0 0"/>
-		<geometry name="pioneer_geom">
-			<mesh filename="package://p2os_urdf/meshes/p3dx_meshes/swivel.stl"/>
+		<origin xyz="-0.179 0 0.034" rpy="0 0 0"/>
+		<geometry name="pioneer_geom">
+			<mesh filename="package://p2os_urdf/correct/pioneer3dx_meshes/swivel.stl"/>
 		</geometry>
 		<material name="swivel">
@@ -88,7 +88,7 @@
   	 	</inertial>
 	<visual name="base_visual">
-		<origin xyz="-0.211 0 0.038" rpy="0 0 0"/>
-		<geometry name="pioneer_geom">
-			<mesh filename="package://p2os_urdf/meshes/p3dx_meshes/center_hubcap.stl"/>
+		<origin xyz="-0.211 0 0.037" rpy="0 0 0"/>
+		<geometry name="pioneer_geom">
+			<mesh filename="package://p2os_urdf/correct/pioneer3dx_meshes/center_hubcap.stl"/>
 		</geometry>
 		<material name="swivel">
@@ -111,7 +111,7 @@
   	 	</inertial>
 	<visual name="base_visual">
-		<origin xyz="-0.211 0.149 0.037" rpy="0 0 0"/>
-		<geometry name="pioneer_geom">
-			<mesh filename="package://p2os_urdf/meshes/p3dx_meshes/center_wheel.stl"/>
+		<origin xyz="-0.179 0 0.034" rpy="0 0 0"/>
+		<geometry name="pioneer_geom">
+			<mesh filename="package://p2os_urdf/correct/pioneer3dx_meshes/center_wheel.stl"/>
 		</geometry>
 		<material name="WheelBlack">
@@ -137,5 +137,5 @@
 		<origin xyz="0 0.158 0.091" rpy="0 0 0"/>
 		<geometry name="pioneer_geom">
-			<mesh filename="package://p2os_urdf/meshes/p3dx_meshes/right_hubcap.stl"/>
+			<mesh filename="package://p2os_urdf/correct/pioneer3dx_meshes/right_hubcap.stl"/>
 		</geometry>
 		<material name="HubcapYellow">
@@ -160,5 +160,5 @@
 		<origin xyz="0 0.158 0.091" rpy="0 0 0"/>
 		<geometry name="pioneer_geom">
-			<mesh filename="package://p2os_urdf/meshes/p3dx_meshes/right_wheel.stl"/>
+			<mesh filename="package://p2os_urdf/correct/pioneer3dx_meshes/right_wheel.stl"/>
 		</geometry>
 		<material name="WheelBlack">
@@ -184,5 +184,5 @@
 		<origin xyz="0 -0.158 0.091" rpy="0 0 0"/>
 		<geometry name="pioneer_geom">
-			<mesh filename="package://p2os_urdf/meshes/p3dx_meshes/left_hubcap.stl"/>
+			<mesh filename="package://p2os_urdf/correct/pioneer3dx_meshes/left_hubcap.stl"/>
 		</geometry>
 		<material name="HubcapYellow">
@@ -207,5 +207,5 @@
 		<origin xyz="0 -0.158 0.091" rpy="0 0 0"/>
 		<geometry name="pioneer_geom">
-			<mesh filename="package://p2os_urdf/meshes/p3dx_meshes/left_wheel.stl"/>
+			<mesh filename="package://p2os_urdf/correct/pioneer3dx_meshes/left_wheel.stl"/>
 		</geometry>
 		<material name="WheelBlack">
@@ -229,7 +229,7 @@
 		</inertial>
 		<visual name="base_visual">
-			<origin xyz="-0.2 0 0.209" rpy="0 0 0"/>
+			<origin xyz="-0.196 0.199 0.218" rpy="0 0 0"/>
 			<geometry name="pioneer_geom">
-				<mesh filename="package://p2os_urdf/meshes/p3dx_meshes/front_sonar.stl"/>
+				<mesh filename="package://p2os_urdf/correct/pioneer3dx_meshes/front_sonar.stl"/>
 			</geometry>
 			<material name="SonarYellow">
@@ -252,7 +252,7 @@
 		</inertial>
 		<visual name="base_visual">
-			<origin xyz="0.109 0 0.209" rpy="0 0 0"/>
+			<origin xyz="0.105 0.199 0.218" rpy="0 0 0"/>
 			<geometry name="pioneer_geom">
-				<mesh filename="package://p2os_urdf/meshes/p3dx_meshes/back_sonar.stl"/>
+				<mesh filename="package://p2os_urdf/correct/pioneer3dx_meshes/back_sonar.stl"/>
 			</geometry>
 			<material name="SonarYellow">
@@ -318,3 +318,2 @@
 		<child link="left_wheel"/>
 	</joint>
-</robot>
