Commit message: updated p3at/p3dx models

File: p2os/p2os_urdf/defs/pioneer3at.xacro (robot description, xacro)
@@ -40,5 +40,5 @@
 		</inertial>
 		<visual name="base_visual">
-			<origin xyz="0.003 0 0.274" rpy="0 0 0"/>
+			<origin xyz="0 0 0" rpy="0 0 0"/>
 			<geometry name="pioneer_geom">
 				<mesh filename="package://p2os_urdf/meshes/p3at_meshes/top.stl"/>
@@ -55,4 +55,9 @@
 		</collision>
 	</link>
+	<joint name="base_top_joint" type="fixed">
+		<origin xyz="0.003 0 0.274" rpy="0 0 0"/>
+		<parent link="base_link"/>
+		<child link="top_plate"/>
+	</joint>
 <!-- Front + Back Sonar -->
 	<link name="front_sonar">
@@ -64,5 +69,5 @@
 		</inertial>
 		<visual name="base_visual">
-			<origin xyz="0.193 0 0.25" rpy="0 0 0"/>
+			<origin xyz="0 0 0" rpy="0 0 0"/>
 			<geometry name="pioneer_geom">
 				<mesh filename="package://p2os_urdf/meshes/p3at_meshes/front_sonar.stl"/>
@@ -79,4 +84,9 @@
 		</collision>
 	</link>
+	<joint name="base_front_joint" type="fixed">
+		<origin xyz="0.193 0 0.25" rpy="0 0 0"/>
+		<parent link="base_link"/>
+		<child link="front_sonar"/>
+	</joint>
 	<link name="back_sonar">
 		<inertial>
@@ -87,5 +97,5 @@
 		</inertial>
 		<visual name="base_visual">
-			<origin xyz="-0.187 0 0.247" rpy="0 0 0"/>
+			<origin xyz="0 0 0" rpy="0 0 0"/>
 			<geometry name="pioneer_geom">
 				<mesh filename="package://p2os_urdf/meshes/p3at_meshes/back_sonar.stl"/>
@@ -102,14 +112,20 @@
 		</collision>
 	</link>
-<!-- Axles -->
-	<link name="fr_axle">
-		<inertial>
-			<mass value="0"/>
-			<origin xyz="0 0 0"/>
-			<inertia ixx="1" ixy="0" ixz="0"
-				 iyy="1" iyz="0" izz="1"/>
-  	 	</inertial>
-	<visual name="base_visual">
-		<origin xyz="0.135 -0.156 0.111" rpy="0 0 0"/>
+	<joint name="base_back_joint" type="fixed">
+		<origin xyz="-0.187 0 0.247" rpy="0 0 0"/>
+		<parent link="base_link"/>
+		<child link="back_sonar"/>
+	</joint>
+<!-- Front Axles + Wheels + Hubcaps -->
+<xacro:macro name="p3at_front" params="suffix reflect">
+	<link name="p3at_front_${suffix}_axle">
+		<inertial>
+			<mass value="0"/>
+			<origin xyz="0 0 0"/>
+			<inertia ixx="1" ixy="0" ixz="0"
+				 iyy="1" iyz="0" izz="1"/>
+  	 	</inertial>
+	<visual name="base_visual">
+		<origin xyz="0 0 0" rpy="0 0 0"/>
 		<geometry name="pioneer_geom">
 			<mesh filename="package://p2os_urdf/meshes/p3at_meshes/axle.stl"/>
@@ -126,13 +142,75 @@
 	</collision>
 	</link>
-	<link name="fl_axle">
-		<inertial>
-			<mass value="0"/>
-			<origin xyz="0 0 0"/>
-			<inertia ixx="1" ixy="0" ixz="0"
-				 iyy="1" iyz="0" izz="1"/>
-  	 	</inertial>
-	<visual name="base_visual">
-		<origin xyz="0.135 0.156 0.111" rpy="0 0 0"/>
+	<joint name="base_front_${suffix}_axle_joint" type="fixed">
+		<origin xyz="0.135 ${reflect*0.156} 0.111" rpy="0 0 0"/>
+		<parent link="base_link"/>
+		<child link="p3at_front_${suffix}_axle"/>
+	</joint>
+	<link name="p3at_front_${suffix}_hub">
+		<inertial>
+			<mass value="0"/>
+			<origin xyz="0 0 0"/>
+			<inertia ixx="1" ixy="0" ixz="0"
+				 iyy="1" iyz="0" izz="1"/>
+  	 	</inertial>
+	<visual name="base_visual">
+		<origin xyz="0 0 0" rpy="0 0 0"/>
+		<geometry name="pioneer_geom">
+			<mesh filename="package://p2os_urdf/meshes/p3at_meshes/${suffix}_hubcap.stl"/>
+		</geometry>
+		<material name="HubcapYellow">
+			<color rgba="1.0 0.811 0.151 1.0"/>
+		</material>
+	</visual>
+	<collision>
+		<origin xyz="0 0 0" rpy="0 0 0"/>
+		<geometry>
+			<box size="0 0 0"/>
+		</geometry>
+	</collision>
+	</link>
+	<joint name="base_front_${suffix}_hub_joint" type="fixed">
+		<origin xyz="0 ${reflect*0.041} 0" rpy="0 0 0"/>
+		<parent link="p3at_front_${suffix}_axle"/>
+		<child link="p3at_front_${suffix}_hub"/>
+	</joint>
+	<link name="p3at_front_${suffix}_wheel">
+		<inertial>
+			<mass value="0"/>
+			<origin xyz="0 0 0"/>
+			<inertia ixx="1" ixy="0" ixz="0"
+				 iyy="1" iyz="0" izz="1"/>
+  	 	</inertial>
+	<visual name="base_visual">
+		<origin xyz="0 0 0" rpy="0 0 0"/>
+		<geometry name="pioneer_geom">
+			<mesh filename="package://p2os_urdf/meshes/p3at_meshes/wheel.stl"/>
+		</geometry>
+		<material name="WheelBlack">
+			<color rgba="0.117 0.117 0.117 1"/>
+		</material>
+	</visual>
+	<collision>
+		<origin xyz="0 0 0" rpy="0 0 0"/>
+		<geometry>
+			<box size="0 0 0"/>
+		</geometry>
+	</collision>
+	</link>
+	<joint name="base_front_${suffix}_wheel_joint" type="fixed">
+		<origin xyz="0 0 0" rpy="0 0 0"/>
+		<parent link="p3at_front_${suffix}_hub"/>
+		<child link="p3at_front_${suffix}_wheel"/>
+	</joint>
+<!-- Back Axles + Wheels + Hubcaps -->
+	<link name="p3at_back_${suffix}_axle">
+		<inertial>
+			<mass value="0"/>
+			<origin xyz="0 0 0"/>
+			<inertia ixx="1" ixy="0" ixz="0"
+				 iyy="1" iyz="0" izz="1"/>
+  	 	</inertial>
+	<visual name="base_visual">
+		<origin xyz="0 0 0" rpy="0 0 0"/>
 		<geometry name="pioneer_geom">
 			<mesh filename="package://p2os_urdf/meshes/p3at_meshes/axle.stl"/>
@@ -149,86 +227,47 @@
 	</collision>
 	</link>
-	<link name="br_axle">
-		<inertial>
-			<mass value="0"/>
-			<origin xyz="0 0 0"/>
-			<inertia ixx="1" ixy="0" ixz="0"
-				 iyy="1" iyz="0" izz="1"/>
-  	 	</inertial>
-	<visual name="base_visual">
-		<origin xyz="-0.134 -0.156 0.111" rpy="0 0 0"/>
-		<geometry name="pioneer_geom">
-			<mesh filename="package://p2os_urdf/meshes/p3at_meshes/axle.stl"/>
-		</geometry>
-		<material name="AxleGrey">
-			<color rgba="0.5 0.5 0.5 1"/>
-		</material>
-	</visual>
-	<collision>
-		<origin xyz="0 0 0" rpy="0 0 0"/>
-		<geometry>
-			<box size="0 0 0"/>
-		</geometry>
-	</collision>
-	</link>
-	<link name="bl_axle">
-		<inertial>
-			<mass value="0"/>
-			<origin xyz="0 0 0"/>
-			<inertia ixx="1" ixy="0" ixz="0"
-				 iyy="1" iyz="0" izz="1"/>
-  	 	</inertial>
-	<visual name="base_visual">
-		<origin xyz="-0.134 0.156 0.111" rpy="0 0 0"/>
-		<geometry name="pioneer_geom">
-			<mesh filename="package://p2os_urdf/meshes/p3at_meshes/axle.stl"/>
-		</geometry>
-		<material name="AxleGrey">
-			<color rgba="0.5 0.5 0.5 1"/>
-		</material>
-	</visual>
-	<collision>
-		<origin xyz="0 0 0" rpy="0 0 0"/>
-		<geometry>
-			<box size="0 0 0"/>
-		</geometry>
-	</collision>
-	</link>
-<!-- Wheels -->
-	<link name="fr_wheel">
-		<inertial>
-			<mass value="0"/>
-			<origin xyz="0 0 0"/>
-			<inertia ixx="1" ixy="0" ixz="0"
-				 iyy="1" iyz="0" izz="1"/>
-  	 	</inertial>
-	<visual name="base_visual">
-		<origin xyz="0.135 -0.199 0.111" rpy="0 0 0"/>
+	<joint name="bp3at_back_${suffix}_axle_joint" type="fixed">
+		<origin xyz="-0.134 ${reflect*0.156} 0.111" rpy="0 0 0"/>
+		<parent link="base_link"/>
+		<child link="p3at_back_${suffix}_axle"/>
+	</joint>
+	<link name="p3at_back_${suffix}_hub">
+		<inertial>
+			<mass value="0"/>
+			<origin xyz="0 0 0"/>
+			<inertia ixx="1" ixy="0" ixz="0"
+				 iyy="1" iyz="0" izz="1"/>
+  	 	</inertial>
+	<visual name="base_visual">
+		<origin xyz="0 0 0" rpy="0 0 0"/>
+		<geometry name="pioneer_geom">
+			<mesh filename="package://p2os_urdf/meshes/p3at_meshes/${suffix}_hubcap.stl"/>
+		</geometry>
+		<material name="HubcapYellow"/>
+	</visual>
+	<collision>
+		<origin xyz="0 0 0" rpy="0 0 0"/>
+		<geometry>
+			<box size="0 0 0"/>
+		</geometry>
+	</collision>
+	</link>
+	<joint name="p3at_back_${suffix}_hub_joint" type="fixed">
+		<origin xyz="-0 ${reflect*0.041} 0" rpy="0 0 0"/>
+		<parent link="p3at_back_${suffix}_axle"/>
+		<child link="p3at_back_${suffix}_hub"/>
+	</joint>
+	<link name="p3at_back_${suffix}_wheel">
+		<inertial>
+			<mass value="0"/>
+			<origin xyz="0 0 0"/>
+			<inertia ixx="1" ixy="0" ixz="0"
+				 iyy="1" iyz="0" izz="1"/>
+  	 	</inertial>
+	<visual name="base_visual">
+		<origin xyz="0 0 0" rpy="0 0 0"/>
 		<geometry name="pioneer_geom">
 			<mesh filename="package://p2os_urdf/meshes/p3at_meshes/wheel.stl"/>
 		</geometry>
-		<material name="WheelBlack">
-			<color rgba="0.117 0.117 0.117 1"/>
-		</material>
-	</visual>
-	<collision>
-		<origin xyz="0 0 0" rpy="0 0 0"/>
-		<geometry>
-			<box size="0 0 0"/>
-		</geometry>
-	</collision>
-	</link>
-	<link name="fl_wheel">
-		<inertial>
-			<mass value="0"/>
-			<origin xyz="0 0 0"/>
-			<inertia ixx="1" ixy="0" ixz="0"
-				 iyy="1" iyz="0" izz="1"/>
-  	 	</inertial>
-	<visual name="base_visual">
-		<origin xyz="0.135 0.199 0.111" rpy="0 0 0"/>
-		<geometry name="pioneer_geom">
-			<mesh filename="package://p2os_urdf/meshes/p3at_meshes/wheel.stl"/>
-		</geometry>
 		<material name="WheelBlack"/>
 	</visual>
@@ -240,208 +279,13 @@
 	</collision>
 	</link>
-	<link name="br_wheel">
-		<inertial>
-			<mass value="0"/>
-			<origin xyz="0 0 0"/>
-			<inertia ixx="1" ixy="0" ixz="0"
-				 iyy="1" iyz="0" izz="1"/>
-  	 	</inertial>
-	<visual name="base_visual">
-		<origin xyz="-0.134 -0.199 0.111" rpy="0 0 0"/>
-		<geometry name="pioneer_geom">
-			<mesh filename="package://p2os_urdf/meshes/p3at_meshes/wheel.stl"/>
-		</geometry>
-		<material name="WheelBlack"/>
-	</visual>
-	<collision>
-		<origin xyz="0 0 0" rpy="0 0 0"/>
-		<geometry>
-			<box size="0 0 0"/>
-		</geometry>
-	</collision>
-	</link>
-	<link name="bl_wheel">
-		<inertial>
-			<mass value="0"/>
-			<origin xyz="0 0 0"/>
-			<inertia ixx="1" ixy="0" ixz="0"
-				 iyy="1" iyz="0" izz="1"/>
-  	 	</inertial>
-	<visual name="base_visual">
-		<origin xyz="-0.134 0.199 0.111" rpy="0 0 0"/>
-		<geometry name="pioneer_geom">
-			<mesh filename="package://p2os_urdf/meshes/p3at_meshes/wheel.stl"/>
-		</geometry>
-		<material name="WheelBlack"/>
-	</visual>
-	<collision>
-		<origin xyz="0 0 0" rpy="0 0 0"/>
-		<geometry>
-			<box size="0 0 0"/>
-		</geometry>
-	</collision>
-	</link>
-<!-- Hubcaps -->
-	<link name="fr_hub">
-		<inertial>
-			<mass value="0"/>
-			<origin xyz="0 0 0"/>
-			<inertia ixx="1" ixy="0" ixz="0"
-				 iyy="1" iyz="0" izz="1"/>
-  	 	</inertial>
-	<visual name="base_visual">
-		<origin xyz="0.135 -0.199 0.111" rpy="0 0 0"/>
-		<geometry name="pioneer_geom">
-			<mesh filename="package://p2os_urdf/meshes/p3at_meshes/right_hubcap.stl"/>
-		</geometry>
-		<material name="HubcapYellow">
-			<color rgba="1.0 0.811 0.151 1.0"/>
-		</material>
-	</visual>
-	<collision>
-		<origin xyz="0 0 0" rpy="0 0 0"/>
-		<geometry>
-			<box size="0 0 0"/>
-		</geometry>
-	</collision>
-	</link>
-	<link name="fl_hub">
-		<inertial>
-			<mass value="0"/>
-			<origin xyz="0 0 0"/>
-			<inertia ixx="1" ixy="0" ixz="0"
-				 iyy="1" iyz="0" izz="1"/>
-  	 	</inertial>
-	<visual name="base_visual">
-		<origin xyz="0.135 0.199 0.111" rpy="0 0 0"/>
-		<geometry name="pioneer_geom">
-			<mesh filename="package://p2os_urdf/meshes/p3at_meshes/left_hubcap.stl"/>
-		</geometry>
-		<material name="HubcapYellow"/>
-	</visual>
-	<collision>
-		<origin xyz="0 0 0" rpy="0 0 0"/>
-		<geometry>
-			<box size="0 0 0"/>
-		</geometry>
-	</collision>
-	</link>
-	<link name="br_hub">
-		<inertial>
-			<mass value="0"/>
-			<origin xyz="0 0 0"/>
-			<inertia ixx="1" ixy="0" ixz="0"
-				 iyy="1" iyz="0" izz="1"/>
-  	 	</inertial>
-	<visual name="base_visual">
-		<origin xyz="-0.134 -0.199 0.111" rpy="0 0 0"/>
-		<geometry name="pioneer_geom">
-			<mesh filename="package://p2os_urdf/meshes/p3at_meshes/right_hubcap.stl"/>
-		</geometry>
-		<material name="HubcapYellow"/>
-	</visual>
-	<collision>
-		<origin xyz="0 0 0" rpy="0 0 0"/>
-		<geometry>
-			<box size="0 0 0"/>
-		</geometry>
-	</collision>
-	</link>
-	<link name="bl_hub">
-		<inertial>
-			<mass value="0"/>
-			<origin xyz="0 0 0"/>
-			<inertia ixx="1" ixy="0" ixz="0"
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