Commit message: p2os_urdf: some changes to make joints and visuals be in the correct place

File: p2os/p2os_urdf/defs/pioneer3dx.xacro (robot description, xacro)
@@ -9,5 +9,6 @@
 		<inertial>
 			<mass value="3.5"/>
-			<origin xyz="-0.025 0 -0.223"/>
+			<!--<origin xyz="-0.025 0 -0.223"/>-->
+			<origin xyz="0 0 0"/>
 			<inertia ixx="1" ixy="0" ixz="0"
 				 iyy="1" iyz="0"
@@ -34,5 +35,5 @@
 		<inertial>
 			<mass value="0"/>
-			<origin xyz="-0.025 0 -0.223"/>
+			<origin xyz="0 0 0"/>
 			<inertia ixx="1" ixy="0" ixz="0"
 				 iyy="1" iyz="0"
@@ -40,5 +41,5 @@
 		</inertial>
 		<visual name="base_visual">
-			<origin xyz="-0.045 0 0.234" rpy="0 0 0"/>
+			<origin xyz="0 0 0" rpy="0 0 0"/>
 			<geometry name="pioneer_geom">
 				<mesh filename="package://p2os_urdf/meshes/p3dx_meshes/top.stl"/>
@@ -55,4 +56,9 @@
 		</collision>
 	</link>
+  <joint name="base_top_joint" type="fixed">
+		<origin xyz="-0.045 0 0.234" rpy="0 0 0"/>
+		<parent link="base_link"/>
+		<child link="top_plate"/>
+	</joint>
 <!-- Swivel -->
 	<link name="swivel">
@@ -64,5 +70,5 @@
   	 	</inertial>
 	<visual name="base_visual">
-		<origin xyz="-0.185 0 0.055" rpy="0 0 0"/>
+		<origin xyz="0 0 0" rpy="0 0 0"/>
 		<geometry name="pioneer_geom">
 			<mesh filename="package://p2os_urdf/meshes/p3dx_meshes/swivel.stl"/>
@@ -79,4 +85,9 @@
 	</collision>
 	</link>
+ 	<joint name="base_swivel_joint" type="fixed">
+		<origin xyz="-0.185 0 0.055" rpy="0 0 0"/>
+		<parent link="base_link"/>
+		<child link="swivel"/>
+	</joint>
 <!-- Center Wheel + Hubcap -->
 	<link name="center_hubcap">
@@ -88,5 +99,5 @@
   	 	</inertial>
 	<visual name="base_visual">
-		<origin xyz="-0.211 0 0.038" rpy="0 0 0"/>
+		<origin xyz="0 0 0" rpy="0 0 0"/>
 		<geometry name="pioneer_geom">
 			<mesh filename="package://p2os_urdf/meshes/p3dx_meshes/center_hubcap.stl"/>
@@ -103,4 +114,9 @@
 	</collision>
 	</link>
+  <joint name="swivel_hubcap_joint" type="fixed">
+		<origin xyz="-0.211 0 0.038" rpy="0 0 0"/>
+		<parent link="swivel"/>
+		<child link="center_hubcap"/>
+	</joint>
 	<link name="center_wheel">
 		<inertial>
@@ -135,5 +151,5 @@
   	 	</inertial>
 	<visual name="base_visual">
-		<origin xyz="0 0.158 0.091" rpy="0 0 0"/>
+		<origin xyz="0 0 0" rpy="0 0 0"/>
 		<geometry name="pioneer_geom">
 			<mesh filename="package://p2os_urdf/meshes/p3dx_meshes/right_hubcap.stl"/>
@@ -268,9 +284,4 @@
 	</link>
 <!-- Joints -->
-	<joint name="base_top_joint" type="fixed">
-		<origin xyz="0 0 0" rpy="0 0 0"/>
-		<parent link="base_link"/>
-		<child link="top_plate"/>
-	</joint>
 	<joint name="base_front_joint" type="fixed">
 		<origin xyz="0 0 0" rpy="0 0 0"/>
@@ -282,14 +293,4 @@
 		<parent link="base_link"/>
 		<child link="back_sonar"/>
-	</joint>
-	<joint name="base_swivel_joint" type="fixed">
-		<origin xyz="0 0 0" rpy="0 0 0"/>
-		<parent link="base_link"/>
-		<child link="swivel"/>
-	</joint>
-	<joint name="swivel_hubcap_joint" type="fixed">
-		<origin xyz="0 0 0" rpy="0 0 0"/>
-		<parent link="swivel"/>
-		<child link="center_hubcap"/>
 	</joint>
 	<joint name="center_wheel_joint" type="fixed">

Commit message: working model

File: p2os/p2os_urdf/defs/pioneer3dx.xacro (robot description, xacro)
@@ -56,5 +56,5 @@
 		</collision>
 	</link>
-  <joint name="base_top_joint" type="fixed">
+	<joint name="base_top_joint" type="fixed">
 		<origin xyz="-0.045 0 0.234" rpy="0 0 0"/>
 		<parent link="base_link"/>
@@ -114,6 +114,6 @@
 	</collision>
 	</link>
-  <joint name="swivel_hubcap_joint" type="fixed">
-		<origin xyz="-0.211 0 0.038" rpy="0 0 0"/>
+	<joint name="swivel_hubcap_joint" type="fixed">
+		<origin xyz="-0.026 0 -0.016" rpy="0 0 0"/>
 		<parent link="swivel"/>
 		<child link="center_hubcap"/>
@@ -127,5 +127,5 @@
   	 	</inertial>
 	<visual name="base_visual">
-		<origin xyz="-0.211 0.149 0.037" rpy="0 0 0"/>
+		<origin xyz="0 0 0" rpy="0 0 0"/>
 		<geometry name="pioneer_geom">
 			<mesh filename="package://p2os_urdf/meshes/p3dx_meshes/center_wheel.stl"/>
@@ -142,16 +142,50 @@
 	</collision>
 	</link>
-<!-- Right Wheel + Hubcap -->
-	<link name="right_hubcap">
-		<inertial>
-			<mass value="0"/>
-			<origin xyz="0 0 0"/>
-			<inertia ixx="1" ixy="0" ixz="0"
-				 iyy="1" iyz="0" izz="1"/>
-  	 	</inertial>
-	<visual name="base_visual">
-		<origin xyz="0 0 0" rpy="0 0 0"/>
-		<geometry name="pioneer_geom">
-			<mesh filename="package://p2os_urdf/meshes/p3dx_meshes/right_hubcap.stl"/>
+	<joint name="center_wheel_joint" type="fixed">
+		<origin xyz="-0.0035 0 -0.001" rpy="0 0 0"/>
+		<parent link="center_hubcap"/>
+		<child link="center_wheel"/>
+	</joint>
+<!-- Right/Left Hubcap + Wheel -->
+<xacro:macro name="p3dx_wheel" params="suffix parent reflect">
+	<link name="p3dx_${suffix}_wheel">
+		<inertial>
+			<mass value="0"/>
+			<origin xyz="0 0 0"/>
+			<inertia ixx="1" ixy="0" ixz="0"
+				 iyy="1" iyz="0" izz="1"/>
+  	 	</inertial>
+	<visual name="base_visual">
+		<origin xyz="0 0 0" rpy="0 0 0"/>
+		<geometry name="pioneer_geom">
+			<mesh filename="package://p2os_urdf/meshes/p3dx_meshes/${suffix}_wheel.stl"/>
+		</geometry>
+		<material name="WheelBlack">
+			<color rgba="0.117 0.117 0.117 1"/>
+		</material>
+	</visual>
+	<collision>
+		<origin xyz="0 0 0" rpy="0 0 0"/>
+		<geometry>
+			<box size="0 0 0"/>
+		</geometry>
+	</collision>
+	</link>
+	<joint name="base_${suffix}_wheel_joint" type="fixed">
+		<origin xyz="0 ${reflect*0.158} 0.091" rpy="0 0 0"/>
+		<parent link="${parent}"/>
+		<child link="p3dx_${suffix}_wheel"/>
+	</joint>
+	<link name="p3dx_${suffix}_hubcap">
+		<inertial>
+			<mass value="0"/>
+			<origin xyz="0 0 0"/>
+			<inertia ixx="1" ixy="0" ixz="0"
+				 iyy="1" iyz="0" izz="1"/>
+  	 	</inertial>
+	<visual name="base_visual">
+		<origin xyz="0 0 0" rpy="0 0 0"/>
+		<geometry name="pioneer_geom">
+			<mesh filename="package://p2os_urdf/meshes/p3dx_meshes/${suffix}_hubcap.stl"/>
 		</geometry>
 		<material name="HubcapYellow">
@@ -166,74 +200,12 @@
 	</collision>
 	</link>
-	<link name="right_wheel">
-		<inertial>
-			<mass value="0"/>
-			<origin xyz="0 0 0"/>
-			<inertia ixx="1" ixy="0" ixz="0"
-				 iyy="1" iyz="0" izz="1"/>
-  	 	</inertial>
-	<visual name="base_visual">
-		<origin xyz="0 0.158 0.091" rpy="0 0 0"/>
-		<geometry name="pioneer_geom">
-			<mesh filename="package://p2os_urdf/meshes/p3dx_meshes/right_wheel.stl"/>
-		</geometry>
-		<material name="WheelBlack">
-			<color rgba="0.117 0.117 0.117 1"/>
-		</material>
-	</visual>
-	<collision>
-		<origin xyz="0 0 0" rpy="0 0 0"/>
-		<geometry>
-			<box size="0 0 0"/>
-		</geometry>
-	</collision>
-	</link>
-<!-- Left Wheel + Hubcap -->
-	<link name="left_hubcap">
-		<inertial>
-			<mass value="0"/>
-			<origin xyz="0 0 0"/>
-			<inertia ixx="1" ixy="0" ixz="0"
-				 iyy="1" iyz="0" izz="1"/>
-  	 	</inertial>
-	<visual name="base_visual">
-		<origin xyz="0 -0.158 0.091" rpy="0 0 0"/>
-		<geometry name="pioneer_geom">
-			<mesh filename="package://p2os_urdf/meshes/p3dx_meshes/left_hubcap.stl"/>
-		</geometry>
-		<material name="HubcapYellow">
-			<color rgba="1.0 0.811 0.151 1.0"/>
-		</material>
-	</visual>
-	<collision>
-		<origin xyz="0 0 0" rpy="0 0 0"/>
-		<geometry>
-			<box size="0 0 0"/>
-		</geometry>
-	</collision>
-	</link>
-	<link name="left_wheel">
-		<inertial>
-			<mass value="0"/>
-			<origin xyz="0 0 0"/>
-			<inertia ixx="1" ixy="0" ixz="0"
-				 iyy="1" iyz="0" izz="1"/>
-  	 	</inertial>
-	<visual name="base_visual">
-		<origin xyz="0 -0.158 0.091" rpy="0 0 0"/>
-		<geometry name="pioneer_geom">
-			<mesh filename="package://p2os_urdf/meshes/p3dx_meshes/left_wheel.stl"/>
-		</geometry>
-		<material name="WheelBlack">
-			<color rgba="0.117 0.117 0.117 1"/>
-		</material>
-	</visual>
-	<collision>
-		<origin xyz="0 0 0" rpy="0 0 0"/>
-		<geometry>
-			<box size="0 0 0"/>
-		</geometry>
-	</collision>
-	</link>
+	<joint name="base_${suffix}_hubcap_joint" type="fixed">
+		<origin xyz="0 ${reflect*0.158} 0.091" rpy="0 0 0"/>
+		<parent link="base_link"/>
+		<child link="p3dx_${suffix}_hubcap"/>
+	</joint>
+</xacro:macro>
+<xacro:p3dx_wheel suffix="left" parent="base_link" reflect="1"/>
+<xacro:p3dx_wheel suffix="right" parent="base_link" reflect="-1"/>
 <!-- Front + Back Sonar -->
 	<link name="front_sonar">
@@ -245,5 +217,5 @@
 		</inertial>
 		<visual name="base_visual">
-			<origin xyz="-0.2 0 0.209" rpy="0 0 0"/>
+			<origin xyz="0 0 0" rpy="0 0 0"/>
 			<geometry name="pioneer_geom">
 				<mesh filename="package://p2os_urdf/meshes/p3dx_meshes/front_sonar.stl"/>
@@ -260,4 +232,9 @@
 		</collision>
 	</link>
+	<joint name="base_front_joint" type="fixed">
+		<origin xyz="-0.198 0 0.208" rpy="0 0 0"/>
+		<parent link="base_link"/>
+		<child link="front_sonar"/>
+	</joint>
 	<link name="back_sonar">
 		<inertial>
@@ -268,5 +245,5 @@
 		</inertial>
 		<visual name="base_visual">
-			<origin xyz="0.109 0 0.209" rpy="0 0 0"/>
+			<origin xyz="0 0 0" rpy="0 0 0"/>
 			<geometry name="pioneer_geom">
 				<mesh filename="package://p2os_urdf/meshes/p3dx_meshes/back_sonar.stl"/>
@@ -283,39 +260,8 @@
 		</collision>
 	</link>
-<!-- Joints -->
-	<joint name="base_front_joint" type="fixed">
-		<origin xyz="0 0 0" rpy="0 0 0"/>
-		<parent link="base_link"/>
-		<child link="front_sonar"/>
-	</joint>
 	<joint name="base_back_joint" type="fixed">
-		<origin xyz="0 0 0" rpy="0 0 0"/>
+		<origin xyz="0.109 0 0.209" rpy="0 0 0"/>
 		<parent link="base_link"/>
 		<child link="back_sonar"/>
 	</joint>
-	<joint name="center_wheel_joint" type="fixed">
-		<origin xyz="0 0 0" rpy="0 0 0"/>
-		<parent link="center_hubcap"/>
-		<child link="center_wheel"/>
-	</joint>
-	<joint name="base_right_joint" type="fixed">
-		<origin xyz="0 0 0" rpy="0 0 0"/>
-		<parent link="base_link"/>
-		<child link="right_hubcap"/>
-	</joint>
-	<joint name="right_wheel_joint" type="fixed">
-		<origin xyz="0 0 0" rpy="0 0 0"/>
-		<parent link="right_hubcap"/>
-		<child link="right_wheel"/>
-	</joint>
-	<joint name="base_left_joint" type="fixed">
-		<origin xyz="0 0 0" rpy="0 0 0"/>
-		<parent link="base_link"/>
-		<child link="left_hubcap"/>
-	</joint>
-	<joint name="left_wheel_joint" type="fixed">
-		<origin xyz="0 0 0" rpy="0 0 0"/>
-		<parent link="left_hubcap"/>
-		<child link="left_wheel"/>
-	</joint>
 </robot>

Commit message: p2os_urdf: actuatable pioneer3dx in gazebo * needs tuning so it doesnt jump around as much * needs to fix colors of hubcaps * masses may not be right * inertial values are total guesses

File: p2os/p2os_urdf/defs/pioneer3dx.xacro (robot description, xacro)
@@ -10,5 +10,5 @@
 			<mass value="3.5"/>
 			<!--<origin xyz="-0.025 0 -0.223"/>-->
-			<origin xyz="0 0 0"/>
+			<origin xyz="-0.05 0 0"/>
 			<inertia ixx="1" ixy="0" ixz="0"
 				 iyy="1" iyz="0"
@@ -25,14 +25,17 @@
 		</visual>
 		<collision>
-			<origin xyz="0 0 0" rpy="0 0 0"/>
+			<origin xyz="-0.045 0 0.145" rpy="0 0 0"/>
 				<geometry>
-					<box size="0.01 0.01 0.01"/>
+					<box size="0.35 0.25 0.14"/>
 				</geometry>
 		</collision>
 	</link>
+	<gazebo reference="base_link">
+		<material value="Gazebo/Red"/>
+	</gazebo>
 <!-- Top -->
 	<link name="top_plate">
 		<inertial>
-			<mass value="0"/>
+			<mass value="0.01"/>
 			<origin xyz="0 0 0"/>
 			<inertia ixx="1" ixy="0" ixz="0"
@@ -42,5 +45,5 @@
 		<visual name="base_visual">
 			<origin xyz="0 0 0" rpy="0 0 0"/>
-			<geometry name="pioneer_geom">
+			<geometry name="top_geom">
 				<mesh filename="package://p2os_urdf/meshes/p3dx_meshes/top.stl"/>
 			</geometry>
@@ -50,10 +53,13 @@
 		</visual>
 		<collision>
-			<origin xyz="0 0 0" rpy="0 0 0"/>
-			<geometry>
-				<box size="0 0 0"/>
-			</geometry>
-		</collision>
-	</link>
+			<origin xyz="0.0 0 0" rpy="0 0 0"/>
+			<geometry name="pioneer_geom">
+				<box size="0.45 0.38 0.01"/>
+			</geometry>
+		</collision>
+	</link>
+	<gazebo reference="top_plate">
+		<material value="Gazebo/Black"/>
+	</gazebo>
 	<joint name="base_top_joint" type="fixed">
 		<origin xyz="-0.045 0 0.234" rpy="0 0 0"/>
@@ -64,8 +70,8 @@
 	<link name="swivel">
 		<inertial>
-			<mass value="0"/>
-			<origin xyz="0 0 0"/>
-			<inertia ixx="1" ixy="0" ixz="0"
-				 iyy="1" iyz="0" izz="1"/>
+			<mass value="0.1"/>
+			<origin xyz="0 0 0"/>
+			<inertia ixx="0.01" ixy="0" ixz="0"
+				 iyy="0.01" iyz="0" izz="0.01"/>
   	 	</inertial>
 	<visual name="base_visual">
@@ -85,6 +91,13 @@
 	</collision>
 	</link>
- 	<joint name="base_swivel_joint" type="fixed">
+	<gazebo reference="swivel">
+		<material value="Gazebo/Grey"/>
+	</gazebo>
+ 	<joint name="base_swivel_joint" type="continuous">
 		<origin xyz="-0.185 0 0.055" rpy="0 0 0"/>
+		<axis xyz="0 0 1"/>
+		<anchor xyz="0 0 0"/>
+    <limit effort="100" velocity="100" k_velocity="0" />
+    <joint_properties damping="0.0" friction="0.0" />
 		<parent link="base_link"/>
 		<child link="swivel"/>
@@ -93,8 +106,8 @@
 	<link name="center_hubcap">
 		<inertial>
-			<mass value="0"/>
-			<origin xyz="0 0 0"/>
-			<inertia ixx="1" ixy="0" ixz="0"
-				 iyy="1" iyz="0" izz="1"/>
+			<mass value="0.01"/>
+			<origin xyz="0 0 0"/>
+			<inertia ixx="0.012411765597" ixy="-0.000711733678" ixz="0.00050272983"
+				 iyy="0.015218160428" iyz="-0.000004273467" izz="0.011763977943"/>
   	 	</inertial>
 	<visual name="base_visual">
@@ -114,15 +127,22 @@
 	</collision>
 	</link>
-	<joint name="swivel_hubcap_joint" type="fixed">
+		<gazebo reference="center_hubcap">
+		<material value="Gazebo/Grey"/>
+	</gazebo>
+	<joint name="swivel_hubcap_joint" type="continuous">
 		<origin xyz="-0.026 0 -0.016" rpy="0 0 0"/>
-		<parent link="swivel"/>
+		<axis xyz="0 1 0"/>
+		<anchor xyz="0 0 0"/>
+    <limit effort="100" velocity="100" k_velocity="0" />
+    <joint_properties damping="0.0" friction="0.0" />
+	<parent link="swivel"/>
 		<child link="center_hubcap"/>
 	</joint>
 	<link name="center_wheel">
 		<inertial>
-			<mass value="0"/>
-			<origin xyz="0 0 0"/>
-			<inertia ixx="1" ixy="0" ixz="0"
-				 iyy="1" iyz="0" izz="1"/>
+			<mass value="0.1"/>
+			<origin xyz="0 0 0"/>
+			<inertia ixx="0.012411765597" ixy="-0.000711733678" ixz="0.00050272983"
+				 iyy="0.015218160428" iyz="-0.000004273467" izz="0.011763977943"/>
   	 	</inertial>
 	<visual name="base_visual">
@@ -136,7 +156,8 @@
 	</visual>
 	<collision>
-		<origin xyz="0 0 0" rpy="0 0 0"/>
+		<origin xyz="0 0 0" rpy="${-3.1415927/2.0} 0 0"/>
 		<geometry>
-			<box size="0 0 0"/>
+			<!--<mesh filename="package://p2os_urdf/meshes/p3dx_meshes/center_wheel.stl"/>-->
+			<cylinder radius="0.0375" length="0.01"/>
 		</geometry>
 	</collision>
@@ -147,40 +168,49 @@
 		<child link="center_wheel"/>
 	</joint>
+	<gazebo reference="center_wheel">
+		<material value="Gazebo/Black"/>
+    <elem key="mu1" value="50.0" />
+    <elem key="mu2" value="50.0" />
+    <elem key="kp"  value="100000000.0" />
+    <elem key="kd"  value="1.0" />
+	</gazebo>
 <!-- Right/Left Hubcap + Wheel -->
 <xacro:macro name="p3dx_wheel" params="suffix parent reflect">
 	<link name="p3dx_${suffix}_wheel">
 		<inertial>
-			<mass value="0"/>
-			<origin xyz="0 0 0"/>
-			<inertia ixx="1" ixy="0" ixz="0"
-				 iyy="1" iyz="0" izz="1"/>
-  	 	</inertial>
-	<visual name="base_visual">
-		<origin xyz="0 0 0" rpy="0 0 0"/>
-		<geometry name="pioneer_geom">
-			<mesh filename="package://p2os_urdf/meshes/p3dx_meshes/${suffix}_wheel.stl"/>
-		</geometry>
-		<material name="WheelBlack">
-			<color rgba="0.117 0.117 0.117 1"/>
-		</material>
-	</visual>
-	<collision>
-		<origin xyz="0 0 0" rpy="0 0 0"/>
-		<geometry>
-			<box size="0 0 0"/>
-		</geometry>
-	</collision>
+			<mass value="0.5"/>
+			<origin xyz="0 0 0"/>
+			<inertia ixx="0.012411765597" ixy="0" ixz="0"
+				 iyy="0.015218160428" iyz="0" izz="0.011763977943"/>
+  	 	</inertial>
+		<visual name="base_visual">
+			<origin xyz="0 0 0" rpy="0 0 0"/>
+			<geometry name="pioneer_geom">
+				<mesh filename="package://p2os_urdf/meshes/p3dx_meshes/${suffix}_wheel.stl"/>
+			</geometry>
+			<material name="WheelBlack">
+				<color rgba="0.117 0.117 0.117 1"/>
+			</material>
+		</visual>
+		<collision>
+			<origin xyz="0 0 0" rpy="${-3.1415927/2} 0 0"/>
+			<geometry>
+				<!--<mesh filename="package://p2os_urdf/meshes/p3dx_meshes/${suffix}_wheel.stl"/>-->
+				<cylinder radius="0.09" length="0.01"/>
+			</geometry>
+		</collision>
 	</link>
 	<joint name="base_${suffix}_wheel_joint" type="fixed">
-		<origin xyz="0 ${reflect*0.158} 0.091" rpy="0 0 0"/>
-		<parent link="${parent}"/>
+		<!--<origin xyz="0 ${reflect*0.158} 0.091" rpy="0 0 0"/>-->
+		<origin xyz="0 0 0" rpy="0 0 0"/>
+		<parent link="p3dx_${suffix}_hubcap"/>
 		<child link="p3dx_${suffix}_wheel"/>
 	</joint>
 	<link name="p3dx_${suffix}_hubcap">
 		<inertial>
-			<mass value="0"/>
-			<origin xyz="0 0 0"/>
-			<inertia ixx="1" ixy="0" ixz="0"
-				 iyy="1" iyz="0" izz="1"/>
+			<mass value="0.01"/>
+			<origin xyz="0 0 0"/>
+			<inertia ixx="0.012411765597" ixy="0" ixz="0"
+				 iyy="0.015218160428" iyz="0" izz="0.011763977943"/>
   	 	</inertial>
 	<visual name="base_visual">
@@ -200,9 +230,25 @@
 	</collision>
 	</link>
-	<joint name="base_${suffix}_hubcap_joint" type="fixed">
+  <transmission type="SimpleTransmission" name="${parent}_${suffix}_wheel_trans">
+		<actuator name="base_${suffix}_wheel_motor" />
+    <joint name="base_${suffix}_hubcap_joint" />
+    <mechanicalReduction>${reflect * 624/35 * 80/19}</mechanicalReduction>
+  </transmission>
+	<joint name="base_${suffix}_hubcap_joint" type="continuous">
+		<axis xyz="0 1 0"/>
+		<anchor xyz="0 0 0"/>
+    <limit effort="100" velocity="100" />
+    <joint_properties damping="0.0" friction="0.0" />
 		<origin xyz="0 ${reflect*0.158} 0.091" rpy="0 0 0"/>
 		<parent link="base_link"/>
 		<child link="p3dx_${suffix}_hubcap"/>
 	</joint>
+	<gazebo reference="p3dx_${suffix}_wheel">
+			<material value="Gazebo/Black"/>
+      <elem key="mu1" value="0.5" />
+      <elem key="mu2" value="50.0" />
+      <elem key="kp"  value="100000000.0" />
+      <elem key="kd"  value="1.0" />
+	</gazebo>
 </xacro:macro>
 <xacro:p3dx_wheel suffix="left" parent="base_link" reflect="1"/>
@@ -265,3 +311,33 @@
 		<child link="back_sonar"/>
 	</joint>
+  <gazebo>
+    <controller:differential_position2d name="controller1">
+      <update>100</update>
+      <leftJoint>base_right_hubcap_joint</leftJoint>
+      <rightJoint>base_left_hubcap_joint</rightJoint>
+      <wheelSeparation>0.39</wheelSeparation>
+      <wheelDiameter>0.15</wheelDiameter>
+      <torque>5</torque>
+      <interface:position name="position_iface_0"/>
+    </controller:differential_position2d>
+    <controller:gazebo_ros_p3d name="p3d_base_controller" plugin="libgazebo_ros_p3d.so">
+      <alwaysOn>true</alwaysOn>
+      <updateRate>100.0</updateRate>
+      <bodyName>base_link</bodyName>
+      <topicName>base_pose_ground_truth</topicName>
+      <gaussianNoise>0.01</gaussianNoise>
+      <frameName>map</frameName>
+      <xyzOffsets>0 0 0</xyzOffsets> <!-- initialize odometry for fake localization-->
+      <rpyOffsets>0 0 0</rpyOffsets>
+      <interface:position name="p3d_base_position"/>
+    </controller:gazebo_ros_p3d>
+    <!-- this publishes empty joint_states due to no transmission, but
+         triggering robot_state_puublisher to publish tf between fixed joints in erratic,
+         (e.g. base_laser_link for the base_scan frame) -->
+    <controller:gazebo_ros_controller_manager name="gazebo_ros_controller_manager" plugin="libgazebo_ros_controller_manager.so">
+      <alwaysOn>true</alwaysOn>
+      <updateRate>1000.0</updateRate>
+      <interface:audio name="gazebo_ros_controller_manager_dummy_iface" />
+    </controller:gazebo_ros_controller_manager>
+  </gazebo>
 </robot>
