Commit message: updated p3dx.urdf file

File: p2os/p2os_urdf/defs/pioneer3dx.urdf.xacro (robot description, xacro)
@@ -1,291 +1,315 @@
 <?xml version="1.0"?>
 <robot name="pioneer3dx"
-       xmlns:sensor="http://playerstage.sourceforge.net/gazebo/xmlschema/#sensor"
-       xmlns:controller="http://playerstage.sourceforge.net/gazebo/xmlschema/#controller"
-       xmlns:xacro="http://ros.org/wiki/fixme"
-       xmlns:interface="http://playerstage.sourceforge.net/gazebo/xmlschema/#interface">
-  <property name="M_PI" value="3.14159"/>
-  <property name="base_size_x" value="0.41" />
-  <property name="base_size_y" value="0.385" />
-  <property name="base_size_z" value="0.18" />
-  <property name="wheel_radius" value="0.075" />
-  <property name="wheel_length" value="0.02" />
-  <property name="caster_wheel_offset_y" value="0.17" />
-<!-- chassis -->
-  <link name="base_link">
-    <inertial>
-      <mass value="10" />
-      <origin xyz="-0.1 0 ${base_size_z/2}" />
-      <inertia ixx="1.0" ixy="0.0" ixz="0.0"
-               iyy="1.0" iyz="0.0"
-               izz="1.0" />
-    </inertial>
-    <visual>
-      <origin xyz="-0.045 0 0.148" rpy="0 0 0" />
-      <geometry>
-        <box size="0.22 0.29 0.14" />
-      </geometry>
-    </visual>
-    <collision>
-      <origin xyz="-0.075 0 0.115" rpy="0 0 0" />
-      <geometry>
-        <box size="0.22 0.29 0.14" />
-      </geometry>
-    </collision>
-  </link>
-<!-- top -->
-  <joint name="base_top_joint" type="fixed" >
-    <origin xyz="0 0 0.051" rpy="0 0 0" />
-    <parent link="base_link" />
-    <child link="base_top_link"/>
-  </joint>
-  <link name="base_top_link">
-    <inertial>
-      <mass value="1.0"/>
-      <origin xyz="0 0 ${base_size_z/2}" />
-      <inertia ixx="0.0652232699207" ixy="0.0" ixz="0.0"
-               iyy="0.0669473158652" iyz="0.0"
-               izz="0.0683196351726" />
-    </inertial>
-    <visual>
-      <origin xyz="-0.045 0 0.234" rpy="0 0 0" />
-      <geometry>
-        <box size="${base_size_x} ${base_size_y} 0.01" />
-      </geometry>
-    </visual>
-    <collision>
-      <origin xyz="-0.08 0 0.13" rpy="0 0 0" />
-      <geometry>
-        <box size="${base_size_x} ${base_size_y} 0.01" />
-      </geometry>
-    </collision>
-  </link>
-<!-- swivel -->
-  <joint name="base_swivel_joint" type="continuous" >
-    <origin xyz="0 0 ${wheel_radius}" rpy="0 0 0" />
-    <axis xyz="0 1 0" />
-    <anchor xyz="0 0 0" />
-    <limit effort="100" velocity="100" />
-    <joint_properties damping="0.0" friction="0.0" />
-    <parent link="base_link" />
-    <child link="base_swivel_link" />
-  </joint>
-  <link name="base_swivel_link">
-    <inertial>
-      <mass value="0.1" />
-      <origin xyz=" 0 0 0 " />
-      <inertia  ixx="0.012411765597" ixy="0.0" ixz="0.0"
-                iyy="0.015218160428" iyz="0.0"
-                izz="0.011763977943" />
-    </inertial>
-    <visual>
-      <origin xyz="-0.185 0 0.055" rpy="0 0 0" />
-      <geometry>
-        <cylinder radius="0.0375" length="0.01" />
-      </geometry>
-    </visual>
-    <collision>
-      <origin xyz="0 0 0" rpy="${M_PI/2} 0 0" />
-      <geometry>
-        <cylinder radius="0.0375" length="0.01" />
-      </geometry>
-    </collision>
-  </link>
-<!-- center wheel -->
-  <joint name="p3dx_center_wheel_joint" type="continuous">
-    <origin xyz="0 0 0" rpy="0 0 0" />
-    <axis xyz="0 0 0" />
-    <axis xyz="0 1 0" />
-    <anchor xyz="0 0 0" />
-    <limit effort="100" velocity="100" />
-    <joint_properties damping="0.0" friction="0.0" />
-    <parent link="base_swivel_link" />
-    <child link="p3dx_center_wheel_joint" />
-  </joint>
-  <link name="p3dx_center_wheel_joint">
-    <inertial>
-      <mass value="0.1" />
-      <origin xyz=" 0 0 0 " />
-      <inertia  ixx="0.012411765597" ixy="0.0" ixz="0.0"
-                iyy="0.015218160428" iyz="0.0"
-                izz="0.011763977943" />
-    </inertial>
-    <visual>
-      <origin xyz="-0.211 0.149 0.037" rpy="0 0 0" />
-      <geometry>
-        <cylinder radius="0.0375" length="0.01" />
-      </geometry>
-    </visual>
-    <collision>
-      <origin xyz="0 0 0" rpy="${M_PI/2} 0 0" />
-      <geometry>
-        <cylinder radius="0.0375" length="0.01" />
-      </geometry>
-    </collision>
-  </link>
-<!-- side wheels -->
-  <xacro:macro name="p3dx_wheel" params="suffix parent reflect">
-    <joint name="${parent}_${suffix}_wheel_joint" type="continuous">
-      <origin xyz="0 ${reflect*caster_wheel_offset_y} ${wheel_radius}" rpy="0 0 0" />
-      <axis xyz="0 1 0" />
-      <anchor xyz="0 0 0" />
-      <limit effort="100" velocity="100" />
-      <joint_properties damping="0.0" friction="0.0" />
-      <parent link="${parent}" />
-      <child link="${parent}_${suffix}_wheel_link" />
-    </joint>
-    <link name="${parent}_${suffix}_wheel_link">
-      <inertial>
-        <mass value="0.1" /> <!-- check jmh 20081205 -->
-        <origin xyz=" 0 0 0 " />
-        <inertia  ixx="0.012411765597" ixy="0.0" ixz="0.0"
-                  iyy="0.015218160428" iyz="0.0"
-                  izz="0.011763977943" />
-      </inertial>
-      <visual>
-        <origin xyz="0 ${reflect*0.158} 0.091" rpy="0 0 0" />
-        <geometry>
-          <cylinder radius="${wheel_radius}" length="${wheel_length}" />
-        </geometry>
-      </visual>
-      <collision>
-        <origin xyz="0 0 0" rpy="${M_PI/2} 0 0" />
-        <geometry>
-          <cylinder radius="${wheel_radius}" length="${wheel_length}" />
-        </geometry>
-      </collision>
-    </link>
-    <gazebo reference="${parent}_${suffix}_wheel_link" >
-      <elem key="mu1" value="50.0" />
-      <elem key="mu2" value="50.0" />
-      <elem key="kp"  value="100000000.0" />
-      <elem key="kd"  value="1.0" />
-    </gazebo>
-  </xacro:macro>
-  <xacro:p3dx_wheel suffix="left" parent="base_link" reflect="1"/>
-  <xacro:p3dx_wheel suffix="right" parent="base_link" reflect="-1"/>
-<!-- what is this? -->
-  <joint name="base_caster_box_joint" type="fixed">
-    <origin xyz="0 0 0.051" rpy="0 0 0" />
-    <parent link="base_link" />
-    <child link="base_caster_box_link"/>
-  </joint>
-  <link name="base_caster_box_link">
-    <inertial>
-      <mass value="0.1"/>
-      <origin xyz="0 0 ${base_size_z/2}" />
-      <inertia ixx="0.01" ixy="0.0" ixz="0.0"
-               iyy="0.01" iyz="0.0"
-               izz="0.01" />
-    </inertial>
-    <visual>
-      <origin xyz="-0.23 0 0.08" rpy="0 0 0" />
-      <geometry>
-        <box size="0.09 0.02 0.10" />
-      </geometry>
-    </visual>
-    <collision>
-      <origin xyz="-0.23 0 0.08" rpy="0 0 0" />
-      <geometry>
-        <box size="0.09 0.02 0.10" />
-      </geometry>
-    </collision>
-  </link>
-  <joint name="base_caster_support_joint" type="continuous">
-    <axis xyz="0 0 1" />
-    <anchor xyz="0.01 0 0" />
-    <limit effort="100" velocity="100" k_velocity="0" />
-    <joint_properties damping="0.0" friction="0.0" />
-    <parent link="base_caster_box_link" />
-    <origin xyz="-0.265 0 0.0" rpy="0 0 0" />
-    <child link="base_caster_support_link"/>
-  </joint>
-  <link name="base_caster_support_link">
-    <inertial>
-      <mass value="0.1"/>
-      <origin xyz="0 0 0" />
-      <inertia ixx="0.01" ixy="0.0" ixz="0.0"
-               iyy="0.01" iyz="0.0"
-               izz="0.01" />
-    </inertial>
-    <visual>
-      <origin xyz="0.0 0.0 0.0" rpy="0 0 0" />
-      <geometry>
-        <box size="0.03 0.02 0.06" />
-      </geometry>
-    </visual>
-    <collision>
-      <origin xyz="0.0 0.0 0.0" rpy="0 0 0" />
-      <geometry>
-        <box size="0.03 0.02 0.06" />
-      </geometry>
-    </collision>
-  </link>
-<!-- wheel joints -->
-  <joint name="caster_wheel_joint" type="continuous">
-    <origin xyz="-0.02 0 -0.02" rpy="0 0 0" />
-    <axis xyz="0 1 0" />
-    <anchor xyz="0 0 0" />
-    <limit effort="100" velocity="100" k_velocity="0" />
-    <joint_properties damping="0.0" friction="0.0" />
-    <parent link="base_caster_support_link" />
-    <child link="caster_wheel_link" />
-  </joint>
-  <link name="caster_wheel_link">
-    <inertial>
-      <mass value="0.1" />
-      <origin xyz=" 0 0 0 " />
-      <inertia  ixx="0.012411765597" ixy="-0.000711733678" ixz="0.00050272983"
-                iyy="0.015218160428" iyz="-0.000004273467" izz="0.011763977943" />
-    </inertial>
-    <visual>
-      <origin xyz="0 0 0" rpy="${M_PI/2} 0 0" />
-      <geometry>
-        <cylinder radius="0.03" length="0.01" />
-      </geometry>
-    </visual>
-    <collision>
-      <origin xyz="0 0 0" rpy="${M_PI/2} 0 0" />
-      <geometry>
-        <cylinder radius="0.03" length="0.01" />
-      </geometry>
-    </collision>
-  </link>
-  <gazebo reference="caster_wheel_link">
-    <elem key="mu1" value="50.0" />
-    <elem key="mu2" value="50.0" />
-    <elem key="kp"  value="100000000.0" />
-    <elem key="kd"  value="1.0" />
-  </gazebo>
-<!-- controller -->
-  <gazebo>
-    <controller:differential_position2d name="controller1">
-      <update>100</update>
-      <leftJoint>base_link_right_wheel_joint</leftJoint>
-      <rightJoint>base_link_left_wheel_joint</rightJoint>
-      <wheelSeparation>${caster_wheel_offset_y*2}</wheelSeparation>
-      <wheelDiameter>${wheel_radius*2}</wheelDiameter>
-      <torque>5</torque>
-      <interface:position name="position_iface_0"/>
-    </controller:differential_position2d>
-    <controller:gazebo_ros_p3d name="p3d_base_controller" plugin="libgazebo_ros_p3d.so">
-      <alwaysOn>true</alwaysOn>
-      <updateRate>100.0</updateRate>
-      <bodyName>base_link</bodyName>
-      <topicName>base_pose_ground_truth</topicName>
-      <gaussianNoise>0.01</gaussianNoise>
-      <frameName>map</frameName>
-      <xyzOffsets>25.7 25.7 0</xyzOffsets> <!-- initialize odometry for fake localization-->
-      <rpyOffsets>0 0 0</rpyOffsets>
-      <interface:position name="p3d_base_position"/>
-    </controller:gazebo_ros_p3d>
+	xmlns:sensor="http://playerstage.sourceforge.net/gazebo/xmlschema/#sensor"
+	xmlns:controller="http://playerstage.sourceforge.net/gazebo/xmlschema/#controller"
+	xmlns:interface="http://playerstage.sourceforge.net/gazebo/xmlschema/#interface"
+	xmlns:xacro="http://ros.org/wiki/xacro">
+<!-- Chassis -->
+	<link name="base_link">
+		<inertial>
+			<mass value="3.5"/>
+			<!--<origin xyz="-0.025 0 -0.223"/>-->
+			<origin xyz="0 0 0"/>
+			<inertia ixx="1" ixy="0" ixz="0"
+				 iyy="1" iyz="0"
+				 izz="1"/>
+		</inertial>
+		<visual name="base_visual">
+			<origin xyz="-0.045 0 0.148" rpy="0 0 0"/>
+			<geometry name="pioneer_geom">
+				<mesh filename="package://p2os_urdf/meshes/p3dx_meshes/chassis.stl"/>
+			</geometry>
+			<material name="ChassisRed">
+				<color rgba="0.851 0.0 0.0 1.0"/>
+			</material>
+		</visual>
+		<collision>
+			<origin xyz="0 0 0" rpy="0 0 0"/>
+				<geometry>
+					<box size="0.01 0.01 0.01"/>
+				</geometry>
+		</collision>
+	</link>
+<!-- Top -->
+	<link name="top_plate">
+		<inertial>
+			<mass value="0"/>
+			<origin xyz="0 0 0"/>
+			<inertia ixx="1" ixy="0" ixz="0"
+				 iyy="1" iyz="0"
+ 				izz="1"/>
+		</inertial>
+		<visual name="base_visual">
+			<origin xyz="0 0 0" rpy="0 0 0"/>
+			<geometry name="pioneer_geom">
+				<mesh filename="package://p2os_urdf/meshes/p3dx_meshes/top.stl"/>
+			</geometry>
+			<material name="TopBlack">
+					<color rgba="0.038 0.038 0.038 1.0"/>
+			</material>
+		</visual>
+		<collision>
+			<origin xyz="0 0 0" rpy="0 0 0"/>
+			<geometry>
+				<box size="0 0 0"/>
+			</geometry>
+		</collision>
+	</link>
+	<joint name="base_top_joint" type="fixed">
+		<origin xyz="-0.045 0 0.234" rpy="0 0 0"/>
+		<parent link="base_link"/>
+		<child link="top_plate"/>
+	</joint>
+<!-- Swivel -->
+	<link name="swivel">
+		<inertial>
+			<mass value="0"/>
+			<origin xyz="0 0 0"/>
+			<inertia ixx="1" ixy="0" ixz="0"
+				 iyy="1" iyz="0" izz="1"/>
+  	 	</inertial>
+	<visual name="base_visual">
+		<origin xyz="0 0 0" rpy="0 0 0"/>
+		<geometry name="pioneer_geom">
+			<mesh filename="package://p2os_urdf/meshes/p3dx_meshes/swivel.stl"/>
+		</geometry>
+		<material name="swivel">
+			<color rgba="0.5 0.5 0.5 1"/>
+		</material>
+	</visual>
+	<collision>
+		<origin xyz="0 0 0" rpy="0 0 0"/>
+		<geometry>
+			<box size="0 0 0"/>
+		</geometry>
+	</collision>
+	</link>
+ 	<joint name="base_swivel_joint" type="continuous">
+		<origin xyz="-0.185 0 0.055" rpy="0 0 0"/>
+		<axis xyz="0 0 1" />
+		<anchor xyz="0 0 0" />
+		<limit effort="100" velocity="100" />
+		<joint_properties damping="0.0" friction="0.0" />
+		<parent link="base_link"/>
+		<child link="swivel"/>
+	</joint>
+<!-- Center Wheel + Hubcap -->
+	<link name="center_hubcap">
+		<inertial>
+			<mass value="0"/>
+			<origin xyz="0 0 0"/>
+			<inertia ixx="1" ixy="0" ixz="0"
+				 iyy="1" iyz="0" izz="1"/>
+  	 	</inertial>
+	<visual name="base_visual">
+		<origin xyz="0 0 0" rpy="0 0 0"/>
+		<geometry name="pioneer_geom">
+			<mesh filename="package://p2os_urdf/meshes/p3dx_meshes/center_hubcap.stl"/>
+		</geometry>
+		<material name="swivel">
+			<color rgba="0.5 0.5 0.5 1"/>
+		</material>
+	</visual>
+	<collision>
+		<origin xyz="0 0 0" rpy="0 0 0"/>
+		<geometry>
+			<box size="0 0 0"/>
+		</geometry>
+	</collision>
+	</link>
+	<joint name="swivel_hubcap_joint" type="continuous">
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
File: p2os/p2os_urdf/defs/pioneer3dx.xacro (robot description, xacro)
@@ -1,8 +1,9 @@
 <?xml version="1.0"?>
-<robot xmlns:sensor="http://playerstage.sourceforge.net/gazebo/xmlschema/#sensor"
-       xmlns:controller="http://playerstage.sourceforge.net/gazebo/xmlschema/#controller"
-       xmlns:interface="http://playerstage.sourceforge.net/gazebo/xmlschema/#interface"
-       xmlns:xacro="http://ros.org/wiki/xacro"
-name="pioneer3dx">
+<robot name="pioneer3dx"
+	xmlns:sensor="http://playerstage.sourceforge.net/gazebo/xmlschema/#sensor"
+	xmlns:controller="http://playerstage.sourceforge.net/gazebo/xmlschema/#controller"
+	xmlns:interface="http://playerstage.sourceforge.net/gazebo/xmlschema/#interface"
+	xmlns:xacro="http://ros.org/wiki/xacro"
+	xmlns:xacro="http://ros.org/wiki/fixme">
 <!-- Chassis -->
 	<link name="base_link">

Commit message: working drivable urdf model for gazebo

File: p2os/p2os_urdf/defs/pioneer3dx.urdf.xacro (robot description, xacro)
@@ -5,4 +5,6 @@
 	xmlns:interface="http://playerstage.sourceforge.net/gazebo/xmlschema/#interface"
 	xmlns:xacro="http://ros.org/wiki/xacro">
+  <!--<include filename="$(find p2os_urdf)/defs/materials.xacro"/>-->
+  <include filename="$(find p2os_urdf)/defs/pioneer3dx_wheel.xacro"/>
 <!-- Chassis -->
 	<link name="base_link">
@@ -155,73 +157,4 @@
 		<child link="center_wheel"/>
 	</joint>
-<!-- Right/Left Hubcap + Wheel -->
-<xacro:macro name="p3dx_wheel" params="suffix reflect">
-	<link name="p3dx_${suffix}_wheel">
-		<inertial>
-			<mass value="0"/>
-			<origin xyz="0 0 0"/>
-			<inertia ixx="1" ixy="0" ixz="0"
-				 iyy="1" iyz="0" izz="1"/>
-  	 	</inertial>
-	<visual name="base_visual">
-		<origin xyz="0 0 0" rpy="0 0 0"/>
-		<geometry name="pioneer_geom">
-			<mesh filename="package://p2os_urdf/meshes/p3dx_meshes/${suffix}_wheel.stl"/>
-		</geometry>
-		<material name="WheelBlack">
-			<color rgba="0.117 0.117 0.117 1"/>
-		</material>
-	</visual>
-	<collision>
-		<origin xyz="0 0 0" rpy="0 0 0"/>
-		<geometry>
-			<box size="0 0 0"/>
-		</geometry>
-	</collision>
-	</link>
-	<joint name="base_${suffix}_wheel_joint" type="fixed">
-		<origin xyz="0 0 0" rpy="0 0 0" />
-		<parent link="p3dx_${suffix}_hubcap"/>
-		<child link="p3dx_${suffix}_wheel"/>
-	</joint>
-	<link name="p3dx_${suffix}_hubcap">
-		<inertial>
-			<mass value="0"/>
-			<origin xyz="0 0 0"/>
-			<inertia ixx="1" ixy="0" ixz="0"
-				 iyy="1" iyz="0" izz="1"/>
-  	 	</inertial>
-	<visual name="base_visual">
-		<origin xyz="0 0 0" rpy="0 0 0"/>
-		<geometry name="pioneer_geom">
-			<mesh filename="package://p2os_urdf/meshes/p3dx_meshes/${suffix}_hubcap.stl"/>
-		</geometry>
-		<material name="HubcapYellow">
-			<color rgba="1.0 0.811 0.151 1.0"/>
-		</material>
-	</visual>
-	<collision>
-		<origin xyz="0 0 0" rpy="0 0 0"/>
-		<geometry>
-			<box size="0 0 0"/>
-		</geometry>
-	</collision>
-	</link>
-	<joint name="base_${suffix}_hubcap_joint" type="continuous">
-		<origin xyz="0 ${reflect*0.158} 0.091" rpy="0 0 0" />
-		<axis xyz="0 1 0" />
-		<anchor xyz="0 0 0" />
-		<limit effort="100" velocity="100" />
-		<joint_properties damping="0.0" friction="0.0" />
-		<parent link="base_link"/>
-		<child link="p3dx_${suffix}_hubcap"/>
-	</joint>
-	<gazebo reference="p3dx_${suffix}_hubcap" >
-		<elem key="mu1" value="50.0" />
-		<elem key="mu2" value="50.0" />
-		<elem key="kp"  value="100000000.0" />
-		<elem key="kd"  value="1.0" />
-	</gazebo>
-</xacro:macro>
 <xacro:p3dx_wheel suffix="left" reflect="1"/>
 <xacro:p3dx_wheel suffix="right" reflect="-1"/>

File: p2os/p2os_urdf/defs/pioneer3dx.xacro (robot description, xacro)
@@ -5,4 +5,5 @@
 	xmlns:interface="http://playerstage.sourceforge.net/gazebo/xmlschema/#interface"
 	xmlns:xacro="http://ros.org/wiki/xacro">
+  <include filename="$(find p2os_urdf)/defs/pioneer3dx_wheel.xacro"/>
 <!-- Chassis -->
 	<link name="base_link">
@@ -127,5 +128,5 @@
 	</collision>
 	</link>
-		<gazebo reference="center_hubcap">
+	<gazebo reference="center_hubcap">
 		<material value="Gazebo/Grey"/>
 	</gazebo>
@@ -136,6 +137,6 @@
     <limit effort="100" velocity="100" k_velocity="0" />
     <joint_properties damping="0.0" friction="0.0" />
-	<parent link="swivel"/>
-		<child link="center_hubcap"/>
+	  <parent link="swivel"/>
+		<child link="center_wheel"/>
 	</joint>
 	<link name="center_wheel">
@@ -165,91 +166,14 @@
 	<joint name="center_wheel_joint" type="fixed">
 		<origin xyz="-0.0035 0 -0.001" rpy="0 0 0"/>
-		<parent link="center_hubcap"/>
-		<child link="center_wheel"/>
+		<parent link="center_wheel"/>
+		<child link="center_hubcap"/>
 	</joint>
 	<gazebo reference="center_wheel">
 		<material value="Gazebo/Black"/>
-    <elem key="mu1" value="50.0" />
-    <elem key="mu2" value="50.0" />
-    <elem key="kp"  value="100000000.0" />
+    <elem key="mu1" value="10.0" />
+    <elem key="mu2" value="10.0" />
+    <elem key="kp"  value="1000000.0" />
     <elem key="kd"  value="1.0" />
 	</gazebo>
-<!-- Right/Left Hubcap + Wheel -->
-<xacro:macro name="p3dx_wheel" params="suffix parent reflect">
-	<link name="p3dx_${suffix}_wheel">
-		<inertial>
-			<mass value="0.5"/>
-			<origin xyz="0 0 0"/>
-			<inertia ixx="0.012411765597" ixy="0" ixz="0"
-				 iyy="0.015218160428" iyz="0" izz="0.011763977943"/>
-  	 	</inertial>
-		<visual name="base_visual">
-			<origin xyz="0 0 0" rpy="0 0 0"/>
-			<geometry name="pioneer_geom">
-				<mesh filename="package://p2os_urdf/meshes/p3dx_meshes/${suffix}_wheel.stl"/>
-			</geometry>
-			<material name="WheelBlack">
-				<color rgba="0.117 0.117 0.117 1"/>
-			</material>
-		</visual>
-		<collision>
-			<origin xyz="0 0 0" rpy="${-3.1415927/2} 0 0"/>
-			<geometry>
-				<!--<mesh filename="package://p2os_urdf/meshes/p3dx_meshes/${suffix}_wheel.stl"/>-->
-				<cylinder radius="0.09" length="0.01"/>
-			</geometry>
-		</collision>
-	</link>
-	<joint name="base_${suffix}_wheel_joint" type="fixed">
-		<!--<origin xyz="0 ${reflect*0.158} 0.091" rpy="0 0 0"/>-->
-		<origin xyz="0 0 0" rpy="0 0 0"/>
-		<parent link="p3dx_${suffix}_hubcap"/>
-		<child link="p3dx_${suffix}_wheel"/>
-	</joint>
-	<link name="p3dx_${suffix}_hubcap">
-		<inertial>
-			<mass value="0.01"/>
-			<origin xyz="0 0 0"/>
-			<inertia ixx="0.012411765597" ixy="0" ixz="0"
-				 iyy="0.015218160428" iyz="0" izz="0.011763977943"/>
-  	 	</inertial>
-	<visual name="base_visual">
-		<origin xyz="0 0 0" rpy="0 0 0"/>
-		<geometry name="pioneer_geom">
-			<mesh filename="package://p2os_urdf/meshes/p3dx_meshes/${suffix}_hubcap.stl"/>
-		</geometry>
-		<material name="HubcapYellow">
-			<color rgba="1.0 0.811 0.151 1.0"/>
-		</material>
-	</visual>
-	<collision>
-		<origin xyz="0 0 0" rpy="0 0 0"/>
-		<geometry>
-			<box size="0 0 0"/>
-		</geometry>
-	</collision>
-	</link>
-  <transmission type="SimpleTransmission" name="${parent}_${suffix}_wheel_trans">
-		<actuator name="base_${suffix}_wheel_motor" />
-    <joint name="base_${suffix}_hubcap_joint" />
-    <mechanicalReduction>${reflect * 624/35 * 80/19}</mechanicalReduction>
-  </transmission>
-	<joint name="base_${suffix}_hubcap_joint" type="continuous">
-		<axis xyz="0 1 0"/>
-		<anchor xyz="0 0 0"/>
-    <limit effort="100" velocity="100" />
-    <joint_properties damping="0.0" friction="0.0" />
-		<origin xyz="0 ${reflect*0.158} 0.091" rpy="0 0 0"/>
-		<parent link="base_link"/>
-		<child link="p3dx_${suffix}_hubcap"/>
-	</joint>
-	<gazebo reference="p3dx_${suffix}_wheel">
-			<material value="Gazebo/Black"/>
-      <elem key="mu1" value="0.5" />
-      <elem key="mu2" value="50.0" />
-      <elem key="kp"  value="100000000.0" />
-      <elem key="kd"  value="1.0" />
-	</gazebo>
-</xacro:macro>
 <xacro:p3dx_wheel suffix="left" parent="base_link" reflect="1"/>
 <xacro:p3dx_wheel suffix="right" parent="base_link" reflect="-1"/>
@@ -257,5 +181,5 @@
 	<link name="front_sonar">
 		<inertial>
-			<mass value="0"/>
+			<mass value="0.0001"/>
 			<origin xyz="0 0 0"/>
 			<inertia ixx="1" ixy="0" ixz="0"
@@ -278,4 +202,7 @@
 		</collision>
 	</link>
+	<gazebo reference="front_sonar">
+		<material value="Gazebo/Yellow"/>
+	</gazebo>
 	<joint name="base_front_joint" type="fixed">
 		<origin xyz="-0.198 0 0.208" rpy="0 0 0"/>
@@ -285,10 +212,10 @@
 	<link name="back_sonar">
 		<inertial>
-			<mass value="0"/>
+			<mass value="0.0001"/>
 			<origin xyz="0 0 0"/>
 			<inertia ixx="1" ixy="0" ixz="0"
 				 iyy="1" iyz="0" izz="1"/>
 		</inertial>
-		<visual name="base_visual">
+		<visual name="back_sonar_vis">
 			<origin xyz="0 0 0" rpy="0 0 0"/>
 			<geometry name="pioneer_geom">
@@ -306,4 +233,7 @@
 		</collision>
 	</link>
+	<gazebo reference="back_sonar">
+		<material value="Gazebo/Yellow"/>
+	</gazebo>
 	<joint name="base_back_joint" type="fixed">
 		<origin xyz="0.109 0 0.209" rpy="0 0 0"/>
@@ -314,6 +244,6 @@
     <controller:differential_position2d name="controller1">
       <update>100</update>
-      <leftJoint>base_right_hubcap_joint</leftJoint>
-      <rightJoint>base_left_hubcap_joint</rightJoint>
+      <leftJoint>base_right_wheel_joint</leftJoint>
+      <rightJoint>base_left_wheel_joint</rightJoint>
       <wheelSeparation>0.39</wheelSeparation>
       <wheelDiameter>0.15</wheelDiameter>
