Commit message: edited launch files for new directories

File: bandit_urdf/defs/bandit_defs.xacro (robot description, xacro)
@@ -5,11 +5,11 @@
        xmlns:xacro="http://playerstage.sourceforge.net/gazebo/xmlschema/#interface"
 			 name="bandit">
-	<include filename="$(find interaction_urdf)/defs/common.xacro"/>
+	<include filename="$(find bandit_urdf)/defs/common.xacro"/>
 	<!--<include filename="$(find pr2_description)/urdf/common.xacro"/>-->
-	<include filename="$(find interaction_urdf)/defs/materials.xacro"/>
-	<include filename="$(find interaction_urdf)/defs/torso.xacro"/>
-	<include filename="$(find interaction_urdf)/defs/head.xacro"/>
-	<include filename="$(find interaction_urdf)/defs/shoulder.xacro"/>
-	<include filename="$(find interaction_urdf)/defs/gazebo.urdf.xacro"/>
+	<include filename="$(find bandit_urdf)/defs/materials.xacro"/>
+	<include filename="$(find bandit_urdf)/defs/torso.xacro"/>
+	<include filename="$(find bandit_urdf)/defs/head.xacro"/>
+	<include filename="$(find bandit_urdf)/defs/shoulder.xacro"/>
+	<include filename="$(find bandit_urdf)/defs/gazebo.urdf.xacro"/>
 	<!--<xacro:pr2_base_v0 name="base"/>-->
 	<xacro:bandit_torso name="bandit_torso" parent="/robot/odom">

File: bandit_urdf/defs/bandit_shirt_defs.xacro (robot description, xacro)
@@ -5,13 +5,13 @@
        xmlns:xacro="http://playerstage.sourceforge.net/gazebo/xmlschema/#interface"
 			 name="bandit">
-	<include filename="$(find interaction_urdf)/defs/common.xacro"/>
+	<include filename="$(find bandit_urdf)/defs/common.xacro"/>
 	<!--<include filename="$(find pr2_description)/urdf/common.xacro"/>-->
-	<include filename="$(find interaction_urdf)/defs/materials.xacro"/>
-	<include filename="$(find interaction_urdf)/defs/torso_shirt.xacro"/>
-	<include filename="$(find interaction_urdf)/defs/head.xacro"/>
-	<include filename="$(find interaction_urdf)/defs/shoulder_shirt.xacro"/>
-	<include filename="$(find interaction_urdf)/defs/pioneerbase.xacro"/>
-	<include filename="$(find interaction_urdf)/defs/stage.xacro"/>
-	<include filename="$(find interaction_urdf)/defs/gazebo.urdf.xacro"/>
+	<include filename="$(find bandit_urdf)/defs/materials.xacro"/>
+	<include filename="$(find bandit_urdf)/defs/torso_shirt.xacro"/>
+	<include filename="$(find bandit_urdf)/defs/head.xacro"/>
+	<include filename="$(find bandit_urdf)/defs/shoulder_shirt.xacro"/>
+	<include filename="$(find bandit_urdf)/defs/pioneerbase.xacro"/>
+	<include filename="$(find bandit_urdf)/defs/stage.xacro"/>
+	<include filename="$(find bandit_urdf)/defs/gazebo.urdf.xacro"/>
 	<!--<xacro:pr2_base_v0 name="base"/>-->
 	<xacro:bandit_torso name="bandit_torso" parent="/robot/odom">

File: bandit_urdf/defs/head.xacro (robot description, xacro)
@@ -4,6 +4,6 @@
        xmlns:interface="http://playerstage.sourceforge.net/gazebo/xmlschema/#interface"
        xmlns:xacro="http://ros.org/wiki/xacro">
-  <include filename="$(find interaction_urdf)/defs/head.gazebo.xacro" />
-  <include filename="$(find interaction_urdf)/defs/head.transmission.xacro" />
+  <include filename="$(find bandit_urdf)/defs/head.gazebo.xacro" />
+  <include filename="$(find bandit_urdf)/defs/head.transmission.xacro" />
   <property name="M_PI" value="3.1415926535897931" />
   <property name="neck_height" value="0.076"/>
@@ -38,5 +38,5 @@
         <origin xyz="0 0 0" rpy="${RCon*90} 0 ${RCon*-90}"/>
         <geometry name="${name}_visual_geom">
-					<mesh filename="package://interaction_urdf/meshes/bandit_mesh/neck_small.stl"/>
+					<mesh filename="package://bandit_urdf/meshes/bandit_mesh/neck_small.stl"/>
         </geometry>
 					<material name="NewFace"/>
@@ -76,5 +76,5 @@
 	<!-- -->
         <geometry name="${name}_visual_geom">
-		<mesh filename="package://interaction_urdf/meshes/bandit_mesh/head_small.stl"/>
+		<mesh filename="package://bandit_urdf/meshes/bandit_mesh/head_small.stl"/>
         </geometry>
 					<material name="NewFace"/>
@@ -107,9 +107,9 @@
         <origin xyz="0.035 0 0" rpy="${RCon*90} 0 ${RCon*-90}"/>
         <geometry name="${name}_visual_geom">
-					<mesh filename="package://interaction_urdf/meshes/bandit_mesh/camera_board.stl"/>
+					<mesh filename="package://bandit_urdf/meshes/bandit_mesh/camera_board.stl"/>
         </geometry>
 					<!--  <material name="Silver"/>  -->
 					<material name="texture">
-					<texture filename="package://interaction_urdf/meshes/bandit_mesh/reflect1.jpg"/>
+					<texture filename="package://bandit_urdf/meshes/bandit_mesh/reflect1.jpg"/>
 					</material>
       </visual>
@@ -143,5 +143,5 @@
         <origin xyz="0 0 0" rpy="${RCon*0} 0 ${RCon*-90}"/>
         <geometry name="${name}_visual_geom">
-					<mesh filename="package://interaction_urdf/meshes/bandit_mesh/eyebrow_${side}_small.stl"/>
+					<mesh filename="package://bandit_urdf/meshes/bandit_mesh/eyebrow_${side}_small.stl"/>
         </geometry>
 					<material name="NewEye"/>
@@ -179,5 +179,5 @@
 	<!-- -->
         <geometry name="${name}_visual_geom">
-					<mesh filename="package://interaction_urdf/meshes/bandit_mesh/top_lip_small.STL"/>
+					<mesh filename="package://bandit_urdf/meshes/bandit_mesh/top_lip_small.STL"/>
         </geometry>
 					<material name="LipsPink"/>
@@ -213,5 +213,5 @@
 	<!-- -->
         <geometry name="${name}2_visual_geom">
-					<mesh filename="package://interaction_urdf/meshes/bandit_mesh/bottom_lip_small.stl"/>
+					<mesh filename="package://bandit_urdf/meshes/bandit_mesh/bottom_lip_small.stl"/>
         </geometry>
 					<material name="LipsPink"/>
@@ -266,5 +266,5 @@
 			<origin xyz="0 0 0" rpy="0 0 0"/>
 			<geometry name="pupil_left_geom">
-				<mesh filename="package://interaction_urdf/meshes/bandit_mesh/middle_eye.stl"/>
+				<mesh filename="package://bandit_urdf/meshes/bandit_mesh/middle_eye.stl"/>
 			</geometry>
 		<material name="EyeBlack">

File: bandit_urdf/defs/pioneer2dx.xacro (robot description, xacro)
@@ -5,7 +5,7 @@
        xmlns:xacro="http://playerstage.sourceforge.net/gazebo/xmlschema/#interface"
        name="pioneer2dx">
-  <include filename="$(find interaction_urdf)/defs/common.xacro"/>
+  <include filename="$(find bandit_urdf)/defs/common.xacro"/>
   <!--<include filename="$(find pr2_description)/urdf/common.xacro"/>-->
-  <include filename="$(find interaction_urdf)/defs/materials.xacro"/>
+  <include filename="$(find bandit_urdf)/defs/materials.xacro"/>
  <xacro:macro name="pioneer2dx" params="name">
     <link name="base_link">
@@ -19,5 +19,5 @@
         <origin xyz="0 0 0" rpy="0 0 0"/>
         <geometry>
-          <!--<mesh filename="package://interaction_urdf/meshes/chassis.mesh"/>-->
+          <!--<mesh filename="package://bandit_urdf/meshes/chassis.mesh"/>-->
           <box size="0.445 0.277 0.17"/>
         </geometry>

File: bandit_urdf/defs/pioneerbase.xacro (robot description, xacro)
@@ -18,5 +18,5 @@
 			<origin xyz="0 0 0" rpy="0 0 0"/>
 			<geometry name="8020_geom">
-				<mesh filename="package://interaction_urdf/meshes/bandit_mesh/grid1.stl"/>
+				<mesh filename="package://bandit_urdf/meshes/bandit_mesh/grid1.stl"/>
 			</geometry>
 			<material name="Silver">
@@ -24,5 +24,5 @@
 			</material>
 <!-- 					<material name="texture">
-					<texture filename="package://interaction_urdf/meshes/bandit_mesh/metal1.jpg"/>
+					<texture filename="package://bandit_urdf/meshes/bandit_mesh/metal1.jpg"/>
 					</material> -->
 		</visual>

File: bandit_urdf/defs/shoulder.xacro (robot description, xacro)
@@ -5,5 +5,5 @@
        xmlns:interface="http://playerstage.sourceforge.net/gazebo/xmlschema/#interface"
        xmlns:xacro="http://ros.org/wiki/xacro">
-	<include filename="$(find interaction_urdf)/defs/common.xacro"/>
+	<include filename="$(find bandit_urdf)/defs/common.xacro"/>
 	<property name="PI" value="3.14"/>
 	<property name="RCon" value="0.01744"/>
@@ -39,5 +39,5 @@
 				<origin xyz="0 0 0" rpy="${RCon*90} 0 ${RCon*90}"/>
 				<geometry name="${side}_shoulder_mounting_link_geom">
-					<mesh filename="package://interaction_urdf/meshes/bandit_mesh/shoulder_cover_${side}_small.stl"/>
+					<mesh filename="package://bandit_urdf/meshes/bandit_mesh/shoulder_cover_${side}_small.stl"/>
 					<!--<box size="0.080 0.085 ${shoulder_mounting_link_z}"/>-->
 				</geometry>
@@ -76,5 +76,5 @@
 				<origin xyz="0 ${-reflect*0.0} 0" rpy="0 ${M_PI/2} 0"/>
 				<geometry name="${side}_shoulder_link_geom">
-					<mesh filename="package://interaction_urdf/meshes/bandit_mesh/bicep_cover_${side}_small.stl"/>
+					<mesh filename="package://bandit_urdf/meshes/bandit_mesh/bicep_cover_${side}_small.stl"/>
 				</geometry>
 				<material name="Grey"/>
@@ -112,5 +112,5 @@
 				<origin xyz="0 0 0" rpy="0 ${-M_PI/2} ${-M_PI/2}"/>
 				<geometry name="${side}_bicep_link_geom">
-					<mesh filename="package://interaction_urdf/meshes/bandit_mesh/elbow_cover_${side}_small.stl"/>
+					<mesh filename="package://bandit_urdf/meshes/bandit_mesh/elbow_cover_${side}_small.stl"/>
 					<!--<box size="0.050 0.050 0.065"/>-->
 				</geometry>
@@ -149,5 +149,5 @@
 				<!--<origin xyz="0 0 -0.025" rpy="0 ${M_PI/2} ${M_PI/2}"/>-->
 				<geometry name="${side}_forearm_link_geom">
-					<mesh filename="package://interaction_urdf/meshes/bandit_mesh/forearm_cover_${side}_small.stl"/>
+					<mesh filename="package://bandit_urdf/meshes/bandit_mesh/forearm_cover_${side}_small.stl"/>
 					<!--<box size="0.068 0.065 0.095"/>-->
 				</geometry>
@@ -187,5 +187,5 @@
 				<origin xyz="0 0 -0.01" rpy="${M_PI/2} 0 ${M_PI/2}"/>
 				<geometry name="${side}_wrist_link_geom">
-					<mesh filename="package://interaction_urdf/meshes/bandit_mesh/wrist_cover_${side}_small.stl"/>
+					<mesh filename="package://bandit_urdf/meshes/bandit_mesh/wrist_cover_${side}_small.stl"/>
 					<!--<box size="0.054 0.054 0.055"/>-->
 				</geometry>
@@ -224,5 +224,5 @@
 				<origin xyz="0 0 -.00" rpy="${M_PI/2} 0 0"/>
 				<geometry name="${side}_hand_link_geom">
-					<mesh filename="package://interaction_urdf/meshes/bandit_mesh/${side}_hand_small.stl"/>
+					<mesh filename="package://bandit_urdf/meshes/bandit_mesh/${side}_hand_small.stl"/>
 					<!--<box size="0.060 0.060 0.080"/>-->
 				</geometry>
@@ -260,5 +260,5 @@
 				<origin xyz="0 0 0" rpy="${M_PI/2} ${-M_PI/2} 0"/>
 				<geometry name="${side}_thumb_link_geom">
-					<mesh filename="package://interaction_urdf/meshes/bandit_mesh/${side}_thumb_small.stl"/>
+					<mesh filename="package://bandit_urdf/meshes/bandit_mesh/${side}_thumb_small.stl"/>
 					<!--<box size="0.030 0.025 0.06"/>-->
 				</geometry>

File: bandit_urdf/defs/shoulder_shirt.xacro (robot description, xacro)
@@ -5,5 +5,5 @@
        xmlns:interface="http://playerstage.sourceforge.net/gazebo/xmlschema/#interface"
        xmlns:xacro="http://ros.org/wiki/xacro">
-	<include filename="$(find interaction_urdf)/defs/common.xacro"/>
+	<include filename="$(find bandit_urdf)/defs/common.xacro"/>
 	<property name="PI" value="3.14"/>
 	<property name="RCon" value="0.01744"/>
@@ -39,5 +39,5 @@
 				<origin xyz="0 0 0" rpy="${RCon*90} 0 ${RCon*90}"/>
 				<geometry name="${side}_shoulder_mounting_link_geom">
-					<mesh filename="package://interaction_urdf/meshes/bandit_mesh/shoulder_cover_${side}_small.stl"/>
+					<mesh filename="package://bandit_urdf/meshes/bandit_mesh/shoulder_cover_${side}_small.stl"/>
 					<!--<box size="0.080 0.085 ${shoulder_mounting_link_z}"/>-->
 				</geometry>
@@ -76,5 +76,5 @@
 				<origin xyz="0 ${-reflect*0.0} 0" rpy="0 ${M_PI/2} 0"/>
 				<geometry name="${side}_shoulder_link_geom">
-					<mesh filename="package://interaction_urdf/meshes/bandit_mesh/bicep_cover_${side}_small.stl"/>
+					<mesh filename="package://bandit_urdf/meshes/bandit_mesh/bicep_cover_${side}_small.stl"/>
 				</geometry>
 				<material name="SweaterRed"/>
@@ -112,5 +112,5 @@
 				<origin xyz="0 0 0" rpy="0 ${-M_PI/2} ${-M_PI/2}"/>
 				<geometry name="${side}_bicep_link_geom">
-					<mesh filename="package://interaction_urdf/meshes/bandit_mesh/elbow_cover_${side}_small.stl"/>
+					<mesh filename="package://bandit_urdf/meshes/bandit_mesh/elbow_cover_${side}_small.stl"/>
 					<!--<box size="0.050 0.050 0.065"/>-->
 				</geometry>
@@ -149,5 +149,5 @@
 				<!--<origin xyz="0 0 -0.025" rpy="0 ${M_PI/2} ${M_PI/2}"/>-->
 				<geometry name="${side}_forearm_link_geom">
-					<mesh filename="package://interaction_urdf/meshes/bandit_mesh/forearm_cover_${side}_small.stl"/>
+					<mesh filename="package://bandit_urdf/meshes/bandit_mesh/forearm_cover_${side}_small.stl"/>
 					<!--<box size="0.068 0.065 0.095"/>-->
 				</geometry>
@@ -187,5 +187,5 @@
 				<origin xyz="0 0 -0.01" rpy="${M_PI/2} 0 ${M_PI/2}"/>
 				<geometry name="${side}_wrist_link_geom">
-					<mesh filename="package://interaction_urdf/meshes/bandit_mesh/wrist_cover_${side}_small.stl"/>
+					<mesh filename="package://bandit_urdf/meshes/bandit_mesh/wrist_cover_${side}_small.stl"/>
 					<!--<box size="0.054 0.054 0.055"/>-->
 				</geometry>
@@ -224,5 +224,5 @@
 				<origin xyz="0 0 -.00" rpy="${M_PI/2} 0 0"/>
 				<geometry name="${side}_hand_link_geom">
-					<mesh filename="package://interaction_urdf/meshes/bandit_mesh/${side}_hand_small.stl"/>
+					<mesh filename="package://bandit_urdf/meshes/bandit_mesh/${side}_hand_small.stl"/>
 					<!--<box size="0.060 0.060 0.080"/>-->
 				</geometry>
@@ -260,5 +260,5 @@
 				<origin xyz="0 0 0" rpy="${M_PI/2} ${-M_PI/2} 0"/>
 				<geometry name="${side}_thumb_link_geom">
-					<mesh filename="package://interaction_urdf/meshes/bandit_mesh/${side}_thumb_small.stl"/>
+					<mesh filename="package://bandit_urdf/meshes/bandit_mesh/${side}_thumb_small.stl"/>
 					<!--<box size="0.030 0.025 0.06"/>-->
 				</geometry>

File: bandit_urdf/defs/stage.xacro (robot description, xacro)
@@ -18,8 +18,8 @@
 			<origin xyz="0 0 0" rpy="0 0 ${M_PI/2}"/>
 			<geometry name="background_geom">
-				<mesh filename="package://interaction_urdf/meshes/bandit_mesh/background.stl"/>
+				<mesh filename="package://bandit_urdf/meshes/bandit_mesh/background.stl"/>
 			</geometry>
 			<material name="BackgroundFile">
-				<texture filename="package://interaction_urdf/meshes/bandit_mesh/background6.jpg"/>
+				<texture filename="package://bandit_urdf/meshes/bandit_mesh/background6.jpg"/>
 			</material>
 		</visual>
@@ -48,8 +48,8 @@
 			<origin xyz="0 0 0" rpy="0 0 ${M_PI/2}"/>
 			<geometry name="ground_geom">
-				<mesh filename="package://interaction_urdf/meshes/bandit_mesh/background.stl"/>
+				<mesh filename="package://bandit_urdf/meshes/bandit_mesh/background.stl"/>
 			</geometry>
 			<material name="groundFile">
-				<texture filename="package://interaction_urdf/meshes/bandit_mesh/background5.jpg"/>
+				<texture filename="package://bandit_urdf/meshes/bandit_mesh/background5.jpg"/>
 			</material>
 		</visual>

File: bandit_urdf/defs/torso.xacro (robot description, xacro)
@@ -4,5 +4,5 @@
        xmlns:interface="http://playerstage.sourceforge.net/gazebo/xmlschema/#interface"
        xmlns:xacro="http://ros.org/wiki/xacro">
-  <include filename="$(find interaction_urdf)/defs/torso.gazebo.xacro" />
+  <include filename="$(find bandit_urdf)/defs/torso.gazebo.xacro" />
 	<xacro:macro name="bandit_torso" params="name parent *origin">
   <!--
@@ -28,5 +28,5 @@
     	  <!--<origin xyz="0 0 0.05" rpy="${M_PI/2} 0 ${M_PI/2}"/>-->
       	<geometry name="${name}_geom">
-					<mesh filename="package://interaction_urdf/meshes/bandit_mesh/body_small.stl"/>
+					<mesh filename="package://bandit_urdf/meshes/bandit_mesh/body_small.stl"/>
   	    <!--  <box size="0 0 0"/>-->
 	      </geometry>
@@ -52,5 +52,5 @@
 			<origin xyz="0 0 0" rpy="0 ${M_PI/2} ${M_PI}"/>
 			<geometry name="pioneer_geom">
-				<mesh filename="package://interaction_urdf/meshes/bandit_mesh/stop_switch_small.STL"/>
+				<mesh filename="package://bandit_urdf/meshes/bandit_mesh/stop_switch_small.STL"/>
 			</geometry>
 			<material name="Red"/>

File: bandit_urdf/defs/torso_shirt.xacro (robot description, xacro)
@@ -4,5 +4,5 @@
        xmlns:interface="http://playerstage.sourceforge.net/gazebo/xmlschema/#interface"
        xmlns:xacro="http://ros.org/wiki/xacro">
-  <include filename="$(find interaction_urdf)/defs/torso.gazebo.xacro" />
+  <include filename="$(find bandit_urdf)/defs/torso.gazebo.xacro" />
 	<xacro:macro name="bandit_torso" params="name parent *origin">
 	  <link name = "${name}_link">
@@ -16,5 +16,5 @@
 		    	<origin xyz="0 0 0.0" rpy="${M_PI/2} 0 ${M_PI/2}"/>
 		      	<geometry name="${name}_geom">
-			  <mesh filename="package://interaction_urdf/meshes/bandit_mesh/body_small.stl"/>
+			  <mesh filename="package://bandit_urdf/meshes/bandit_mesh/body_small.stl"/>
 			</geometry>
 	    	</visual>
@@ -44,5 +44,5 @@
 			<origin xyz="0.002 0.003 0" rpy="${M_PI/2} 0 ${M_PI/2}"/>
 			<geometry name="bandit_logo_geom">
-			<mesh filename="package://interaction_urdf/meshes/bandit_mesh/logo2.stl"/>
+			<mesh filename="package://bandit_urdf/meshes/bandit_mesh/logo2.stl"/>
 				<!--<box size="0.005 0.05 0.05"/>-->
 			</geometry>
@@ -69,5 +69,5 @@
 			<origin xyz="0 0 0" rpy="0 ${M_PI/2} ${M_PI}"/>
 			<geometry name="pioneer_geom">
-				<mesh filename="package://interaction_urdf/meshes/bandit_mesh/stop_switch_small.STL"/>
+				<mesh filename="package://bandit_urdf/meshes/bandit_mesh/stop_switch_small.STL"/>
 			</geometry>
 			<material name="Red"/>

Commit message: bandit_urdf: start making bandit_shirt and bandit model the same; minor fix for elbow-shoulder length

File: bandit_urdf/defs/bandit_defs.xacro (robot description, xacro)
@@ -6,5 +6,7 @@
 			 name="bandit">
 	<include filename="$(find bandit_urdf)/defs/common.xacro"/>
-	<!--<include filename="$(find pr2_description)/urdf/common.xacro"/>-->
+  <!-- uncomment the below line for the bandit_shirt materials -->
+  <!--	<include filename="$(find bandit_urdf)/defs/shirt_materials.xacro"/>-->
+  <!-- use the below line for the regular bandit materials -->
 	<include filename="$(find bandit_urdf)/defs/materials.xacro"/>
 	<include filename="$(find bandit_urdf)/defs/torso.xacro"/>
@@ -25,5 +27,5 @@
 	</xacro:bandit_shoulder>
   	<xacro:bandit_shoulder side="right" parent="bandit_torso_link" reflect="-1">
-		<origin xyz="0 -${body_width/2+.01} 0" rpy="0 0 0"/>
+		<origin xyz="0 ${-(body_width/2+.01)} 0" rpy="0 0 0"/>
 	</xacro:bandit_shoulder>
 </robot>

File: bandit_urdf/defs/bandit_shirt_defs.xacro (robot description, xacro)
@@ -7,5 +7,5 @@
 	<include filename="$(find bandit_urdf)/defs/common.xacro"/>
 	<include filename="$(find pr2_description)/urdf/common.xacro"/>
-	<include filename="$(find bandit_urdf)/defs/materials.xacro"/>
+	<include filename="$(find bandit_urdf)/defs/shirt_materials.xacro"/>
 	<include filename="$(find bandit_urdf)/defs/torso_shirt.xacro"/>
 	<include filename="$(find bandit_urdf)/defs/head.xacro"/>

File: bandit_urdf/defs/shirt_materials.xacro (robot description, xacro)
@@ -2,5 +2,5 @@
 <robot>
   <material name="torso">
-    <color rgba="0.3 0.3 0.3 1.0"/>
+    <color rgba="0.45 0.0 0.0 1.0"/>
   </material>
   <material name="Blue">

File: bandit_urdf/defs/shoulder.xacro (robot description, xacro)
@@ -89,5 +89,5 @@
 		<!-- -->
 		<joint name="${side}_shoulder_bicep_joint" type="revolute">
-			<origin xyz="0 0 ${-.150}"/>
+			<origin xyz="0 0 ${-.161}"/>
 			<axis xyz="0 0 ${reflect}"/>
 			<parent link="${side}_shoulder_link"/>
@@ -110,5 +110,5 @@
 			</inertial>
 			<visual name="${side}_bicep_link_visual">
-				<origin xyz="0 0 0" rpy="0 ${-M_PI/2} ${-M_PI/2}"/>
+				<origin xyz="0 0 0.0" rpy="0 ${-M_PI/2} ${M_PI/2}"/>
 				<geometry name="${side}_bicep_link_geom">
 					<mesh filename="package://bandit_urdf/meshes/bandit_mesh/elbow_cover_${side}_small.stl"/>

File: bandit_urdf/defs/torso.xacro (robot description, xacro)
@@ -24,5 +24,5 @@
     	</inertial>
 	    <visual name="${name}_visual">
-  	    <material name="Grey2"/>
+  	    <material name="torso"/>
     	  <origin xyz="0 0 0.0" rpy="${M_PI/2} 0 ${M_PI/2}"/>
     	  <!--<origin xyz="0 0 0.05" rpy="${M_PI/2} 0 ${M_PI/2}"/>-->
