Commit message: added new xacro for screws on 8020

File: bandit_urdf/defs/bandit_shirt_defs.xacro (robot description, xacro)
@@ -12,4 +12,5 @@
 	<include filename="$(find bandit_urdf)/defs/shoulder_shirt.xacro"/>
 	<include filename="$(find bandit_urdf)/defs/pioneerbase.xacro"/>
+	<include filename="$(find bandit_urdf)/defs/screws.xacro"/>
 	<include filename="$(find bandit_urdf)/defs/stage.xacro"/>
 	<include filename="$(find bandit_urdf)/defs/gazebo.urdf.xacro"/>

File: bandit_urdf/defs/pioneerbase.xacro (robot description, xacro)
@@ -23,5 +23,5 @@
 					<color rgba="0.65 0.65 0.65 1.0"/>
 			</material>
-<!-- 					<material name="texture">
+<!-- 					<material name="GridTexture">
 					<texture filename="package://bandit_urdf/meshes/bandit_mesh/metal1.jpg"/>
 					</material> -->
@@ -201,6 +201,9 @@
 			<mesh filename="package://p2os_urdf/meshes/p3dx_meshes/${suffix}_wheel.stl"/>
 		</geometry>
-		<material name="WheelBlack">
+<!--		<material name="WheelBlack">
 			<color rgba="0.117 0.117 0.117 1"/>
+		</material>-->
+		<material name="TireTexture">
+			<texture filename="package://bandit_urdf/meshes/bandit_mesh/tire1.jpg"/>
 		</material>
 	</visual>
@@ -277,4 +280,30 @@
 		<child link="front_sonar"/>
 	</joint>
+	<link name="front_sonar_rim">
+		<inertial>
+			<mass value="0"/>
+			<origin xyz="0 0 0"/>
+			<inertia ixx="1" ixy="0" ixz="0"
+				 iyy="1" iyz="0" izz="1"/>
+		</inertial>
+		<visual name="base_visual">
+			<origin xyz="0 0 0" rpy="0 0 0"/>
+			<geometry name="pioneer_geom">
+				<mesh filename="package://p2os_urdf/meshes/p3dx_meshes/front_rim.stl"/>
+			</geometry>
+			<material name="Black"/>
+		</visual>
+		<collision>
+			<origin xyz="0 0 0" rpy="0 0 0"/>
+			<geometry>
+				<box size="0 0 0"/>
+			</geometry>
+		</collision>
+	</link>
+	<joint name="base_front_rim_joint" type="fixed">
+		<origin xyz="-0.198 0 0.208" rpy="0 0 0"/>
+		<parent link="chassis_link"/>
+		<child link="front_sonar_rim"/>
+	</joint>
 	<link name="back_sonar">
 		<inertial>
@@ -305,3 +334,29 @@
 		<child link="back_sonar"/>
 	</joint>
+	<link name="back_sonar_rim">
+		<inertial>
+			<mass value="0"/>
+			<origin xyz="0 0 0"/>
+			<inertia ixx="1" ixy="0" ixz="0"
+				 iyy="1" iyz="0" izz="1"/>
+		</inertial>
+		<visual name="base_visual">
+			<origin xyz="0 0 0" rpy="0 0 0"/>
+			<geometry name="pioneer_geom">
+				<mesh filename="package://p2os_urdf/meshes/p3dx_meshes/back_rim.stl"/>
+			</geometry>
+			<material name="Black"/>
+		</visual>
+		<collision>
+			<origin xyz="0 0 0" rpy="0 0 0"/>
+			<geometry>
+				<box size="0 0 0"/>
+			</geometry>
+		</collision>
+	</link>
+	<joint name="base_back_rim_joint" type="fixed">
+		<origin xyz="0.109 0 0.209" rpy="0 0 0"/>
+		<parent link="chassis_link"/>
+		<child link="back_sonar_rim"/>
+	</joint>
 </robot>

Commit message: cleaned up code

File: bandit_urdf/defs/bandit_shirt_defs.xacro (robot description, xacro)
@@ -19,9 +19,4 @@
 		<origin xyz="-0.00 0 ${body_height/2}" rpy="0 0 0"/>
 	</xacro:bandit_torso>
-<!--DANGO
-  <xacro:bandit_logo name="bandit_logo" parent="bandit_torso_link">
-    <origin xyz="0 1.0 0" rpy="0 0 0"/>
-  </xacro:bandit_logo>
-DANGO-->
 	<xacro:bandit_head name="bandit_head" parent="bandit_torso_link">
 			<origin xyz="0 0 ${body_height/2 +neck_height/2+0.01}" rpy="0 0 0"/>

File: bandit_urdf/defs/shoulder_shirt.xacro (robot description, xacro)
@@ -90,5 +90,5 @@
 		<joint name="${side}_shoulder_bicep_joint" type="revolute">
 			<origin xyz="0 0 ${-.150}"/>
-			<axis xyz="0 0 1"/>
+			<axis xyz="0 0 ${reflect}"/>
 			<parent link="${side}_shoulder_link"/>
 			<child link="${side}_bicep_link"/>
@@ -163,7 +163,7 @@
 		<!-- -->
 		<joint name="${side}_forearm_wrist_joint" type="revolute">
-			<origin xyz="0 0 -0.145"/>
+			<origin xyz="0 0 -0.145" rpy="0 0 ${-reflect * M_PI/2}"/>
 			<!--<origin xyz="0 0 -0.090"/>-->
-			<axis xyz="0 0 1"/>
+			<axis xyz="0 0 ${reflect}"/>
 			<parent link="${side}_forearm_link"/>
 			<child link="${side}_wrist_link"/>
