Commit message: bandit_urdf: file clean up

File: bandit_urdf/defs/bandit_shirt_defs.xacro (robot description, xacro)
@@ -8,7 +8,8 @@
 	<include filename="$(find pr2_description)/urdf/common.xacro"/>
 	<include filename="$(find bandit_urdf)/defs/shirt_materials.xacro"/>
-	<include filename="$(find bandit_urdf)/defs/torso_shirt.xacro"/>
+	<include filename="$(find bandit_urdf)/defs/torso.xacro"/>
+	<include filename="$(find bandit_urdf)/defs/logo.xacro"/>
 	<include filename="$(find bandit_urdf)/defs/head.xacro"/>
-	<include filename="$(find bandit_urdf)/defs/shoulder_shirt.xacro"/>
+	<include filename="$(find bandit_urdf)/defs/shoulder.xacro"/>
 	<include filename="$(find bandit_urdf)/defs/pioneerbase.xacro"/>
 	<include filename="$(find bandit_urdf)/defs/screws.xacro"/>

File: bandit_urdf/defs/head.xacro (robot description, xacro)
@@ -40,10 +40,10 @@
 					<mesh filename="package://bandit_urdf/meshes/bandit_mesh/neck_small.stl"/>
         </geometry>
-					<material name="NewFace"/>
-      </visual>
-      <collision name="${name}_collision">
-        <origin xyz="0 0 0" rpy="${RCon*90} 0 ${RCon*90}"/>
-        <geometry name="${name}_visual_geom">
-		<box size="0.063 0.063 0.076"/>
+					<material name="Neck"/>
+      </visual>
+      <collision name="${name}_collision">
+        <origin xyz="0 0 0" rpy="${RCon*90} 0 ${RCon*90}"/>
+        <geometry name="${name}_visual_geom">
+		<box size="0 0 0"/>
         </geometry>
       </collision>
@@ -78,10 +78,10 @@
 		<mesh filename="package://bandit_urdf/meshes/bandit_mesh/head_small.stl"/>
         </geometry>
-					<material name="NewFace"/>
-      </visual>
-      <collision name="${name}_collision">
-         <origin xyz="0 0 0" rpy="0 0 0 " />
-        <geometry name="${name}_visual_geom">
-		<box size="0.127 0.158 0.175"/>
+					<material name="Head"/>
+      </visual>
+      <collision name="${name}_collision">
+         <origin xyz="0.008 0 0.055" rpy="0 0 0 " />
+        <geometry name="${name}_visual_geom">
+		<box size="0.147 0.156 0.16"/>
         </geometry>
       </collision>
@@ -111,5 +111,5 @@
 					<!--  <material name="Silver"/>  -->
 					<material name="texture">
-					<texture filename="package://bandit_urdf/meshes/bandit_mesh/reflect1.jpg"/>
+					<texture filename="package://bandit_urdf/meshes/bandit_mesh/gradients/reflect1.jpg"/>
 					</material>
       </visual>
@@ -117,5 +117,5 @@
          <origin xyz="0 0 0" rpy="0 0 0 " />
         <geometry name="${name}_visual_geom">
-					<box size="0.127 0.158 0.175"/>
+					<box size="0 0 0"/>
         </geometry>
       </collision>
@@ -141,9 +141,9 @@
       </inertial>
       <visual name="${name}_visual">
-        <origin xyz="0 0 0" rpy="${RCon*0} 0 ${RCon*-90}"/>
+        <origin xyz="0 0 0" rpy="0 0 ${RCon*-90}"/>
         <geometry name="${name}_visual_geom">
 					<mesh filename="package://bandit_urdf/meshes/bandit_mesh/eyebrow_${side}_small.stl"/>
         </geometry>
-					<material name="NewEye"/>
+					<material name="Eyebrows"/>
       </visual>
       <collision name="${name}_collision">
@@ -174,5 +174,5 @@
       </inertial>
       <visual name="${name}_visual">
-        <origin xyz="0 0 .002" rpy="${RCon*0} 0 ${RCon*-90}"/>
+        <origin xyz="0 0 .002" rpy="0 0 ${RCon*-90}"/>
         <!--<origin xyz="0 0 -0.035" rpy="${RCon*0} 0 ${RCon*-90}"/>-->
         <!--<origin xyz="0 0 0" rpy="${RCon*90} 0 ${RCon*90}"/>-->
@@ -181,10 +181,10 @@
 					<mesh filename="package://bandit_urdf/meshes/bandit_mesh/top_lip_small.STL"/>
         </geometry>
-					<material name="LipsPink"/>
-      </visual>
-      <collision name="${name}_collision">
-         <origin xyz="0 0 0" rpy="0 0 0 " />
-        <geometry name="${name}_visual_geom">
-					<box size="0.127 0.158 0.175"/>
+					<material name="Lips"/>
+      </visual>
+      <collision name="${name}_collision">
+         <origin xyz="0 0 0" rpy="0 0 0 " />
+        <geometry name="${name}_visual_geom">
+					<box size="0 0 0"/>
         </geometry>
       </collision>
@@ -215,10 +215,10 @@
 					<mesh filename="package://bandit_urdf/meshes/bandit_mesh/bottom_lip_small.stl"/>
         </geometry>
-					<material name="LipsPink"/>
+					<material name="Lips"/>
       </visual>
       <collision name="${name}2_collision">
          <origin xyz="0 0 0" rpy="0 0 0 " />
         <geometry name="${name}2_visual_geom">
-					<box size="0.127 0.158 0.175"/>
+					<box size="0 0 0"/>
         </geometry>
       </collision>
@@ -267,5 +267,5 @@
 				<mesh filename="package://bandit_urdf/meshes/bandit_mesh/middle_eye.stl"/>
 			</geometry>
-		<material name="EyeBlack">
+		<material name="Pupil">
 			<color rgba="0 0 0 1"/>
 		</material>

File: bandit_urdf/defs/materials.xacro (robot description, xacro)
@@ -1,6 +1,6 @@
 <?xml version="1.0"?>
 <robot>
-  <material name="torso">
-    <color rgba="0.3 0.3 0.3 1.0"/>
+  <material name="Red">
+    <color rgba="0.8 0.0 0.0 1.0"/>
   </material>
   <material name="Blue">
@@ -10,22 +10,4 @@
     <color rgba="0.0 0.8 0.0 1.0"/>
   </material>
-  <material name="Grey">
-    <color rgba="0.5 0.5 0.5 1.0"/>
-  </material>
-  <material name="Grey2">
-    <color rgba="0.3 0.3 0.3 1.0"/>
-  </material>
-  <material name="Red">
-    <color rgba="0.8 0.0 0.0 1.0"/>
-  </material>
-  <material name="FaceGrey">
-    <color rgba="0.35 0.35 0.35 1.0"/>
-  </material>
-  <material name="White">
-    <color rgba="1.0 1.0 1.0 1.0"/>
-  </material>
-  <material name="SweaterRed">
-    <color rgba="0.45 0.0 0.0 1.0"/>
-  </material>
   <material name="Yellow">
     <color rgba="0.75 0.75 0.0 1.0"/>
@@ -34,12 +16,36 @@
     <color rgba="0 0 0 1.0"/>
   </material>
-  <material name="LipsPink">
+  <material name="White">
+    <color rgba="1.0 1.0 1.0 1.0"/>
+  </material>
+  <material name="Head">
+    <color rgba="0.5 0.5 0.5 1.0"/>
+  </material>
+  <material name="Eyebrows">
+    <color rgba="0.35 0.35 0.35 1.0"/>
+  </material>
+  <material name="Pupil">
+    <color rgba="0 0 0 1"/>
+  </material>
+  <material name="Lips">
     <color rgba="0.737 0.118 0.193 1.0"/>
   </material>
-  <material name="NewFace">
+  <material name="Neck">
     <color rgba="0.5 0.5 0.5 1.0"/>
   </material>
-  <material name="NewEye">
-    <color rgba="0.35 0.35 0.35 1.0"/>
+  <material name="Torso">
+    <color rgba="0.3 0.3 0.3 1.0"/>
+  </material>
+  <material name="Arms">
+    <color rgba="0.5 0.5 0.5 1.0"/>
+  </material>
+  <material name="Wrist">
+    <color rgba="0.5 0.5 0.5 1.0"/>
+  </material>
+  <material name="Hands">
+    <color rgba="0.5 0.5 0.5 1.0"/>
+  </material>
+  <material name="SweaterRed">
+    <color rgba="0.45 0.0 0.0 1.0"/>
   </material>
 </robot>

File: bandit_urdf/defs/pioneerbase.xacro (robot description, xacro)
@@ -205,5 +205,5 @@
 		</material>-->
 		<material name="TireTexture">
-			<texture filename="package://bandit_urdf/meshes/bandit_mesh/tire1.jpg"/>
+			<texture filename="package://bandit_urdf/meshes/bandit_mesh/gradients/tire1.jpg"/>
 		</material>
 	</visual>

File: bandit_urdf/defs/screws.xacro (robot description, xacro)
@@ -17,5 +17,5 @@
 			<origin xyz="0 0 0" rpy="0 0 0"/>
 			<geometry name="pioneer_geom">
-				<mesh filename="package://bandit_urdf/meshes/bandit_mesh/screw.stl"/>
+				<mesh filename="package://bandit_urdf/meshes/bandit_mesh/screw_small.stl"/>
 			</geometry>
 			<material name="Black"/>
@@ -43,5 +43,5 @@
 			<origin xyz="0 0 0" rpy="0 0 0"/>
 			<geometry name="pioneer_geom">
-				<mesh filename="package://bandit_urdf/meshes/bandit_mesh/screw.stl"/>
+				<mesh filename="package://bandit_urdf/meshes/bandit_mesh/screw_small.stl"/>
 			</geometry>
 			<material name="Black"/>
@@ -69,5 +69,5 @@
 			<origin xyz="0 0 0" rpy="0 0 0"/>
 			<geometry name="pioneer_geom">
-				<mesh filename="package://bandit_urdf/meshes/bandit_mesh/screw.stl"/>
+				<mesh filename="package://bandit_urdf/meshes/bandit_mesh/screw_small.stl"/>
 			</geometry>
 			<material name="Black"/>
@@ -95,5 +95,5 @@
 			<origin xyz="0 0 0" rpy="0 0 0"/>
 			<geometry name="pioneer_geom">
-				<mesh filename="package://bandit_urdf/meshes/bandit_mesh/screw.stl"/>
+				<mesh filename="package://bandit_urdf/meshes/bandit_mesh/screw_small.stl"/>
 			</geometry>
 			<material name="Black"/>
@@ -121,5 +121,5 @@
 			<origin xyz="0 0 0" rpy="0 0 0"/>
 			<geometry name="pioneer_geom">
-				<mesh filename="package://bandit_urdf/meshes/bandit_mesh/screw.stl"/>
+				<mesh filename="package://bandit_urdf/meshes/bandit_mesh/screw_small.stl"/>
 			</geometry>
 			<material name="Black"/>
@@ -147,5 +147,5 @@
 			<origin xyz="0 0 0" rpy="0 0 0"/>
 			<geometry name="pioneer_geom">
-				<mesh filename="package://bandit_urdf/meshes/bandit_mesh/screw.stl"/>
+				<mesh filename="package://bandit_urdf/meshes/bandit_mesh/screw_small.stl"/>
 			</geometry>
 			<material name="Black"/>
@@ -173,5 +173,5 @@
 			<origin xyz="0 0 0" rpy="0 0 0"/>
 			<geometry name="pioneer_geom">
-				<mesh filename="package://bandit_urdf/meshes/bandit_mesh/screw.stl"/>
+				<mesh filename="package://bandit_urdf/meshes/bandit_mesh/screw_small.stl"/>
 			</geometry>
 			<material name="Black"/>
@@ -199,5 +199,5 @@
 			<origin xyz="0 0 0" rpy="0 0 0"/>
 			<geometry name="pioneer_geom">
-				<mesh filename="package://bandit_urdf/meshes/bandit_mesh/screw.stl"/>
+				<mesh filename="package://bandit_urdf/meshes/bandit_mesh/screw_small.stl"/>
 			</geometry>
 			<material name="Black"/>
@@ -225,5 +225,5 @@
 			<origin xyz="0 0 0" rpy="0 0 0"/>
 			<geometry name="pioneer_geom">
-				<mesh filename="package://bandit_urdf/meshes/bandit_mesh/screw.stl"/>
+				<mesh filename="package://bandit_urdf/meshes/bandit_mesh/screw_small.stl"/>
 			</geometry>
 			<material name="Black"/>
@@ -251,5 +251,5 @@
 			<origin xyz="0 0 0" rpy="0 0 0"/>
 			<geometry name="pioneer_geom">
-				<mesh filename="package://bandit_urdf/meshes/bandit_mesh/screw.stl"/>
+				<mesh filename="package://bandit_urdf/meshes/bandit_mesh/screw_small.stl"/>
 			</geometry>
 			<material name="Black"/>
@@ -277,5 +277,5 @@
 			<origin xyz="0 0 0" rpy="0 0 0"/>
 			<geometry name="pioneer_geom">
-				<mesh filename="package://bandit_urdf/meshes/bandit_mesh/screw.stl"/>
+				<mesh filename="package://bandit_urdf/meshes/bandit_mesh/screw_small.stl"/>
 			</geometry>
 			<material name="Black"/>
@@ -303,5 +303,5 @@
 			<origin xyz="0 0 0" rpy="0 0 0"/>
 			<geometry name="pioneer_geom">
-				<mesh filename="package://bandit_urdf/meshes/bandit_mesh/screw.stl"/>
+				<mesh filename="package://bandit_urdf/meshes/bandit_mesh/screw_small.stl"/>
 			</geometry>
 			<material name="Black"/>
@@ -329,5 +329,5 @@
 			<origin xyz="0 0 0" rpy="0 0 0"/>
 			<geometry name="pioneer_geom">
-				<mesh filename="package://bandit_urdf/meshes/bandit_mesh/screw.stl"/>
+				<mesh filename="package://bandit_urdf/meshes/bandit_mesh/screw_small.stl"/>
 			</geometry>
 			<material name="Black"/>
@@ -355,5 +355,5 @@
 			<origin xyz="0 0 0" rpy="0 0 0"/>
 			<geometry name="pioneer_geom">
-				<mesh filename="package://bandit_urdf/meshes/bandit_mesh/screw.stl"/>
+				<mesh filename="package://bandit_urdf/meshes/bandit_mesh/screw_small.stl"/>
 			</geometry>
 			<material name="Black"/>
@@ -381,5 +381,5 @@
 			<origin xyz="0 0 0" rpy="0 0 0"/>
 			<geometry name="pioneer_geom">
-				<mesh filename="package://bandit_urdf/meshes/bandit_mesh/screw.stl"/>
+				<mesh filename="package://bandit_urdf/meshes/bandit_mesh/screw_small.stl"/>
 			</geometry>
 			<material name="Black"/>
@@ -407,5 +407,5 @@
 			<origin xyz="0 0 0" rpy="0 0 0"/>
 			<geometry name="pioneer_geom">
-				<mesh filename="package://bandit_urdf/meshes/bandit_mesh/screw.stl"/>
+				<mesh filename="package://bandit_urdf/meshes/bandit_mesh/screw_small.stl"/>
 			</geometry>
 			<material name="Black"/>
@@ -433,5 +433,5 @@
 			<origin xyz="0 0 0" rpy="0 0 0"/>
 			<geometry name="pioneer_geom">
-				<mesh filename="package://bandit_urdf/meshes/bandit_mesh/screw.stl"/>
+				<mesh filename="package://bandit_urdf/meshes/bandit_mesh/screw_small.stl"/>
 			</geometry>
 			<material name="Black"/>
@@ -459,5 +459,5 @@
 			<origin xyz="0 0 0" rpy="0 0 0"/>
 			<geometry name="pioneer_geom">
-				<mesh filename="package://bandit_urdf/meshes/bandit_mesh/screw.stl"/>
+				<mesh filename="package://bandit_urdf/meshes/bandit_mesh/screw_small.stl"/>
 			</geometry>
 			<material name="Black"/>
@@ -485,5 +485,5 @@
 			<origin xyz="0 0 0" rpy="0 0 0"/>
 			<geometry name="pioneer_geom">
-				<mesh filename="package://bandit_urdf/meshes/bandit_mesh/screw.stl"/>
+				<mesh filename="package://bandit_urdf/meshes/bandit_mesh/screw_small.stl"/>
 			</geometry>
 			<material name="Black"/>
@@ -511,5 +511,5 @@
 			<origin xyz="0 0 0" rpy="0 0 0"/>
 			<geometry name="pioneer_geom">
-				<mesh filename="package://bandit_urdf/meshes/bandit_mesh/screw.stl"/>
+				<mesh filename="package://bandit_urdf/meshes/bandit_mesh/screw_small.stl"/>
 			</geometry>
 			<material name="Black"/>
@@ -537,5 +537,5 @@
 			<origin xyz="0 0 0" rpy="0 0 0"/>
 			<geometry name="pioneer_geom">
-				<mesh filename="package://bandit_urdf/meshes/bandit_mesh/screw.stl"/>
+				<mesh filename="package://bandit_urdf/meshes/bandit_mesh/screw_small.stl"/>
 			</geometry>
 			<material name="Black"/>
@@ -563,5 +563,5 @@
 			<origin xyz="0 0 0" rpy="0 0 0"/>
 			<geometry name="pioneer_geom">
-				<mesh filename="package://bandit_urdf/meshes/bandit_mesh/screw.stl"/>
+				<mesh filename="package://bandit_urdf/meshes/bandit_mesh/screw_small.stl"/>
 			</geometry>
 			<material name="Black"/>
@@ -589,5 +589,5 @@
 			<origin xyz="0 0 0" rpy="0 0 0"/>
 			<geometry name="pioneer_geom">
-				<mesh filename="package://bandit_urdf/meshes/bandit_mesh/screw.stl"/>
+				<mesh filename="package://bandit_urdf/meshes/bandit_mesh/screw_small.stl"/>
 			</geometry>
 			<material name="Black"/>
@@ -615,5 +615,5 @@
 			<origin xyz="0 0 0" rpy="0 0 0"/>
 			<geometry name="pioneer_geom">
-				<mesh filename="package://bandit_urdf/meshes/bandit_mesh/screw.stl"/>
+				<mesh filename="package://bandit_urdf/meshes/bandit_mesh/screw_small.stl"/>
 			</geometry>
 			<material name="Black"/>
@@ -641,5 +641,5 @@
 			<origin xyz="0 0 0" rpy="0 0 0"/>
 			<geometry name="pioneer_geom">
-				<mesh filename="package://bandit_urdf/meshes/bandit_mesh/screw.stl"/>
+				<mesh filename="package://bandit_urdf/meshes/bandit_mesh/screw_small.stl"/>
 			</geometry>
 			<material name="Black"/>
@@ -667,5 +667,5 @@
 			<origin xyz="0 0 0" rpy="0 0 0"/>
 			<geometry name="pioneer_geom">
-				<mesh filename="package://bandit_urdf/meshes/bandit_mesh/screw.stl"/>
+				<mesh filename="package://bandit_urdf/meshes/bandit_mesh/screw_small.stl"/>
 			</geometry>
 			<material name="Black"/>
@@ -693,5 +693,5 @@
 			<origin xyz="0 0 0" rpy="0 0 0"/>
 			<geometry name="pioneer_geom">
-				<mesh filename="package://bandit_urdf/meshes/bandit_mesh/screw.stl"/>
+				<mesh filename="package://bandit_urdf/meshes/bandit_mesh/screw_small.stl"/>
 			</geometry>
 			<material name="Black"/>
@@ -719,5 +719,5 @@
 			<origin xyz="0 0 0" rpy="0 0 0"/>
 			<geometry name="pioneer_geom">
-				<mesh filename="package://bandit_urdf/meshes/bandit_mesh/screw.stl"/>
+				<mesh filename="package://bandit_urdf/meshes/bandit_mesh/screw_small.stl"/>
 			</geometry>
 			<material name="Black"/>
@@ -745,5 +745,5 @@
 			<origin xyz="0 0 0" rpy="0 0 0"/>
 			<geometry name="pioneer_geom">
-				<mesh filename="package://bandit_urdf/meshes/bandit_mesh/screw.stl"/>
+				<mesh filename="package://bandit_urdf/meshes/bandit_mesh/screw_small.stl"/>
 			</geometry>
 			<material name="Black"/>
@@ -771,5 +771,5 @@
 			<origin xyz="0 0 0" rpy="0 0 0"/>
 			<geometry name="pioneer_geom">
-				<mesh filename="package://bandit_urdf/meshes/bandit_mesh/screw.stl"/>
+				<mesh filename="package://bandit_urdf/meshes/bandit_mesh/screw_small.stl"/>
 			</geometry>
 			<material name="Black"/>
@@ -797,5 +797,5 @@
 			<origin xyz="0 0 0" rpy="0 0 0"/>
 			<geometry name="pioneer_geom">
-				<mesh filename="package://bandit_urdf/meshes/bandit_mesh/screw.stl"/>
+				<mesh filename="package://bandit_urdf/meshes/bandit_mesh/screw_small.stl"/>
 			</geometry>
 			<material name="Black"/>
@@ -823,5 +823,5 @@
 			<origin xyz="0 0 0" rpy="0 0 0"/>
 			<geometry name="pioneer_geom">
-				<mesh filename="package://bandit_urdf/meshes/bandit_mesh/screw.stl"/>
+				<mesh filename="package://bandit_urdf/meshes/bandit_mesh/screw_small.stl"/>
 			</geometry>
 			<material name="Black"/>
@@ -852,5 +852,5 @@
 			<origin xyz="0 0 0" rpy="0 0 0"/>
 			<geometry name="pioneer_geom">
-				<mesh filename="package://bandit_urdf/meshes/bandit_mesh/screw.stl"/>
+				<mesh filename="package://bandit_urdf/meshes/bandit_mesh/screw_small.stl"/>
 			</geometry>
 			<material name="Black"/>
@@ -878,5 +878,5 @@
 			<origin xyz="0 0 0" rpy="0 0 0"/>
 			<geometry name="pioneer_geom">
-				<mesh filename="package://bandit_urdf/meshes/bandit_mesh/screw.stl"/>
+				<mesh filename="package://bandit_urdf/meshes/bandit_mesh/screw_small.stl"/>
 			</geometry>
 			<material name="Black"/>
@@ -904,5 +904,5 @@
 			<origin xyz="0 0 0" rpy="0 0 0"/>
 			<geometry name="pioneer_geom">
-				<mesh filename="package://bandit_urdf/meshes/bandit_mesh/screw.stl"/>
+				<mesh filename="package://bandit_urdf/meshes/bandit_mesh/screw_small.stl"/>
 			</geometry>
 			<material name="Black"/>
@@ -930,5 +930,5 @@
 			<origin xyz="0 0 0" rpy="0 0 0"/>
 			<geometry name="pioneer_geom">
-				<mesh filename="package://bandit_urdf/meshes/bandit_mesh/screw.stl"/>
+				<mesh filename="package://bandit_urdf/meshes/bandit_mesh/screw_small.stl"/>
 			</geometry>
 			<material name="Black"/>

File: bandit_urdf/defs/shirt_materials.xacro (robot description, xacro)
@@ -1,6 +1,6 @@
 <?xml version="1.0"?>
 <robot>
-  <material name="torso">
-    <color rgba="0.45 0.0 0.0 1.0"/>
+  <material name="Red">
+    <color rgba="0.8 0.0 0.0 1.0"/>
   </material>
   <material name="Blue">
@@ -10,22 +10,4 @@
     <color rgba="0.0 0.8 0.0 1.0"/>
   </material>
-  <material name="Grey">
-    <color rgba="0.5 0.5 0.5 1.0"/>
-  </material>
-  <material name="Grey2">
-    <color rgba="0.3 0.3 0.3 1.0"/>
-  </material>
-  <material name="Red">
-    <color rgba="0.8 0.0 0.0 1.0"/>
-  </material>
-  <material name="FaceGrey">
-    <color rgba="0.35 0.35 0.35 1.0"/>
-  </material>
-  <material name="White">
-    <color rgba="1.0 1.0 1.0 1.0"/>
-  </material>
-  <material name="SweaterRed">
-    <color rgba="0.45 0.0 0.0 1.0"/>
-  </material>
   <material name="Yellow">
     <color rgba="0.75 0.75 0.0 1.0"/>
@@ -34,12 +16,36 @@
     <color rgba="0 0 0 1.0"/>
   </material>
-  <material name="LipsPink">
+  <material name="White">
+    <color rgba="1.0 1.0 1.0 1.0"/>
+  </material>
+  <material name="Head">
+    <color rgba="0.5 0.5 0.5 1.0"/>
+  </material>
+  <material name="Eyebrows">
+    <color rgba="0.35 0.35 0.35 1.0"/>
+  </material>
+  <material name="Pupil">
+    <color rgba="0 0 0 1"/>
+  </material>
+  <material name="Lips">
     <color rgba="0.737 0.118 0.193 1.0"/>
   </material>
-  <material name="NewFace">
+  <material name="Neck">
     <color rgba="0.5 0.5 0.5 1.0"/>
   </material>
-  <material name="NewEye">
-    <color rgba="0.35 0.35 0.35 1.0"/>
+  <material name="Torso">
+    <color rgba="0.45 0.0 0.0 1.0"/>
+  </material>
+  <material name="Arms">
+    <color rgba="0.45 0.0 0.0 1.0"/>
+  </material>
+  <material name="Wrist">
+    <color rgba="0.5 0.5 0.5 1.0"/>
+  </material>
+  <material name="Hands">
+    <color rgba="0.5 0.5 0.5 1.0"/>
+  </material>
+  <material name="SweaterRed">
+    <color rgba="0.45 0.0 0.0 1.0"/>
   </material>
 </robot>

File: bandit_urdf/defs/shoulder.xacro (robot description, xacro)
@@ -42,10 +42,10 @@
 					<!--<box size="0.080 0.085 ${shoulder_mounting_link_z}"/>-->
 				</geometry>
-				<material name="Grey"/>
+				<material name="Arms"/>
 			</visual>
 			<collision name="${side}_shoulder_mounting_link_collision">
-				<origin xyz="0 0 0" rpy="${RCon*90} 0 ${RCon*90}"/>
+				<origin xyz="0 0 -0.05" rpy="${RCon*90} 0 ${RCon*90}"/>
 				<geometry name="${side}_shoulder_mounting_link_geom">
-					<box size="0.080 0.085 ${shoulder_mounting_link_z}"/>
+					<box size="0.105 0.175 ${shoulder_mounting_link_z}"/>
 				</geometry>
 			</collision>
@@ -78,10 +78,10 @@
 					<mesh filename="package://bandit_urdf/meshes/bandit_mesh/bicep_cover_${side}_small.stl"/>
 				</geometry>
-				<material name="Grey"/>
+				<material name="Arms"/>
 			</visual>
 			<collision name="${side}_shoulder_link_collision">
 				<origin xyz="0 0 -0.04" rpy="0 0 0"/>
 				<geometry name="${side}_shoulder_link_geom">
-					<box size="0.080 0.080 ${shoulder_link_z}"/>
+					<box size="0 0 0"/>
 				</geometry>
 			</collision>
@@ -115,10 +115,10 @@
 					<!--<box size="0.050 0.050 0.065"/>-->
 				</geometry>
-				<material name="Grey"/>
+				<material name="Arms"/>
 			</visual>
 			<collision name="${side}_bicep_link_collision">
 				<origin xyz="0 0 0" rpy="0 0 0"/>
 				<geometry name="${side}_bicep_link_geom">
-					<box size="0.050 0.050 0.065"/>
+					<box size="0 0 0"/>
 				</geometry>
 			</collision>
@@ -152,10 +152,10 @@
 					<!--<box size="0.068 0.065 0.095"/>-->
 				</geometry>
-				<material name="Grey"/>
+				<material name="Arms"/>
 			</visual>
 			<collision name="${side}_forearm_link_collision">
-				<origin xyz="0 0 -0.025" rpy="0 0 0"/>
+				<origin xyz="0 0 -0.075" rpy="0 0 0"/>
 				<geometry name="${side}_forearm_link_geom">
-					<box size="0.068 0.065 0.095"/>
+					<box size="0 0 0"/>
 				</geometry>
 			</collision>
@@ -190,10 +190,10 @@
 					<!--<box size="0.054 0.054 0.055"/>-->
 				</geometry>
-				<material name="Grey"/>
+				<material name="Wrist"/>
 			</visual>
 			<collision name="">
 				<origin xyz="0 0 -0.01" rpy="0 0 0"/>
 				<geometry name="${side}_wrist_link_geom">
-					<box size="0.054 0.054 0.055"/>
+					<box size="0 0 0"/>
 				</geometry>
 			</collision>
@@ -227,10 +227,10 @@
 					<!--<box size="0.060 0.060 0.080"/>-->
 				</geometry>
-				<material name="Grey"/>
+				<material name="Hands"/>
 			</visual>
 			<collision name="${side}_hand_link_collision">
-				<origin xyz="0 0 -.03" rpy="0 0 0"/>
+				<origin xyz="-0.05 0 -0.06" rpy="0 0 0"/>
 				<geometry name="${side}_hand_link_geom">
-					<box size="0.060 0.060 0.080"/>
+					<box size="0.03 0.06 0.080"/>
 				</geometry>
 			</collision>
@@ -263,5 +263,5 @@
 					<!--<box size="0.030 0.025 0.06"/>-->
 				</geometry>
-				<material name="Grey"/>
+				<material name="Hands"/>
 			</visual>
 			<collision name="${side}_thumb_link_collision">
