Commit message: bandit_urdf: file clean up

File: bandit_urdf/defs/stage.xacro (robot description, xacro)
@@ -21,5 +21,5 @@
 			</geometry>
 			<material name="BackgroundFile">
-				<texture filename="package://bandit_urdf/meshes/bandit_mesh/background6.jpg"/>
+				<texture filename="package://bandit_urdf/meshes/bandit_mesh/gradients/background6.jpg"/>
 			</material>
 		</visual>
@@ -51,5 +51,5 @@
 			</geometry>
 			<material name="groundFile">
-				<texture filename="package://bandit_urdf/meshes/bandit_mesh/background5.jpg"/>
+				<texture filename="package://bandit_urdf/meshes/bandit_mesh/gradients/background5.jpg"/>
 			</material>
 		</visual>

File: bandit_urdf/defs/torso.xacro (robot description, xacro)
@@ -24,5 +24,5 @@
     	</inertial>
 	    <visual name="${name}_visual">
-  	    <material name="torso"/>
+  	    <material name="Torso"/>
     	  <origin xyz="0 0 0.0" rpy="${M_PI/2} 0 ${M_PI/2}"/>
     	  <!--<origin xyz="0 0 0.05" rpy="${M_PI/2} 0 ${M_PI/2}"/>-->
@@ -33,7 +33,7 @@
     	</visual>
 	    <collision>
-  	    <origin xyz="0 0 0" rpy="0 0 0"/>
+  	    <origin xyz="0 0 -0.067" rpy="0 0 0"/>
     	  <geometry>
-      	  <box size="0 0 0"/>
+      	  <box size="0.152 0.228 0.282"/>
 	      </geometry>
   	  </collision>
