Commit message: bandit_urdf: updated def files

File: bandit_urdf/defs/screws.xacro (robot description, xacro)
@@ -17,5 +17,5 @@
 			<origin xyz="0 0 0" rpy="0 0 0"/>
 			<geometry name="pioneer_geom">
-				<mesh filename="package://bandit_urdf/meshes/bandit_mesh/screw_small.stl"/>
+				<mesh filename="package://bandit_urdf/meshes/bandit_mesh/screw.stl"/>
 			</geometry>
 			<material name="Black"/>
@@ -43,5 +43,5 @@
 			<origin xyz="0 0 0" rpy="0 0 0"/>
 			<geometry name="pioneer_geom">
-				<mesh filename="package://bandit_urdf/meshes/bandit_mesh/screw_small.stl"/>
+				<mesh filename="package://bandit_urdf/meshes/bandit_mesh/screw.stl"/>
 			</geometry>
 			<material name="Black"/>
@@ -69,5 +69,5 @@
 			<origin xyz="0 0 0" rpy="0 0 0"/>
 			<geometry name="pioneer_geom">
-				<mesh filename="package://bandit_urdf/meshes/bandit_mesh/screw_small.stl"/>
+				<mesh filename="package://bandit_urdf/meshes/bandit_mesh/screw.stl"/>
 			</geometry>
 			<material name="Black"/>
@@ -95,5 +95,5 @@
 			<origin xyz="0 0 0" rpy="0 0 0"/>
 			<geometry name="pioneer_geom">
-				<mesh filename="package://bandit_urdf/meshes/bandit_mesh/screw_small.stl"/>
+				<mesh filename="package://bandit_urdf/meshes/bandit_mesh/screw.stl"/>
 			</geometry>
 			<material name="Black"/>
@@ -121,5 +121,5 @@
 			<origin xyz="0 0 0" rpy="0 0 0"/>
 			<geometry name="pioneer_geom">
-				<mesh filename="package://bandit_urdf/meshes/bandit_mesh/screw_small.stl"/>
+				<mesh filename="package://bandit_urdf/meshes/bandit_mesh/screw.stl"/>
 			</geometry>
 			<material name="Black"/>
@@ -147,5 +147,5 @@
 			<origin xyz="0 0 0" rpy="0 0 0"/>
 			<geometry name="pioneer_geom">
-				<mesh filename="package://bandit_urdf/meshes/bandit_mesh/screw_small.stl"/>
+				<mesh filename="package://bandit_urdf/meshes/bandit_mesh/screw.stl"/>
 			</geometry>
 			<material name="Black"/>
@@ -173,5 +173,5 @@
 			<origin xyz="0 0 0" rpy="0 0 0"/>
 			<geometry name="pioneer_geom">
-				<mesh filename="package://bandit_urdf/meshes/bandit_mesh/screw_small.stl"/>
+				<mesh filename="package://bandit_urdf/meshes/bandit_mesh/screw.stl"/>
 			</geometry>
 			<material name="Black"/>
@@ -199,5 +199,5 @@
 			<origin xyz="0 0 0" rpy="0 0 0"/>
 			<geometry name="pioneer_geom">
-				<mesh filename="package://bandit_urdf/meshes/bandit_mesh/screw_small.stl"/>
+				<mesh filename="package://bandit_urdf/meshes/bandit_mesh/screw.stl"/>
 			</geometry>
 			<material name="Black"/>
@@ -225,5 +225,5 @@
 			<origin xyz="0 0 0" rpy="0 0 0"/>
 			<geometry name="pioneer_geom">
-				<mesh filename="package://bandit_urdf/meshes/bandit_mesh/screw_small.stl"/>
+				<mesh filename="package://bandit_urdf/meshes/bandit_mesh/screw.stl"/>
 			</geometry>
 			<material name="Black"/>
@@ -251,5 +251,5 @@
 			<origin xyz="0 0 0" rpy="0 0 0"/>
 			<geometry name="pioneer_geom">
-				<mesh filename="package://bandit_urdf/meshes/bandit_mesh/screw_small.stl"/>
+				<mesh filename="package://bandit_urdf/meshes/bandit_mesh/screw.stl"/>
 			</geometry>
 			<material name="Black"/>
@@ -277,5 +277,5 @@
 			<origin xyz="0 0 0" rpy="0 0 0"/>
 			<geometry name="pioneer_geom">
-				<mesh filename="package://bandit_urdf/meshes/bandit_mesh/screw_small.stl"/>
+				<mesh filename="package://bandit_urdf/meshes/bandit_mesh/screw.stl"/>
 			</geometry>
 			<material name="Black"/>
@@ -303,5 +303,5 @@
 			<origin xyz="0 0 0" rpy="0 0 0"/>
 			<geometry name="pioneer_geom">
-				<mesh filename="package://bandit_urdf/meshes/bandit_mesh/screw_small.stl"/>
+				<mesh filename="package://bandit_urdf/meshes/bandit_mesh/screw.stl"/>
 			</geometry>
 			<material name="Black"/>
@@ -329,5 +329,5 @@
 			<origin xyz="0 0 0" rpy="0 0 0"/>
 			<geometry name="pioneer_geom">
-				<mesh filename="package://bandit_urdf/meshes/bandit_mesh/screw_small.stl"/>
+				<mesh filename="package://bandit_urdf/meshes/bandit_mesh/screw.stl"/>
 			</geometry>
 			<material name="Black"/>
@@ -355,5 +355,5 @@
 			<origin xyz="0 0 0" rpy="0 0 0"/>
 			<geometry name="pioneer_geom">
-				<mesh filename="package://bandit_urdf/meshes/bandit_mesh/screw_small.stl"/>
+				<mesh filename="package://bandit_urdf/meshes/bandit_mesh/screw.stl"/>
 			</geometry>
 			<material name="Black"/>
@@ -381,5 +381,5 @@
 			<origin xyz="0 0 0" rpy="0 0 0"/>
 			<geometry name="pioneer_geom">
-				<mesh filename="package://bandit_urdf/meshes/bandit_mesh/screw_small.stl"/>
+				<mesh filename="package://bandit_urdf/meshes/bandit_mesh/screw.stl"/>
 			</geometry>
 			<material name="Black"/>
@@ -407,5 +407,5 @@
 			<origin xyz="0 0 0" rpy="0 0 0"/>
 			<geometry name="pioneer_geom">
-				<mesh filename="package://bandit_urdf/meshes/bandit_mesh/screw_small.stl"/>
+				<mesh filename="package://bandit_urdf/meshes/bandit_mesh/screw.stl"/>
 			</geometry>
 			<material name="Black"/>
@@ -433,5 +433,5 @@
 			<origin xyz="0 0 0" rpy="0 0 0"/>
 			<geometry name="pioneer_geom">
-				<mesh filename="package://bandit_urdf/meshes/bandit_mesh/screw_small.stl"/>
+				<mesh filename="package://bandit_urdf/meshes/bandit_mesh/screw.stl"/>
 			</geometry>
 			<material name="Black"/>
@@ -459,5 +459,5 @@
 			<origin xyz="0 0 0" rpy="0 0 0"/>
 			<geometry name="pioneer_geom">
-				<mesh filename="package://bandit_urdf/meshes/bandit_mesh/screw_small.stl"/>
+				<mesh filename="package://bandit_urdf/meshes/bandit_mesh/screw.stl"/>
 			</geometry>
 			<material name="Black"/>
@@ -485,5 +485,5 @@
 			<origin xyz="0 0 0" rpy="0 0 0"/>
 			<geometry name="pioneer_geom">
-				<mesh filename="package://bandit_urdf/meshes/bandit_mesh/screw_small.stl"/>
+				<mesh filename="package://bandit_urdf/meshes/bandit_mesh/screw.stl"/>
 			</geometry>
 			<material name="Black"/>
@@ -511,5 +511,5 @@
 			<origin xyz="0 0 0" rpy="0 0 0"/>
 			<geometry name="pioneer_geom">
-				<mesh filename="package://bandit_urdf/meshes/bandit_mesh/screw_small.stl"/>
+				<mesh filename="package://bandit_urdf/meshes/bandit_mesh/screw.stl"/>
 			</geometry>
 			<material name="Black"/>
@@ -537,5 +537,5 @@
 			<origin xyz="0 0 0" rpy="0 0 0"/>
 			<geometry name="pioneer_geom">
-				<mesh filename="package://bandit_urdf/meshes/bandit_mesh/screw_small.stl"/>
+				<mesh filename="package://bandit_urdf/meshes/bandit_mesh/screw.stl"/>
 			</geometry>
 			<material name="Black"/>
@@ -563,5 +563,5 @@
 			<origin xyz="0 0 0" rpy="0 0 0"/>
 			<geometry name="pioneer_geom">
-				<mesh filename="package://bandit_urdf/meshes/bandit_mesh/screw_small.stl"/>
+				<mesh filename="package://bandit_urdf/meshes/bandit_mesh/screw.stl"/>
 			</geometry>
 			<material name="Black"/>
@@ -589,5 +589,5 @@
 			<origin xyz="0 0 0" rpy="0 0 0"/>
 			<geometry name="pioneer_geom">
-				<mesh filename="package://bandit_urdf/meshes/bandit_mesh/screw_small.stl"/>
+				<mesh filename="package://bandit_urdf/meshes/bandit_mesh/screw.stl"/>
 			</geometry>
 			<material name="Black"/>
@@ -615,5 +615,5 @@
 			<origin xyz="0 0 0" rpy="0 0 0"/>
 			<geometry name="pioneer_geom">
-				<mesh filename="package://bandit_urdf/meshes/bandit_mesh/screw_small.stl"/>
+				<mesh filename="package://bandit_urdf/meshes/bandit_mesh/screw.stl"/>
 			</geometry>
 			<material name="Black"/>
@@ -641,5 +641,5 @@
 			<origin xyz="0 0 0" rpy="0 0 0"/>
 			<geometry name="pioneer_geom">
-				<mesh filename="package://bandit_urdf/meshes/bandit_mesh/screw_small.stl"/>
+				<mesh filename="package://bandit_urdf/meshes/bandit_mesh/screw.stl"/>
 			</geometry>
 			<material name="Black"/>
@@ -667,5 +667,5 @@
 			<origin xyz="0 0 0" rpy="0 0 0"/>
 			<geometry name="pioneer_geom">
-				<mesh filename="package://bandit_urdf/meshes/bandit_mesh/screw_small.stl"/>
+				<mesh filename="package://bandit_urdf/meshes/bandit_mesh/screw.stl"/>
 			</geometry>
 			<material name="Black"/>
@@ -693,5 +693,5 @@
 			<origin xyz="0 0 0" rpy="0 0 0"/>
 			<geometry name="pioneer_geom">
-				<mesh filename="package://bandit_urdf/meshes/bandit_mesh/screw_small.stl"/>
+				<mesh filename="package://bandit_urdf/meshes/bandit_mesh/screw.stl"/>
 			</geometry>
 			<material name="Black"/>
@@ -719,5 +719,5 @@
 			<origin xyz="0 0 0" rpy="0 0 0"/>
 			<geometry name="pioneer_geom">
-				<mesh filename="package://bandit_urdf/meshes/bandit_mesh/screw_small.stl"/>
+				<mesh filename="package://bandit_urdf/meshes/bandit_mesh/screw.stl"/>
 			</geometry>
 			<material name="Black"/>
@@ -745,5 +745,5 @@
 			<origin xyz="0 0 0" rpy="0 0 0"/>
 			<geometry name="pioneer_geom">
-				<mesh filename="package://bandit_urdf/meshes/bandit_mesh/screw_small.stl"/>
+				<mesh filename="package://bandit_urdf/meshes/bandit_mesh/screw.stl"/>
 			</geometry>
 			<material name="Black"/>
@@ -771,5 +771,5 @@
 			<origin xyz="0 0 0" rpy="0 0 0"/>
 			<geometry name="pioneer_geom">
-				<mesh filename="package://bandit_urdf/meshes/bandit_mesh/screw_small.stl"/>
+				<mesh filename="package://bandit_urdf/meshes/bandit_mesh/screw.stl"/>
 			</geometry>
 			<material name="Black"/>
@@ -797,5 +797,5 @@
 			<origin xyz="0 0 0" rpy="0 0 0"/>
 			<geometry name="pioneer_geom">
-				<mesh filename="package://bandit_urdf/meshes/bandit_mesh/screw_small.stl"/>
+				<mesh filename="package://bandit_urdf/meshes/bandit_mesh/screw.stl"/>
 			</geometry>
 			<material name="Black"/>
@@ -823,5 +823,5 @@
 			<origin xyz="0 0 0" rpy="0 0 0"/>
 			<geometry name="pioneer_geom">
-				<mesh filename="package://bandit_urdf/meshes/bandit_mesh/screw_small.stl"/>
+				<mesh filename="package://bandit_urdf/meshes/bandit_mesh/screw.stl"/>
 			</geometry>
 			<material name="Black"/>
@@ -852,5 +852,5 @@
 			<origin xyz="0 0 0" rpy="0 0 0"/>
 			<geometry name="pioneer_geom">
-				<mesh filename="package://bandit_urdf/meshes/bandit_mesh/screw_small.stl"/>
+				<mesh filename="package://bandit_urdf/meshes/bandit_mesh/screw.stl"/>
 			</geometry>
 			<material name="Black"/>
@@ -878,5 +878,5 @@
 			<origin xyz="0 0 0" rpy="0 0 0"/>
 			<geometry name="pioneer_geom">
-				<mesh filename="package://bandit_urdf/meshes/bandit_mesh/screw_small.stl"/>
+				<mesh filename="package://bandit_urdf/meshes/bandit_mesh/screw.stl"/>
 			</geometry>
 			<material name="Black"/>
@@ -904,5 +904,5 @@
 			<origin xyz="0 0 0" rpy="0 0 0"/>
 			<geometry name="pioneer_geom">
-				<mesh filename="package://bandit_urdf/meshes/bandit_mesh/screw_small.stl"/>
+				<mesh filename="package://bandit_urdf/meshes/bandit_mesh/screw.stl"/>
 			</geometry>
 			<material name="Black"/>
@@ -930,5 +930,5 @@
 			<origin xyz="0 0 0" rpy="0 0 0"/>
 			<geometry name="pioneer_geom">
-				<mesh filename="package://bandit_urdf/meshes/bandit_mesh/screw_small.stl"/>
+				<mesh filename="package://bandit_urdf/meshes/bandit_mesh/screw.stl"/>
 			</geometry>
 			<material name="Black"/>
