Commit message: bandit_urdf: returned lips to original

File: bandit_urdf/defs/head.xacro (robot description, xacro)
@@ -155,6 +155,6 @@
     </link>
 	</xacro:macro>
-	<xacro:macro name="bandit_mouth" params="name parent side reflect *origin">
-	  <joint name="${name}_${side}_joint" type="revolute">
+	<xacro:macro name="bandit_lips" params="name parent *origin">
+	  <joint name="${name}_joint" type="revolute">
 		<axis xyz="0 -1 0" />
 		<limit lower="-0.261799388" upper="0.261799388" effort="2.645" velocity="6" />
@@ -164,7 +164,7 @@
       		<insert_block name="origin" />
       		<parent link="${parent}"/>
-      		<child link="${name}_${side}_link"/>
+      		<child link="${name}_link"/>
    	  </joint>
-    <link name="${name}_${side}_link">
+    <link name="${name}_link">
       <inertial>
         <mass value="0" />
@@ -173,11 +173,11 @@
                  iyy="0.005218991412"  iyz="-0.000314239509"  izz="0.008618784925"/>
       </inertial>
-      <visual name="${name}_${side}_visual">
-        <origin xyz="0 0 ${reflect*.002}" rpy="0 0 ${RCon*-90}"/>
+      <visual name="${name}_visual">
+        <origin xyz="0 0 .002" rpy="0 0 ${RCon*-90}"/>
         <!--<origin xyz="0 0 -0.035" rpy="${RCon*0} 0 ${RCon*-90}"/>-->
         <!--<origin xyz="0 0 0" rpy="${RCon*90} 0 ${RCon*90}"/>-->
 	<!-- -->
         <geometry name="${name}_visual_geom">
-					<mesh filename="package://bandit_urdf/meshes/bandit_mesh/${side}_lip_small.STL"/>
+					<mesh filename="package://bandit_urdf/meshes/bandit_mesh/top_lip_small.STL"/>
         </geometry>
 					<material name="Lips"/>
@@ -190,5 +190,5 @@
       </collision>
     </link>
-<!--	  <joint name="${name}2_joint" type="revolute">
+	  <joint name="${name}2_joint" type="revolute">
 		<axis xyz="0 -1 0"/>
 		<limit lower="-0.261799388" upper="0.261799388" effort="2.645" velocity="6" />
@@ -209,6 +209,9 @@
       <visual name="${name}2_visual">
         <origin xyz="0 0 -0.002" rpy="0 0 ${RCon*-90}"/>
+        <!--<origin xyz="0 0 -0.035" rpy="${RCon*0} 0 ${RCon*-90}"/>-->
+        <!--<origin xyz="0 0 0" rpy="${RCon*90} 0 ${RCon*90}"/>-->
+	<!-- -->
         <geometry name="${name}2_visual_geom">
-					<mesh filename="package://bandit_urdf/meshes/bandit_mesh/bottom_lip_small.stl"/>
+					<mesh filename="package://bandit_urdf/meshes/bandit_mesh/bottom_lip_small.STL"/>
         </geometry>
 					<material name="Lips"/>
@@ -220,5 +223,5 @@
         </geometry>
       </collision>
-    </link> -->
+    </link>
 </xacro:macro>
 	<xacro:macro name="bandit_head" params="name parent *origin">
@@ -241,10 +244,7 @@
 			<origin xyz="0.06 -0.0470 .085" rpy="${-M_PI/2} ${-M_PI/2} 0"/>
 		</xacro:bandit_eyebrow>
-		<xacro:bandit_mouth name="${name}_mouth" parent="${name}_tilt_link" reflect="1" side="top">
-			<origin xyz="0.070 0.0 0.0075" rpy="0 0 0"/>
-		</xacro:bandit_mouth>
-		<xacro:bandit_mouth name="${name}_mouth" parent="${name}_tilt_link" reflect="-1" side="bottom">
+		<xacro:bandit_lips name="${name}_lips" parent="${name}_tilt_link">
 			<origin xyz="0.070 0.0 -0.0075" rpy="0 0 0"/>
-		</xacro:bandit_mouth>
+		</xacro:bandit_lips>
 		<!--<xacro:bandit_head_gazebo name="${name}"/>-->
 	</xacro:macro>

Commit message: bandit_urdf: updated head.xacro for mouth

File: bandit_urdf/defs/head.xacro (robot description, xacro)
@@ -156,5 +156,5 @@
 	</xacro:macro>
 	<xacro:macro name="bandit_lips" params="name parent *origin">
-	  <joint name="${name}_joint" type="revolute">
+	  <joint name="mouth_top_joint" type="revolute">
 		<axis xyz="0 -1 0" />
 		<limit lower="-0.261799388" upper="0.261799388" effort="2.645" velocity="6" />
@@ -164,7 +164,7 @@
       		<insert_block name="origin" />
       		<parent link="${parent}"/>
-      		<child link="${name}_link"/>
+      		<child link="mouth_top_link"/>
    	  </joint>
-    <link name="${name}_link">
+    <link name="mouth_top_link">
       <inertial>
         <mass value="0" />
@@ -173,22 +173,19 @@
                  iyy="0.005218991412"  iyz="-0.000314239509"  izz="0.008618784925"/>
       </inertial>
-      <visual name="${name}_visual">
+      <visual name="mouth_top_visual">
         <origin xyz="0 0 .002" rpy="0 0 ${RCon*-90}"/>
-        <!--<origin xyz="0 0 -0.035" rpy="${RCon*0} 0 ${RCon*-90}"/>-->
-        <!--<origin xyz="0 0 0" rpy="${RCon*90} 0 ${RCon*90}"/>-->
-	<!-- -->
-        <geometry name="${name}_visual_geom">
+        <geometry name="mouth_top_visual_geom">
 					<mesh filename="package://bandit_urdf/meshes/bandit_mesh/top_lip_small.STL"/>
         </geometry>
 					<material name="Lips"/>
       </visual>
-      <collision name="${name}_collision">
-         <origin xyz="0 0 0" rpy="0 0 0 " />
-        <geometry name="${name}_visual_geom">
-					<box size="0 0 0"/>
-        </geometry>
-      </collision>
-    </link>
-	  <joint name="${name}2_joint" type="revolute">
+      <collision name="mouth_top_collision">
+         <origin xyz="0 0 0" rpy="0 0 0 " />
+        <geometry name="mouth_top_visual_geom">
+					<box size="0 0 0"/>
+        </geometry>
+      </collision>
+    </link>
+	  <joint name="mouth_bottom_joint" type="revolute">
 		<axis xyz="0 -1 0"/>
 		<limit lower="-0.261799388" upper="0.261799388" effort="2.645" velocity="6" />
@@ -198,26 +195,23 @@
       		<insert_block name="origin" />
       		<parent link="${parent}"/>
-      		<child link="${name}2_link"/>
+      		<child link="mouth_bottom_link"/>
    	  </joint>
-    <link name="${name}2_link">
-      <inertial>
-        <mass value="0" />
-        <origin xyz="0 0 0" rpy="${RCon*90} 0 ${RCon*90}"/>
-        <inertia ixx="0.00482611007"  ixy="-0.000144683999"  ixz="0.000110076136"
-                 iyy="0.005218991412"  iyz="-0.000314239509"  izz="0.008618784925"/>
-      </inertial>
-      <visual name="${name}2_visual">
+    <link name="mouth_bottom_link">
+      <inertial>
+        <mass value="0" />
+        <origin xyz="0 0 0" rpy="${RCon*90} 0 ${RCon*90}"/>
+        <inertia ixx="0.00482611007"  ixy="-0.000144683999"  ixz="0.000110076136"
+                 iyy="0.005218991412"  iyz="-0.000314239509"  izz="0.008618784925"/>
+      </inertial>
+      <visual name="mouth_bottom_visual">
         <origin xyz="0 0 -0.002" rpy="0 0 ${RCon*-90}"/>
-        <!--<origin xyz="0 0 -0.035" rpy="${RCon*0} 0 ${RCon*-90}"/>-->
-        <!--<origin xyz="0 0 0" rpy="${RCon*90} 0 ${RCon*90}"/>-->
-	<!-- -->
-        <geometry name="${name}2_visual_geom">
+        <geometry name="mouth_bottom_visual_geom">
 					<mesh filename="package://bandit_urdf/meshes/bandit_mesh/bottom_lip_small.STL"/>
         </geometry>
 					<material name="Lips"/>
       </visual>
-      <collision name="${name}2_collision">
-         <origin xyz="0 0 0" rpy="0 0 0 " />
-        <geometry name="${name}2_visual_geom">
+      <collision name="mouth_bottom_collision">
+         <origin xyz="0 0 0" rpy="0 0 0 " />
+        <geometry name="mouth_bottom_visual_geom">
 					<box size="0 0 0"/>
         </geometry>
@@ -281,3 +275,63 @@
 <xacro:pupil suffix="left" reflect="-4.8"/>
 <xacro:pupil suffix="right" reflect="-4.6"/>
+<!--	  <joint name="bandit_top_lip_joint" type="revolute">
+		<axis xyz="0 -1 0" />
+		<limit lower="-0.261799388" upper="0.261799388" effort="2.645" velocity="6" />
+      		<safety_controller k_velocity="1.5" soft_lower_limit="${-1.57079633+0.15}" soft_upper_limit="${1.57079633-0.15}" k_position="100" />
+     		<calibration reference_position="0.0" />
+      		<dynamics damping="1.0" />
+      		<parent link="bandit_head_tilt_link"/>
+      		<child link="bandit_top_lip_link"/>
+   	  </joint>
+    <link name="bandit_top_lip_link">
+      <inertial>
+        <mass value="0" />
+        <origin xyz="0 0 0" rpy="0 0 ${RCon*90}"/>
+        <inertia ixx="0.00482611007"  ixy="-0.000144683999"  ixz="0.000110076136"
+                 iyy="0.005218991412"  iyz="-0.000314239509"  izz="0.008618784925"/>
+      </inertial>
+      <visual name="bandit_top_lip_visual">
+        <origin xyz="0 0 .002" rpy="0 0 ${RCon*-90}"/>
+        <geometry name="bandit_top_lip_visual_geom">
+					<mesh filename="package://bandit_urdf/meshes/bandit_mesh/top_lip_small.STL"/>
+        </geometry>
+					<material name="Lips"/>
+      </visual>
+      <collision name="bandit_top_lip_collision">
+         <origin xyz="0 0 0" rpy="0 0 0 " />
+        <geometry name="bandit_top_lip_visual_geom">
+					<box size="0 0 0"/>
+        </geometry>
+      </collision>
+    </link>
+	  <joint name="bandit_bottom_lip_joint" type="revolute">
+		<axis xyz="0 -1 0" />
+		<limit lower="-0.261799388" upper="0.261799388" effort="2.645" velocity="6" />
+      		<safety_controller k_velocity="1.5" soft_lower_limit="${-1.57079633+0.15}" soft_upper_limit="${1.57079633-0.15}" k_position="100" />
+     		<calibration reference_position="0.0" />
+      		<dynamics damping="1.0" />
+      		<parent link="bandit_head_tilt_link"/>
+      		<child link="bandit_bottom_lip_link"/>
+   	  </joint>
+    <link name="bandit_bottom_lip_link">
+      <inertial>
+        <mass value="0" />
+        <origin xyz="0 0 0" rpy="0 0 ${RCon*90}"/>
+        <inertia ixx="0.00482611007"  ixy="-0.000144683999"  ixz="0.000110076136"
+                 iyy="0.005218991412"  iyz="-0.000314239509"  izz="0.008618784925"/>
+      </inertial>
+      <visual name="bandit_bottom_lip_visual">
+        <origin xyz="0 0 .002" rpy="0 0 ${RCon*-90}"/>
+        <geometry name="bandit_bottom_lip_visual_geom">
+					<mesh filename="package://bandit_urdf/meshes/bandit_mesh/bottom_lip_small.STL"/>
+        </geometry>
+					<material name="Lips"/>
+      </visual>
+      <collision name="bandit_bottom_lip_collision">
+         <origin xyz="0 0 0" rpy="0 0 0 " />
+        <geometry name="bandit_bottom_lip_visual_geom">
+					<box size="0 0 0"/>
+        </geometry>
+      </collision>
+    </link> -->
 </robot>

Commit message: 

File: bandit_urdf/defs/head.xacro (robot description, xacro)
@@ -109,5 +109,4 @@
 					<mesh filename="package://bandit_urdf/meshes/bandit_mesh/camera_board.stl"/>
         </geometry>
-					<!--  <material name="Silver"/>  -->
 					<material name="texture">
 					<texture filename="package://bandit_urdf/meshes/bandit_mesh/gradients/reflect1.jpg"/>

Commit message: 

File: bandit_urdf/defs/head.xacro (robot description, xacro)
@@ -76,5 +76,5 @@
 	<!-- -->
         <geometry name="${name}_visual_geom">
-		<mesh filename="package://bandit_urdf/meshes/bandit_mesh/head_small.stl"/>
+		<mesh filename="package://bandit_urdf/meshes/bandit_mesh/head_smaller.stl"/>
         </geometry>
 					<material name="Head"/>

Commit message: bandit_urdf: fixed disappearing head stl

File: bandit_urdf/defs/head.xacro (robot description, xacro)
@@ -76,5 +76,5 @@
 	<!-- -->
         <geometry name="${name}_visual_geom">
-		<mesh filename="package://bandit_urdf/meshes/bandit_mesh/head_smaller.stl"/>
+		<mesh filename="package://bandit_urdf/meshes/bandit_mesh/head_small.stl"/>
         </geometry>
 					<material name="Head"/>

Commit message: bandit_urdf: fixed eye orientation to work with image_proc properly

File: bandit_urdf/defs/head.xacro (robot description, xacro)
@@ -226,8 +226,8 @@
 		</xacro:bandit_head_tilt>
 		<xacro:bandit_eye name="${name}_right_camera" parent="${name}_tilt_link">
-			<origin xyz="0.05 -0.0320 .060" rpy="0 ${M_PI/2} 0"/>
+			<origin xyz="0.05 -0.0320 .060" rpy="-${M_PI/2} 0 -${M_PI/2}"/>
 		</xacro:bandit_eye>
 		<xacro:bandit_eye name="${name}_left_camera" parent="${name}_tilt_link">
-			<origin xyz="0.05 0.0320 .060" rpy="0 ${M_PI/2} 0"/>
+      <origin xyz="0.05 0.0320 .060" rpy="-${M_PI/2} 0 -${M_PI/2}"/>
 		</xacro:bandit_eye>
 		<xacro:bandit_eyebrow name="${name}_left_brow" parent="${name}_tilt_link" side="left" reflect="1">

Commit message: fixed the right camera rotation

File: bandit_urdf/defs/head.xacro (robot description, xacro)
@@ -226,5 +226,5 @@
 		</xacro:bandit_head_tilt>
 		<xacro:bandit_eye name="${name}_right_camera" parent="${name}_tilt_link">
-			<origin xyz="0.05 -0.0320 .060" rpy="-${M_PI/2} 0 -${M_PI/2}"/>
+			<origin xyz="0.05 -0.0320 .060" rpy="-${M_PI/2} -0.3 -${M_PI/2}"/>
 		</xacro:bandit_eye>
 		<xacro:bandit_eye name="${name}_left_camera" parent="${name}_tilt_link">
