Commit message: bandit_urdf: changed bandit_lips & bandit_lips2 to bandit_mouth

File: bandit_urdf/defs/gazebo/bandit_shirt_defs.xacro (robot description, xacro)
@@ -9,10 +9,10 @@
 	<include filename="$(find bandit_urdf)/defs/shirt_materials.xacro"/>
 	<include filename="$(find bandit_urdf)/defs/gazebo/torso.xacro"/>
-	<include filename="$(find bandit_urdf)/defs/gazebo/logo.xacro"/>
+<!--	<include filename="$(find bandit_urdf)/defs/logo.xacro"/> -->
 	<include filename="$(find bandit_urdf)/defs/gazebo/head.xacro"/>
 	<include filename="$(find bandit_urdf)/defs/gazebo/shoulder.xacro"/>
-	<include filename="$(find bandit_urdf)/defs/gazebo/pioneerbase.xacro"/>
-	<include filename="$(find bandit_urdf)/defs/gazebo/screws.xacro"/>
-<!--	<include filename="$(find bandit_urdf)/defs/stage.xacro"/> -->
+<!--	<include filename="$(find bandit_urdf)/defs/pioneerbase.xacro"/>
+	<include filename="$(find bandit_urdf)/defs/screws.xacro"/>
+	<include filename="$(find bandit_urdf)/defs/stage.xacro"/> -->
 	<include filename="$(find bandit_urdf)/defs/gazebo.urdf.xacro"/>
 	<!--<xacro:pr2_base_v0 name="base"/>-->

File: bandit_urdf/defs/gazebo/head.xacro (robot description, xacro)
@@ -38,5 +38,5 @@
         <origin xyz="0 0 0" rpy="${RCon*90} 0 ${RCon*-90}"/>
         <geometry name="${name}_visual_geom">
-					<mesh filename="package://bandit_urdf/meshes/bandit_mesh/neck_small.stl"/>
+					<mesh filename="package://bandit_urdf/meshes/bandit_mesh/neck_smallest.stl"/>
         </geometry>
 					<material name="Neck"/>
@@ -76,5 +76,5 @@
 	<!-- -->
         <geometry name="${name}_visual_geom">
-		<mesh filename="package://bandit_urdf/meshes/bandit_mesh/head_small.stl"/>
+		<mesh filename="package://bandit_urdf/meshes/bandit_mesh/head_smallest.stl"/>
         </geometry>
 					<material name="Head"/>
@@ -107,5 +107,5 @@
         <origin xyz="0.035 0 0" rpy="${RCon*90} 0 ${RCon*-90}"/>
         <geometry name="${name}_visual_geom">
-					<mesh filename="package://bandit_urdf/meshes/bandit_mesh/camera_board.stl"/>
+					<mesh filename="package://bandit_urdf/meshes/bandit_mesh/camera_board_smallest.stl"/>
         </geometry>
 					<!--  <material name="Silver"/>  -->
@@ -143,5 +143,5 @@
         <origin xyz="0 0 0" rpy="0 0 ${RCon*-90}"/>
         <geometry name="${name}_visual_geom">
-					<mesh filename="package://bandit_urdf/meshes/bandit_mesh/eyebrow_${side}_small.stl"/>
+					<mesh filename="package://bandit_urdf/meshes/bandit_mesh/eyebrow_${side}_smallest.stl"/>
         </geometry>
 					<material name="Eyebrows"/>
@@ -179,5 +179,5 @@
 	<!-- -->
         <geometry name="${name}_visual_geom">
-					<mesh filename="package://bandit_urdf/meshes/bandit_mesh/top_lip_small.STL"/>
+					<mesh filename="package://bandit_urdf/meshes/bandit_mesh/top_lip_smallest.STL"/>
         </geometry>
 					<material name="Lips"/>
@@ -213,5 +213,5 @@
 	<!-- -->
         <geometry name="${name}2_visual_geom">
-					<mesh filename="package://bandit_urdf/meshes/bandit_mesh/bottom_lip_small.stl"/>
+					<mesh filename="package://bandit_urdf/meshes/bandit_mesh/bottom_lip_smallest.stl"/>
         </geometry>
 					<material name="Lips"/>
@@ -265,5 +265,5 @@
 			<origin xyz="0 0 0" rpy="0 0 0"/>
 			<geometry name="pupil_left_geom">
-				<mesh filename="package://bandit_urdf/meshes/bandit_mesh/middle_eye.stl"/>
+				<mesh filename="package://bandit_urdf/meshes/bandit_mesh/middle_eye_smallest.stl"/>
 			</geometry>
 		<material name="Pupil">

File: bandit_urdf/defs/gazebo/shoulder.xacro (robot description, xacro)
@@ -39,5 +39,5 @@
 				<origin xyz="0 0 0" rpy="${RCon*90} 0 ${RCon*90}"/>
 				<geometry name="${side}_shoulder_mounting_link_geom">
-					<mesh filename="package://bandit_urdf/meshes/bandit_mesh/shoulder_cover_${side}_small.stl"/>
+					<mesh filename="package://bandit_urdf/meshes/bandit_mesh/shoulder_cover_${side}_smallest.stl"/>
 					<!--<box size="0.080 0.085 ${shoulder_mounting_link_z}"/>-->
 				</geometry>
@@ -76,5 +76,5 @@
 				<origin xyz="0 ${-reflect*0.0} 0" rpy="0 ${M_PI/2} 0"/>
 				<geometry name="${side}_shoulder_link_geom">
-					<mesh filename="package://bandit_urdf/meshes/bandit_mesh/bicep_cover_${side}_small.stl"/>
+					<mesh filename="package://bandit_urdf/meshes/bandit_mesh/bicep_cover_${side}_smallest.stl"/>
 				</geometry>
 				<material name="Arms"/>
@@ -112,5 +112,5 @@
 				<origin xyz="0 0 0.0" rpy="0 ${-M_PI/2} ${M_PI/2}"/>
 				<geometry name="${side}_bicep_link_geom">
-					<mesh filename="package://bandit_urdf/meshes/bandit_mesh/elbow_cover_${side}_small.stl"/>
+					<mesh filename="package://bandit_urdf/meshes/bandit_mesh/elbow_cover_${side}_smallest.stl"/>
 					<!--<box size="0.050 0.050 0.065"/>-->
 				</geometry>
@@ -149,5 +149,5 @@
 				<!--<origin xyz="0 0 -0.025" rpy="0 ${M_PI/2} ${M_PI/2}"/>-->
 				<geometry name="${side}_forearm_link_geom">
-					<mesh filename="package://bandit_urdf/meshes/bandit_mesh/forearm_cover_${side}_small.stl"/>
+					<mesh filename="package://bandit_urdf/meshes/bandit_mesh/forearm_cover_${side}_smallest.stl"/>
 					<!--<box size="0.068 0.065 0.095"/>-->
 				</geometry>
@@ -187,5 +187,5 @@
 				<origin xyz="0 0 -0.01" rpy="${M_PI/2} 0 ${M_PI/2}"/>
 				<geometry name="${side}_wrist_link_geom">
-					<mesh filename="package://bandit_urdf/meshes/bandit_mesh/wrist_cover_${side}_small.stl"/>
+					<mesh filename="package://bandit_urdf/meshes/bandit_mesh/wrist_cover_${side}_smallest.stl"/>
 					<!--<box size="0.054 0.054 0.055"/>-->
 				</geometry>
@@ -224,5 +224,5 @@
 				<origin xyz="0 0 -.00" rpy="${M_PI/2} 0 0"/>
 				<geometry name="${side}_hand_link_geom">
-					<mesh filename="package://bandit_urdf/meshes/bandit_mesh/${side}_hand_small.stl"/>
+					<mesh filename="package://bandit_urdf/meshes/bandit_mesh/${side}_hand_smallest.stl"/>
 					<!--<box size="0.060 0.060 0.080"/>-->
 				</geometry>
@@ -260,5 +260,5 @@
 				<origin xyz="0 0 0" rpy="${M_PI/2} ${-M_PI/2} 0"/>
 				<geometry name="${side}_thumb_link_geom">
-					<mesh filename="package://bandit_urdf/meshes/bandit_mesh/${side}_thumb_small.stl"/>
+					<mesh filename="package://bandit_urdf/meshes/bandit_mesh/${side}_thumb_smallest.stl"/>
 					<!--<box size="0.030 0.025 0.06"/>-->
 				</geometry>

File: bandit_urdf/defs/gazebo/torso.xacro (robot description, xacro)
@@ -17,5 +17,5 @@
 	  <link name = "${name}_link">
 	    <inertial>
- 	    <mass value="0"/>
+ 	    <mass value="50"/>
     	  <origin xyz="0 0 0"/>
       	<inertia ixx="1" ixy="0" ixz="0"
@@ -28,5 +28,5 @@
     	  <!--<origin xyz="0 0 0.05" rpy="${M_PI/2} 0 ${M_PI/2}"/>-->
       	<geometry name="${name}_geom">
-					<mesh filename="package://bandit_urdf/meshes/bandit_mesh/body_small.stl"/>
+					<mesh filename="package://bandit_urdf/meshes/bandit_mesh/body_smallest.stl"/>
   	    <!--  <box size="0 0 0"/>-->
 	      </geometry>
@@ -41,5 +41,5 @@
 		<xacro:bandit_torso_gazebo name="${name}"/>
 	</xacro:macro>
-<!-- dasf -->
+<!--
 	<link name="bandit_stop_link">
 		<inertial>
@@ -67,5 +67,4 @@
 		<parent link="bandit_torso_link"/>
 		<child link="bandit_stop_link"/>
-	</joint>
-<!-- dasf -->
+	</joint> -->
 </robot>

File: bandit_urdf/defs/head.xacro (robot description, xacro)
@@ -155,6 +155,6 @@
     </link>
 	</xacro:macro>
-	<xacro:macro name="bandit_lips" params="name parent *origin">
-	  <joint name="${name}_joint" type="revolute">
+	<xacro:macro name="bandit_mouth" params="name parent side reflect *origin">
+	  <joint name="${name}_${side}_joint" type="revolute">
 		<axis xyz="0 -1 0" />
 		<limit lower="-0.261799388" upper="0.261799388" effort="2.645" velocity="6" />
@@ -164,7 +164,7 @@
       		<insert_block name="origin" />
       		<parent link="${parent}"/>
-      		<child link="${name}_link"/>
+      		<child link="${name}_${side}_link"/>
    	  </joint>
-    <link name="${name}_link">
+    <link name="${name}_${side}_link">
       <inertial>
         <mass value="0" />
@@ -173,11 +173,11 @@
                  iyy="0.005218991412"  iyz="-0.000314239509"  izz="0.008618784925"/>
       </inertial>
-      <visual name="${name}_visual">
-        <origin xyz="0 0 .002" rpy="0 0 ${RCon*-90}"/>
+      <visual name="${name}_${side}_visual">
+        <origin xyz="0 0 ${reflect*.002}" rpy="0 0 ${RCon*-90}"/>
         <!--<origin xyz="0 0 -0.035" rpy="${RCon*0} 0 ${RCon*-90}"/>-->
         <!--<origin xyz="0 0 0" rpy="${RCon*90} 0 ${RCon*90}"/>-->
 	<!-- -->
         <geometry name="${name}_visual_geom">
-					<mesh filename="package://bandit_urdf/meshes/bandit_mesh/top_lip_small.STL"/>
+					<mesh filename="package://bandit_urdf/meshes/bandit_mesh/${side}_lip_small.STL"/>
         </geometry>
 					<material name="Lips"/>
@@ -190,5 +190,5 @@
       </collision>
     </link>
-	  <joint name="${name}2_joint" type="revolute">
+<!--	  <joint name="${name}2_joint" type="revolute">
 		<axis xyz="0 -1 0"/>
 		<limit lower="-0.261799388" upper="0.261799388" effort="2.645" velocity="6" />
@@ -209,7 +209,4 @@
       <visual name="${name}2_visual">
         <origin xyz="0 0 -0.002" rpy="0 0 ${RCon*-90}"/>
-        <!--<origin xyz="0 0 -0.035" rpy="${RCon*0} 0 ${RCon*-90}"/>-->
-        <!--<origin xyz="0 0 0" rpy="${RCon*90} 0 ${RCon*90}"/>-->
-	<!-- -->
         <geometry name="${name}2_visual_geom">
 					<mesh filename="package://bandit_urdf/meshes/bandit_mesh/bottom_lip_small.stl"/>
@@ -223,5 +220,5 @@
         </geometry>
       </collision>
-    </link>
+    </link> -->
 </xacro:macro>
 	<xacro:macro name="bandit_head" params="name parent *origin">
@@ -244,7 +241,10 @@
 			<origin xyz="0.06 -0.0470 .085" rpy="${-M_PI/2} ${-M_PI/2} 0"/>
 		</xacro:bandit_eyebrow>
-		<xacro:bandit_lips name="${name}_lips" parent="${name}_tilt_link">
+		<xacro:bandit_mouth name="${name}_mouth" parent="${name}_tilt_link" reflect="1" side="top">
+			<origin xyz="0.070 0.0 0.0075" rpy="0 0 0"/>
+		</xacro:bandit_mouth>
+		<xacro:bandit_mouth name="${name}_mouth" parent="${name}_tilt_link" reflect="-1" side="bottom">
 			<origin xyz="0.070 0.0 -0.0075" rpy="0 0 0"/>
-		</xacro:bandit_lips>
+		</xacro:bandit_mouth>
 		<!--<xacro:bandit_head_gazebo name="${name}"/>-->
 	</xacro:macro>
