Commit message: commit error fix for fake_bandit and bandit_urdf

File: bandit/bandit_urdf/defs/bandit_defs.xacro (robot description, xacro)
@@ -22,4 +22,7 @@
 		<origin xyz="0 0 ${body_height/2 + neck_height/2+0.01}" rpy="0 0 0"/>
 	</xacro:bandit_head-->
+		<!--xacro:bandit_head name="bandit_head" parent="bandit_torso_link">
+		<origin xyz="0 0 ${body_height/2 + neck_height/2+0.01}" rpy="0 0 0"/>
+	</xacro:bandit_head-->
 	<xacro:bandit_shoulder side="left" parent="bandit_torso_link" reflect="1">
 		<origin xyz="0 ${body_width/2+.01} 0" rpy="0 0 0"/>

File: bandit/bandit_urdf/defs/head.xacro (robot description, xacro)
@@ -4,15 +4,14 @@
        xmlns:interface="http://playerstage.sourceforge.net/gazebo/xmlschema/#interface"
        xmlns:xacro="http://ros.org/wiki/xacro">
-	<!-- path to mesh files -->
-	<property name="mesh_path" value="package://bandit_urdf/meshes/bandit_mesh/"/>
+	<!-- use the below line to specify path to meshes and materials -->
+	<property name="mesh_path" value="package://bandit_urdf/meshes/bandit_mesh"/>
 	<!-- other properties -->
-	<!-- head xacro definition -->
+	<!-- start head xacro definition -->
     <xacro:macro name="head" params="name parent *origin">
     	<!-- head_pan_joint -->
-    	<!---->
     	<joint name="head_pan_joint" type="revolute">
     		<axis xyz="0 0 1"/>
-    		<insert_block name="origin" />
-    		<parent link="torso_link"/>
+    		<origin xyz="0 0 ${.0825 + (neck_height/2)-0.01}"/>
+    		<parent link="${parent}"/>
       		<child link="head_pan_link"/>
       		<limit lower="-1.57079633" upper="1.57079633" effort="2.645" velocity="6" />
@@ -22,9 +21,5 @@
       		<dynamics damping="1.0" />
     	</joint>
-       	<!---->
-       	<!-- NOTE - this was for head_pan_joint -->
-       	<!--origin xyz="0 0 ${.0825 + (neck_height/2)-0.01}"/-->
   		<!-- head_pan_link -->
-  		<!---->
     	<link name="head_pan_link">
       		<inertial>
@@ -38,5 +33,5 @@
         		<origin xyz="0 0 0" rpy="${RCon*90} 0 ${RCon*-90}"/>
         		<geometry name="head_pan_visual_geom">
-                    <mesh filename="${mesh_path}/neck_small.stl"/>
+                    <mesh filename="${mesh_path}/neck_smallest.stl"/>
         		</geometry>
         		<material name="Neck"/>
@@ -49,7 +44,5 @@
       		</collision>
     	</link>
-  		<!---->
     	<!-- head_tilt_joint -->
-    	<!--
     	<joint name="head_tilt_joint" type="revolute">
       		<axis xyz="0 -1 ${(head_height/4)}" />
@@ -63,7 +56,5 @@
       		<child link="head_tilt_link"/>
     	</joint>
-    	-->
     	<!-- head_tilt_link -->
-    	<!--
     	<link name="head_tilt_link">
       		<inertial>
@@ -76,5 +67,5 @@
         		<origin xyz="-.02 0 .01" rpy="${RCon*90} 0 ${RCon*90}"/>
         		<geometry name="head_tilt_visual_geom">
-        			<mesh filename="${mesh_path}/head_smaller.stl"/>
+        			<mesh filename="${mesh_path}/head_smallest.stl"/>
         		</geometry>
         		<material name="Head"/>
@@ -87,7 +78,5 @@
       		</collision>
     	</link>
-        -->
     	<!-- mouth_top_joint -->
-    	<!--
       	<joint name="mouth_top_joint" type="revolute">
         	<axis xyz="0 -1 0" />
@@ -101,7 +90,5 @@
             <child link="mouth_top_link"/>
       	</joint>
-      	-->
       	<!-- mouth_top_link -->
-      	<!--
     	<link name="mouth_top_link">
       		<inertial>
@@ -126,22 +113,111 @@
       		</collision>
     	</link>
-    	-->
-    	<!-- mouth_bottom_joint -->
-    	<!--
-      	<joint name="mouth_bottom_joint" type="revolute">
-        	<axis xyz="0 -1 0"/>
-        	<limit lower="-0.261799388" upper="0.261799388" effort="2.645" velocity="6" />
-            <safety_controller k_velocity="1.5" soft_lower_limit="${-1.57079633+0.15}"
-            		soft_upper_limit="${1.57079633-0.15}" k_position="100" />
-            <calibration reference_position="0.0" />
-            <dynamics damping="1.0" />
-            <insert_block name="origin" />
-            <parent link="head_tilt_link"/>
-            <child link="mouth_bottom_link"/>
-      	</joint>
-      	-->
-      	<!-- mouth_bottom_link -->
-      	<!--
-    	<link name="mouth_bottom_link">
+		<!-- start mouth xacro definition -->
+		<!-- mouth_bottom_joint -->
+	  	<joint name="mouth_bottom_joint" type="revolute">
+	    	<axis xyz="0 -1 0"/>
+	    	<limit lower="-0.261799388" upper="0.261799388" effort="2.645" velocity="6" />
+	        <safety_controller k_velocity="1.5" soft_lower_limit="${-1.57079633+0.15}"
+	        		soft_upper_limit="${1.57079633-0.15}" k_position="100" />
+	        <calibration reference_position="0.0" />
+	        <dynamics damping="1.0" />
+	        <insert_block name="origin" />
+	        <parent link="head_tilt_link"/>
+	        <child link="mouth_bottom_link"/>
+	  	</joint>
+	  	<!-- mouth_bottom_link -->
+		<link name="mouth_bottom_link">
+	  		<inertial>
+	    		<mass value="0" />
+	    		<origin xyz="0 0 0" rpy="${RCon*90} 0 ${RCon*90}"/>
+	    		<inertia ixx="0.00482611007"  ixy="-0.000144683999"
+	    				ixz="0.000110076136" iyy="0.005218991412"
+	    				iyz="-0.000314239509"  izz="0.008618784925"/>
+	  			</inertial>
+	  		<visual name="mouth_bottom_visual">
+	    		<origin xyz="0 0 -0.002" rpy="0 0 ${RCon*-90}"/>
+	    		<geometry name="mouth_bottom_visual_geom">
+	                <mesh filename="${mesh_path}/bottom_lip_small.STL"/>
+	    		</geometry>
+	        	<material name="Lips"/>
+	  		</visual>
+	  		<collision name="mouth_bottom_collision">
+	     		<origin xyz="0 0 0" rpy="0 0 0 " />
+	    		<geometry name="mouth_bottom_visual_geom">
+	                <box size="0 0 0"/>
+	    		</geometry>
+	  		</collision>
+		</link>
+		<!-- eye xacro instances -->
+        <xacro:eye name="eye_right_camera" parent="${name}_tilt_link">
+            <origin xyz="0.05 -0.0320 .060" rpy="-${M_PI/2} -0.3 -${M_PI/2}"/>
+        </xacro:eye>
+        <xacro:eye name="eye_left_camera" parent="${name}_tilt_link">
+      		<origin xyz="0.05 0.0320 .060" rpy="-${M_PI/2} 0 -${M_PI/2}"/>
+        </xacro:eye>
+		<!-- eyebrow xacro instances -->
+		<xacro:eyebrow name="${name}_left_brow" parent="${name}_tilt_link"
+			side="left" reflect="1">
+            <origin xyz="0.06 0.0470 .085" rpy="${-M_PI/2} ${-M_PI/2} 0"/>
+        </xacro:eyebrow>
+        <xacro:eyebrow name="${name}_right_brow" parent="${name}_tilt_link"
+        	side="right" reflect="-1">
+            <origin xyz="0.06 -0.0470 .085" rpy="${-M_PI/2} ${-M_PI/2} 0"/>
+        </xacro:eyebrow>
+	</xacro:macro>
+	<!-- end head xacro definition -->
+		<!-- pupil xacro instances -->
+		<xacro:pupil suffix="left" reflect="-4.8"/>
+		<xacro:pupil suffix="right" reflect="-4.6"/>
+	<!-- start eye xacro definition -->
+	<xacro:macro name="eye" params="name parent *origin">
+		<!-- eye_{side}_camera_joint -->
+		<joint name="${name}_joint" type="fixed">
+			<insert_block name="origin" />
+			<parent link="${parent}"/>
+			<child link="${name}_link"/>
+		</joint>
+		<!-- eye_{side}_camera_link -->
+		<link name="${name}_link">
+  			<inertial>
+    			<mass value="0" />
+    			<origin xyz="0 0 0" rpy="${RCon*90} 0 ${RCon*90}"/>
+    			<inertia ixx="0.00482611007"  ixy="-0.000144683999"
+    						ixz="0.000110076136" iyy="0.005218991412"
+    						iyz="-0.000314239509"  izz="0.008618784925"/>
+ 			</inertial>
+  			<visual name="${name}_visual">
+    			<origin xyz="0.035 0 0" rpy="${RCon*90} 0 ${RCon*-90}"/>
+    			<geometry name="${name}_visual_geom">
+               		<mesh filename="${mesh_path}/camera_board.stl"/>
+    			</geometry>
+      	    	<material name="texture">
+            		<texture filename="${mesh_path}/gradients/reflect1.jpg"/>
+            	</material>
+  			</visual>
+  			<collision name="${name}_collision">
+     			<origin xyz="0 0 0" rpy="0 0 0 " />
+    			<geometry name="${name}_visual_geom">
+            	 	<box size="0 0 0"/>
+    			</geometry>
+  			</collision>
+		</link>
+	</xacro:macro>
+	<!-- end eye xacro definition -->
+	<!-- start eyebrow xacro definition -->
+	<xacro:macro name="eyebrow" params="name parent side reflect *origin">
+		<!-- head_{side}_brow_joint -->
+    	<joint name="head_${side}_brow_joint" type="revolute">
+      		<axis xyz="0 ${reflect} 0" />
+      		<limit lower="-0.261799388" upper="0.261799388" effort="2.645" velocity="6" />
+      		<safety_controller k_velocity="1.5" soft_lower_limit="${-1.57079633+0.15}" 						soft_upper_limit="${1.57079633-0.15}" k_position="100" />
+      		<calibration reference_position="0.0" />
+      		<dynamics damping="1.0" />
+      		<insert_block name="origin" />
+      		<parent link="${parent}"/>
+      		<child link="${name}_link"/>
+    	</joint>
+    	<!-- eyebrow_link -->
+    	<link name="${name}_link">
       		<inertial>
         		<mass value="0" />
@@ -150,129 +226,53 @@
         				ixz="0.000110076136" iyy="0.005218991412"
         				iyz="-0.000314239509"  izz="0.008618784925"/>
-      			</inertial>
-      		<visual name="mouth_bottom_visual">
-        		<origin xyz="0 0 -0.002" rpy="0 0 ${RCon*-90}"/>
-        		<geometry name="mouth_bottom_visual_geom">
-                    <mesh filename="${mesh_path}/bottom_lip_small.STL"/>
-        		</geometry>
-            	<material name="Lips"/>
-      		</visual>
-      		<collision name="mouth_bottom_collision">
-         		<origin xyz="0 0 0" rpy="0 0 0 " />
-        		<geometry name="mouth_bottom_visual_geom">
+      		</inertial>
+      		<visual name="${name}_visual">
+        		<origin xyz="0 0 0" rpy="0 0 ${RCon*-90}"/>
+        		<geometry name="${name}_visual_geom">
+                    <mesh filename="${mesh_path}/eyebrow_${side}_small.stl"/>
+        		</geometry>
+                <material name="Eyebrows"/>
+      		</visual>
+      		<collision name="${name}_collision">
+         		<origin xyz="0 0 0" rpy="0 0 0 "/>
+        		<geometry name="${name}_visual_geom">
                     <box size="0 0 0"/>
         		</geometry>
       		</collision>
     	</link>
-		-->
-        <!-- ~~~~~~~~~~~~~~~~~~~
-        <xacro:eye name="eye_right_camera" parent="head_tilt_link">
-            <origin xyz="0.05 -0.0320 .060" rpy="-${M_PI/2} -0.3 -${M_PI/2}"/>
-        </xacro:eye>
-        <xacro:eye name="eye_left_camera" parent="head_tilt_link">
-      <origin xyz="0.05 0.0320 .060" rpy="-${M_PI/2} 0 -${M_PI/2}"/>
-        </xacro:eye>
-        <xacro:eyebrow name="${name}_left_brow" parent="${name}_tilt_link" side="left" reflect="1">
-            <origin xyz="0.06 0.0470 .085" rpy="${-M_PI/2} ${-M_PI/2} 0"/>
-        </xacro:eyebrow>
-        <xacro:eyebrow name="${name}_right_brow" parent="${name}_tilt_link" side="right" reflect="-1">
-            <origin xyz="0.06 -0.0470 .085" rpy="${-M_PI/2} ${-M_PI/2} 0"/>
-        </xacro:eyebrow>
-    <xacro:macro name="eye" params="name parent *origin">
-      <joint name="${name}_joint" type="fixed">
-      <insert_block name="origin" />
-      <parent link="${parent}"/>
-      <child link="${name}_link"/>
-    </joint>
-    <link name="${name}_link">
-      <inertial>
-        <mass value="0" />
-        <origin xyz="0 0 0" rpy="${RCon*90} 0 ${RCon*90}"/>
-        <inertia ixx="0.00482611007"  ixy="-0.000144683999"  ixz="0.000110076136"
-                 iyy="0.005218991412"  iyz="-0.000314239509"  izz="0.008618784925"/>
-      </inertial>
-      <visual name="${name}_visual">
-        <origin xyz="0.035 0 0" rpy="${RCon*90} 0 ${RCon*-90}"/>
-        <geometry name="${name}_visual_geom">
-                    <mesh filename="package://bandit_urdf/meshes/bandit_mesh/camera_board.stl"/>
-        </geometry>
-                    <material name="texture">
-                    <texture filename="package://bandit_urdf/meshes/bandit_mesh/gradients/reflect1.jpg"/>
-                    </material>
-      </visual>
-      <collision name="${name}_collision">
-         <origin xyz="0 0 0" rpy="0 0 0 " />
-        <geometry name="${name}_visual_geom">
-                    <box size="0 0 0"/>
-        </geometry>
-      </collision>
-    </link>
-</xacro:macro>
-    <xacro:macro name="eyebrow" params="name parent side reflect *origin">
-    <joint name="head_${side}_brow_joint" type="revolute">
-      <axis xyz="0 ${reflect} 0" />
-      <limit lower="-0.261799388" upper="0.261799388" effort="2.645" velocity="6" />
-      <safety_controller k_velocity="1.5" soft_lower_limit="${-1.57079633+0.15}" soft_upper_limit="${1.57079633-0.15}" k_position="100" />
-      <calibration reference_position="0.0" />
-      <dynamics damping="1.0" />
-      <insert_block name="origin" />
-      <parent link="${parent}"/>
-      <child link="${name}_link"/>
-    </joint>
-    <link name="${name}_link">
-      <inertial>
-        <mass value="0" />
-        <origin xyz="0 0 0" rpy="${RCon*90} 0 ${RCon*90}"/>
-        <inertia ixx="0.00482611007"  ixy="-0.000144683999"  ixz="0.000110076136"
-                 iyy="0.005218991412"  iyz="-0.000314239509"  izz="0.008618784925"/>
-      </inertial>
-      <visual name="${name}_visual">
-        <origin xyz="0 0 0" rpy="0 0 ${RCon*-90}"/>
-        <geometry name="${name}_visual_geom">
-                    <mesh filename="package://bandit_urdf/meshes/bandit_mesh/eyebrow_${side}_small.stl"/>
-        </geometry>
-                    <material name="Eyebrows"/>
-      </visual>
-      <collision name="${name}_collision">
-         <origin xyz="0 0 0" rpy="0 0 0 " />
-        <geometry name="${name}_visual_geom">
-                    <box size="0 0 0"/>
-        </geometry>
-      </collision>
-    </link>
     </xacro:macro>
-<xacro:macro name="pupil" params="suffix reflect">
-    <joint name="pupil_${suffix}_joint" type="fixed">
-        <origin xyz="0.0012 ${reflect*0.001} -0.032" rpy="0 0 0"/>
-        <parent link="head_${suffix}_camera_link"/>
-        <child link="pupil_${suffix}_link"/>
-    </joint>
-    <link name="pupil_${suffix}_link">
-        <inertial>
-            <mass value="0"/>
-            <origin xyz="0 0 0"/>
-            <inertia ixx="1" ixy="0" ixz="0"
-                 iyy="1" iyz="0" izz="1"/>
-        </inertial>
-        <visual name="pupil_visual">
-            <origin xyz="0 0 0" rpy="0 0 0"/>
-            <geometry name="pupil_left_geom">
-                <mesh filename="package://bandit_urdf/meshes/bandit_mesh/middle_eye.stl"/>
-            </geometry>
-        <material name="Pupil">
-            <color rgba="0 0 0 1"/>
-        </material>
-        </visual>
-        <collision>
-            <origin xyz="0 0 0" rpy="0 0 0"/>
-            <geometry>
-                <box size="0 0 0"/>
-            </geometry>
-        </collision>
-    </link>
-</xacro:macro>
-<xacro:pupil suffix="left" reflect="-4.8"/>
-<xacro:pupil suffix="right" reflect="-4.6"/>
-~~~~~~~~~~~~~~`-->
+    <!-- end eyebrow xacro definition -->
+	<!-- start pupil xacro definition -->
+	<xacro:macro name="pupil" params="suffix reflect">
+		<!-- pupil_{side}_joint -->
+		<joint name="pupil_${suffix}_joint" type="fixed">
+    		<origin xyz="0.0012 ${reflect*0.001} -0.032" rpy="0 0 0"/>
+    		<parent link="eye_${suffix}_camera_link"/>
+    		<child link="pupil_${suffix}_link"/>
+		</joint>
+		<!-- pupil_{side}_link -->
+		<link name="pupil_${suffix}_link">
+    		<inertial>
+        		<mass value="0"/>
+        		<origin xyz="0 0 0"/>
+        		<inertia ixx="1" ixy="0" ixz="0" iyy="1" iyz="0" izz="1"/>
+    		</inertial>
+    		<visual name="pupil_visual">
+        		<origin xyz="0 0 0" rpy="0 0 0"/>
+        		<geometry name="pupil_left_geom">
+            		<mesh filename="${mesh_path}/middle_eye.stl"/>
+        		</geometry>
+    			<material name="Pupil">
+        			<color rgba="0 0 0 1"/>
+    			</material>
+    		</visual>
+    		<collision>
+        		<origin xyz="0 0 0" rpy="0 0 0"/>
+        		<geometry>
+            		<box size="0 0 0"/>
+        		</geometry>
+    		</collision>
+		</link>
 	</xacro:macro>
+	<!-- end pupil xacro definition -->
 </robot>

File: bandit/bandit_urdf/defs/shoulder.xacro (robot description, xacro)
@@ -4,6 +4,6 @@
        xmlns:interface="http://playerstage.sourceforge.net/gazebo/xmlschema/#interface"
        xmlns:xacro="http://ros.org/wiki/xacro">
-	<!-- path to mesh files -->
-	<property name="mesh_path" value="package://bandit_urdf/meshes/bandit_mesh/"/>
+	<!-- use the below line to specify path to meshes and materials -->
+	<property name="mesh_path" value="package://bandit_urdf/meshes/bandit_mesh"/>
 	<!-- other properties -->
     <property name="RCon" value="0.01744"/>

File: bandit/bandit_urdf/defs/torso.xacro (robot description, xacro)
@@ -4,6 +4,6 @@
        xmlns:interface="http://playerstage.sourceforge.net/gazebo/xmlschema/#interface"
        xmlns:xacro="http://ros.org/wiki/xacro">
-	<!-- path to mesh files -->
-	<property name="mesh_path" value="package://bandit_urdf/meshes/bandit_mesh/"/>
+	<!-- use the below line to specify path to meshes and materials -->
+	<property name="mesh_path" value="package://bandit_urdf/meshes/bandit_mesh"/>
 	<!-- other properties -->
 	<!-- torso xacro definition -->
