Commit message: Gazebo Fix for Loading Bandit From URDF Description -- set mass of bandit componnents to fractional non-zero

File: bandit/bandit_urdf/defs/head.xacro (robot description, xacro)
@@ -25,5 +25,5 @@
       		<inertial>
       			<origin xyz="-0.05 0 -0.101" rpy="183.928 0 -90"/>
-        		<mass value="0"/>
+        		<mass value="0.01"/>
         		<inertia ixx="0.00482611007"  ixy="-0.000144683999"
         				ixz="0.000110076136" iyy="0.005218991412"
@@ -59,5 +59,5 @@
     	<link name="head_tilt_link">
       		<inertial>
-        		<mass value="0" />
+        		<mass value="0.01" />
         		<origin xyz="0 0 0" rpy="${RCon*90} 0 ${RCon*90}"/>
         		<inertia ixx="0.00482611007"  ixy="-0.000144683999"  ixz="0.000110076136"
@@ -93,5 +93,5 @@
     	<link name="mouth_top_link">
       		<inertial>
-        		<mass value="0" />
+        		<mass value="0.01" />
         		<origin xyz="0 0 0" rpy="0 0 ${RCon*90}"/>
         		<inertia ixx="0.00482611007"  ixy="-0.000144683999"
@@ -129,5 +129,5 @@
 		<link name="mouth_bottom_link">
 	  		<inertial>
-	    		<mass value="0" />
+	    		<mass value="0.01" />
 	    		<origin xyz="0 0 0" rpy="${RCon*90} 0 ${RCon*90}"/>
 	    		<inertia ixx="0.00482611007"  ixy="-0.000144683999"
@@ -181,5 +181,5 @@
 		<link name="${name}_link">
   			<inertial>
-    			<mass value="0" />
+    			<mass value="0.01" />
     			<origin xyz="0 0 0" rpy="${RCon*90} 0 ${RCon*90}"/>
     			<inertia ixx="0.00482611007"  ixy="-0.000144683999"
@@ -221,5 +221,5 @@
     	<link name="${name}_link">
       		<inertial>
-        		<mass value="0" />
+        		<mass value="0.01" />
         		<origin xyz="0 0 0" rpy="${RCon*90} 0 ${RCon*90}"/>
         		<inertia ixx="0.00482611007"  ixy="-0.000144683999"
@@ -254,5 +254,5 @@
 		<link name="pupil_${suffix}_link">
     		<inertial>
-        		<mass value="0"/>
+        		<mass value="0.01"/>
         		<origin xyz="0 0 0"/>
         		<inertia ixx="1" ixy="0" ixz="0" iyy="1" iyz="0" izz="1"/>

File: bandit/bandit_urdf/defs/logo.xacro (robot description, xacro)
@@ -13,5 +13,5 @@
 		<inertial>
 			<origin xyz="0 0.15 0" rpy="${RCon*90} 0 ${RCon*90}"/>
-			<mass value="0"/>
+			<mass value="0.01"/>
 			<inertia ixx="0.866179142480" ixy="-0.06086507933"
 			ixz="-0.12118061183" iyy="0.87421714893"

File: bandit/bandit_urdf/defs/screws.xacro (robot description, xacro)
@@ -9,5 +9,5 @@
 	<link name="screw1_${suffix}_link">
 		<inertial>
-			<mass value="0"/>
+			<mass value="0.01"/>
 			<origin xyz="0 0 0"/>
 			<inertia ixx="1" ixy="0" ixz="0"
@@ -35,5 +35,5 @@
 	<link name="screw2_${suffix}_link">
 		<inertial>
-			<mass value="0"/>
+			<mass value="0.01"/>
 			<origin xyz="0 0 0"/>
 			<inertia ixx="1" ixy="0" ixz="0"
@@ -61,5 +61,5 @@
 	<link name="screw3_${suffix}_link">
 		<inertial>
-			<mass value="0"/>
+			<mass value="0.01"/>
 			<origin xyz="0 0 0"/>
 			<inertia ixx="1" ixy="0" ixz="0"
@@ -87,5 +87,5 @@
 	<link name="screw4_${suffix}_link">
 		<inertial>
-			<mass value="0"/>
+			<mass value="0.01"/>
 			<origin xyz="0 0 0"/>
 			<inertia ixx="1" ixy="0" ixz="0"
@@ -113,5 +113,5 @@
 	<link name="screw5_${suffix}_link">
 		<inertial>
-			<mass value="0"/>
+			<mass value="0.01"/>
 			<origin xyz="0 0 0"/>
 			<inertia ixx="1" ixy="0" ixz="0"
@@ -139,5 +139,5 @@
 	<link name="screw6_${suffix}_link">
 		<inertial>
-			<mass value="0"/>
+			<mass value="0.01"/>
 			<origin xyz="0 0 0"/>
 			<inertia ixx="1" ixy="0" ixz="0"
@@ -165,5 +165,5 @@
 	<link name="screw7_${suffix}_link">
 		<inertial>
-			<mass value="0"/>
+			<mass value="0.01"/>
 			<origin xyz="0 0 0"/>
 			<inertia ixx="1" ixy="0" ixz="0"
@@ -191,5 +191,5 @@
 	<link name="screw8_${suffix}_link">
 		<inertial>
-			<mass value="0"/>
+			<mass value="0.01"/>
 			<origin xyz="0 0 0"/>
 			<inertia ixx="1" ixy="0" ixz="0"
@@ -217,5 +217,5 @@
 	<link name="screw9_${suffix}_link">
 		<inertial>
-			<mass value="0"/>
+			<mass value="0.01"/>
 			<origin xyz="0 0 0"/>
 			<inertia ixx="1" ixy="0" ixz="0"
@@ -243,5 +243,5 @@
 	<link name="screw10_${suffix}_link">
 		<inertial>
-			<mass value="0"/>
+			<mass value="0.01"/>
 			<origin xyz="0 0 0"/>
 			<inertia ixx="1" ixy="0" ixz="0"
@@ -269,5 +269,5 @@
 	<link name="screw11_${suffix}_link">
 		<inertial>
-			<mass value="0"/>
+			<mass value="0.01"/>
 			<origin xyz="0 0 0"/>
 			<inertia ixx="1" ixy="0" ixz="0"
@@ -295,5 +295,5 @@
 	<link name="screw12_${suffix}_link">
 		<inertial>
-			<mass value="0"/>
+			<mass value="0.01"/>
 			<origin xyz="0 0 0"/>
 			<inertia ixx="1" ixy="0" ixz="0"
@@ -321,5 +321,5 @@
 	<link name="screw13_${suffix}_link">
 		<inertial>
-			<mass value="0"/>
+			<mass value="0.01"/>
 			<origin xyz="0 0 0"/>
 			<inertia ixx="1" ixy="0" ixz="0"
@@ -347,5 +347,5 @@
 	<link name="screw14_${suffix}_link">
 		<inertial>
-			<mass value="0"/>
+			<mass value="0.01"/>
 			<origin xyz="0 0 0"/>
 			<inertia ixx="1" ixy="0" ixz="0"
@@ -373,5 +373,5 @@
 	<link name="screw15_${suffix}_link">
 		<inertial>
-			<mass value="0"/>
+			<mass value="0.01"/>
 			<origin xyz="0 0 0"/>
 			<inertia ixx="1" ixy="0" ixz="0"
@@ -399,5 +399,5 @@
 	<link name="screw16_${suffix}_link">
 		<inertial>
-			<mass value="0"/>
+			<mass value="0.01"/>
 			<origin xyz="0 0 0"/>
 			<inertia ixx="1" ixy="0" ixz="0"
@@ -425,5 +425,5 @@
 	<link name="screw17_${suffix}_link">
 		<inertial>
-			<mass value="0"/>
+			<mass value="0.01"/>
 			<origin xyz="0 0 0"/>
 			<inertia ixx="1" ixy="0" ixz="0"
@@ -451,5 +451,5 @@
 	<link name="screw18_${suffix}_link">
 		<inertial>
-			<mass value="0"/>
+			<mass value="0.01"/>
 			<origin xyz="0 0 0"/>
 			<inertia ixx="1" ixy="0" ixz="0"
@@ -503,5 +503,5 @@
 	<link name="screw20_${suffix}_link">
 		<inertial>
-			<mass value="0"/>
+			<mass value="0.01"/>
 			<origin xyz="0 0 0"/>
 			<inertia ixx="1" ixy="0" ixz="0"
@@ -529,5 +529,5 @@
 	<link name="screw21_${suffix}_link">
 		<inertial>
-			<mass value="0"/>
+			<mass value="0.01"/>
 			<origin xyz="0 0 0"/>
 			<inertia ixx="1" ixy="0" ixz="0"
@@ -555,5 +555,5 @@
 	<link name="screw22_${suffix}_link">
 		<inertial>
-			<mass value="0"/>
+			<mass value="0.01"/>
 			<origin xyz="0 0 0"/>
 			<inertia ixx="1" ixy="0" ixz="0"
@@ -581,5 +581,5 @@
 	<link name="screw23_${suffix}_link">
 		<inertial>
-			<mass value="0"/>
+			<mass value="0.01"/>
 			<origin xyz="0 0 0"/>
 			<inertia ixx="1" ixy="0" ixz="0"
@@ -607,5 +607,5 @@
 	<link name="screw24_${suffix}_link">
 		<inertial>
-			<mass value="0"/>
+			<mass value="0.01"/>
 			<origin xyz="0 0 0"/>
 			<inertia ixx="1" ixy="0" ixz="0"
@@ -633,5 +633,5 @@
 	<link name="screw25_${suffix}_link">
 		<inertial>
-			<mass value="0"/>
+			<mass value="0.01"/>
 			<origin xyz="0 0 0"/>
 			<inertia ixx="1" ixy="0" ixz="0"
@@ -659,5 +659,5 @@
 	<link name="screw26_${suffix}_link">
 		<inertial>
-			<mass value="0"/>
+			<mass value="0.01"/>
 			<origin xyz="0 0 0"/>
 			<inertia ixx="1" ixy="0" ixz="0"
@@ -685,5 +685,5 @@
 	<link name="screw27_${suffix}_link">
 		<inertial>
-			<mass value="0"/>
+			<mass value="0.01"/>
 			<origin xyz="0 0 0"/>
 			<inertia ixx="1" ixy="0" ixz="0"
@@ -711,5 +711,5 @@
 	<link name="screw28_${suffix}_link">
 		<inertial>
-			<mass value="0"/>
+			<mass value="0.01"/>
 			<origin xyz="0 0 0"/>
 			<inertia ixx="1" ixy="0" ixz="0"
@@ -737,5 +737,5 @@
 	<link name="screw29_${suffix}_link">
 		<inertial>
-			<mass value="0"/>
+			<mass value="0.01"/>
 			<origin xyz="0 0 0"/>
 			<inertia ixx="1" ixy="0" ixz="0"
@@ -763,5 +763,5 @@
 	<link name="screw30_${suffix}_link">
 		<inertial>
-			<mass value="0"/>
+			<mass value="0.01"/>
 			<origin xyz="0 0 0"/>
 			<inertia ixx="1" ixy="0" ixz="0"
@@ -789,5 +789,5 @@
 	<link name="screw31_${suffix}_link">
 		<inertial>
-			<mass value="0"/>
+			<mass value="0.01"/>
 			<origin xyz="0 0 0"/>
 			<inertia ixx="1" ixy="0" ixz="0"
@@ -815,5 +815,5 @@
 	<link name="screw32_${suffix}_link">
 		<inertial>
-			<mass value="0"/>
+			<mass value="0.01"/>
 			<origin xyz="0 0 0"/>
 			<inertia ixx="1" ixy="0" ixz="0"
@@ -844,5 +844,5 @@
 	<link name="screwA_link">
 		<inertial>
-			<mass value="0"/>
+			<mass value="0.01"/>
 			<origin xyz="0 0 0"/>
 			<inertia ixx="1" ixy="0" ixz="0"
@@ -870,5 +870,5 @@
 	<link name="screwB_link">
 		<inertial>
-			<mass value="0"/>
+			<mass value="0.01"/>
 			<origin xyz="0 0 0"/>
 			<inertia ixx="1" ixy="0" ixz="0"
@@ -896,5 +896,5 @@
 	<link name="screwC_link">
 		<inertial>
-			<mass value="0"/>
+			<mass value="0.01"/>
 			<origin xyz="0 0 0"/>
 			<inertia ixx="1" ixy="0" ixz="0"
@@ -922,5 +922,5 @@
 	<link name="screwD_link">
 		<inertial>
-			<mass value="0"/>
+			<mass value="0.01"/>
 			<origin xyz="0 0 0"/>
 			<inertia ixx="1" ixy="0" ixz="0"

File: bandit/bandit_urdf/defs/shoulder.xacro (robot description, xacro)
@@ -31,5 +31,5 @@
             <inertial>
                 <origin xyz="-0.035 0.131 ${reflect*0.168}" rpy="${M_PI} 0 0"/>
-                <mass value="0"/>
+                <mass value="0.01"/>
                 <inertia ixx="0.866179142480" ixy="-0.06086507933"
                 		ixz="-0.12118061183" iyy="0.87421714893"
@@ -66,5 +66,5 @@
             <inertial>
                 <origin xyz="-0.030 -0. -0" rpy="0 ${RCon*180} 0"/>
-                <mass value="0"/>
+                <mass value="0.01"/>
                 <inertia ixx="0.866179142480" ixy="-0.06086507933"
                 		ixz="-0.12118061183" iyy="0.87421714893"
@@ -101,5 +101,5 @@
             <inertial>
                 <origin xyz="-0.0 0.0 -0.288" rpy="0 0 ${RCon*90}"/>
-                <mass value="0"/>
+                <mass value="0.01"/>
                 <inertia ixx="0.866179142480" ixy="-0.06086507933"
                 		ixz="-0.12118061183" iyy="0.87421714893"
@@ -136,5 +136,5 @@
             <inertial>
                 <origin xyz="-0.028 0.163 -0.372" rpy="0 ${RCon*180} ${RCon*180}"/>
-                <mass value="0"/>
+                <mass value="0.01"/>
                 <inertia ixx="0.866179142480" ixy="-0.06086507933"
                 		ixz="-0.12118061183" iyy="0.87421714893"
@@ -171,5 +171,5 @@
             <inertial>
                 <origin xyz="-0.026 0.163 -0.434" rpy="0 0 0"/>
-                <mass value="0"/>
+                <mass value="0.01"/>
                 <inertia ixx="0.866179142480" ixy="-0.06086507933"
                 		ixz="-0.12118061183" iyy="0.87421714893"
@@ -206,5 +206,5 @@
             <inertial>
                 <origin xyz="-0.015 0.163 -0.486" rpy="${RCon*57} 0 ${RCon*90}"/>
-                <mass value="0"/>
+                <mass value="0.01"/>
                 <inertia ixx="0.866179142480" ixy="-0.06086507933"
                 		ixz="-0.12118061183" iyy="0.87421714893"
@@ -241,5 +241,5 @@
             <inertial>
                 <origin xyz="0.037 0.163 -0.484" rpy="${RCon*90} 0 ${RCon*90}"/>
-                <mass value="0"/>
+                <mass value="0.01"/>
                 <inertia ixx="0.866179142480" ixy="-0.06086507933"
                 		ixz="-0.12118061183" iyy="0.87421714893"

File: bandit/bandit_urdf/defs/torso.xacro (robot description, xacro)
@@ -12,5 +12,5 @@
     	<link name = "${name}_link">
         	<inertial>
-        		<mass value="0"/>
+        		<mass value="0.01"/>
         		<origin xyz="0 0 0"/>
         		<inertia ixx="1" ixy="0" ixz="0" iyy="1" iyz="0" izz="1"/>
@@ -33,5 +33,5 @@
 		<link name="stop_link">
 		    <inertial>
-		        <mass value="0"/>
+		        <mass value="0.01"/>
 		        <origin xyz="0 0 0"/>
 		        <inertia ixx="1" ixy="0" ixz="0" iyy="1" iyz="0" izz="1"/>

File: bandit/bandit_urdf/urdf/bandit_defs.urdf (robot description, URDF)
Before this commit: robot bandit, 26 links, 25 joints
Links:
- link eye_left_camera_link: mass 0 -> 0.01
- link eye_right_camera_link: mass 0 -> 0.01
- link head_left_brow_link: mass 0 -> 0.01
- link head_pan_link: mass 0 -> 0.01
- link head_right_brow_link: mass 0 -> 0.01
- link head_tilt_link: mass 0 -> 0.01
- link left_bicep_link: mass 0 -> 0.01
- link left_forearm_link: mass 0 -> 0.01
- link left_hand_link: mass 0 -> 0.01
- link left_shoulder_link: mass 0 -> 0.01
- link left_shoulder_mounting_link: mass 0 -> 0.01
- link left_thumb_link: mass 0 -> 0.01
- link left_wrist_link: mass 0 -> 0.01
- link mouth_bottom_link: mass 0 -> 0.01
- link mouth_top_link: mass 0 -> 0.01
- link pupil_left_link: mass 0 -> 0.01
- link pupil_right_link: mass 0 -> 0.01
- link right_bicep_link: mass 0 -> 0.01
- link right_forearm_link: mass 0 -> 0.01
- link right_hand_link: mass 0 -> 0.01
- link right_shoulder_link: mass 0 -> 0.01
- link right_shoulder_mounting_link: mass 0 -> 0.01
- link right_thumb_link: mass 0 -> 0.01
- link right_wrist_link: mass 0 -> 0.01
- link stop_link: mass 0 -> 0.01
- link torso_link: mass 0 -> 0.01

File: bandit/bandit_urdf/urdf/bandit_shirt_defs.urdf (robot description, URDF)
Before this commit: robot bandit, 109 links, 108 joints
Links:
- link bandit_logo: mass 0 -> 0.01
- link eye_left_camera_link: mass 0 -> 0.01
- link eye_right_camera_link: mass 0 -> 0.01
- link head_left_brow_link: mass 0 -> 0.01
- link head_pan_link: mass 0 -> 0.01
- link head_right_brow_link: mass 0 -> 0.01
- link head_tilt_link: mass 0 -> 0.01
- link left_bicep_link: mass 0 -> 0.01
- link left_forearm_link: mass 0 -> 0.01
- link left_hand_link: mass 0 -> 0.01
- link left_shoulder_link: mass 0 -> 0.01
- link left_shoulder_mounting_link: mass 0 -> 0.01
- link left_thumb_link: mass 0 -> 0.01
- link left_wrist_link: mass 0 -> 0.01
- link mouth_bottom_link: mass 0 -> 0.01
- link mouth_top_link: mass 0 -> 0.01
- link pupil_left_link: mass 0 -> 0.01
- link pupil_right_link: mass 0 -> 0.01
- link right_bicep_link: mass 0 -> 0.01
- link right_forearm_link: mass 0 -> 0.01
- link right_hand_link: mass 0 -> 0.01
- link right_shoulder_link: mass 0 -> 0.01
- link right_shoulder_mounting_link: mass 0 -> 0.01
- link right_thumb_link: mass 0 -> 0.01
- link right_wrist_link: mass 0 -> 0.01
- link screw10_left_link: mass 0 -> 0.01
- link screw10_right_link: mass 0 -> 0.01
- link screw11_left_link: mass 0 -> 0.01
- link screw11_right_link: mass 0 -> 0.01
- link screw12_left_link: mass 0 -> 0.01
- link screw12_right_link: mass 0 -> 0.01
- link screw13_left_link: mass 0 -> 0.01
- link screw13_right_link: mass 0 -> 0.01
- link screw14_left_link: mass 0 -> 0.01
- link screw14_right_link: mass 0 -> 0.01
- link screw15_left_link: mass 0 -> 0.01
- link screw15_right_link: mass 0 -> 0.01
- link screw16_left_link: mass 0 -> 0.01
- link screw16_right_link: mass 0 -> 0.01
- link screw17_left_link: mass 0 -> 0.01
- link screw17_right_link: mass 0 -> 0.01
- link screw18_left_link: mass 0 -> 0.01
- link screw18_right_link: mass 0 -> 0.01
- link screw1_left_link: mass 0 -> 0.01
- link screw1_right_link: mass 0 -> 0.01
- link screw20_left_link: mass 0 -> 0.01
- link screw20_right_link: mass 0 -> 0.01
- link screw21_left_link: mass 0 -> 0.01
- link screw21_right_link: mass 0 -> 0.01
- link screw22_left_link: mass 0 -> 0.01
- link screw22_right_link: mass 0 -> 0.01
- link screw23_left_link: mass 0 -> 0.01
- link screw23_right_link: mass 0 -> 0.01
- link screw24_left_link: mass 0 -> 0.01
- link screw24_right_link: mass 0 -> 0.01
- link screw25_left_link: mass 0 -> 0.01
- link screw25_right_link: mass 0 -> 0.01
- link screw26_left_link: mass 0 -> 0.01
- link screw26_right_link: mass 0 -> 0.01
- link screw27_left_link: mass 0 -> 0.01
- link screw27_right_link: mass 0 -> 0.01
- link screw28_left_link: mass 0 -> 0.01
- link screw28_right_link: mass 0 -> 0.01
- link screw29_left_link: mass 0 -> 0.01
- link screw29_right_link: mass 0 -> 0.01
- link screw2_left_link: mass 0 -> 0.01
- link screw2_right_link: mass 0 -> 0.01
- link screw30_left_link: mass 0 -> 0.01
- link screw30_right_link: mass 0 -> 0.01
- link screw31_left_link: mass 0 -> 0.01
- link screw31_right_link: mass 0 -> 0.01
- link screw32_left_link: mass 0 -> 0.01
- link screw32_right_link: mass 0 -> 0.01
- link screw3_left_link: mass 0 -> 0.01
- link screw3_right_link: mass 0 -> 0.01
- link screw4_left_link: mass 0 -> 0.01
- link screw4_right_link: mass 0 -> 0.01
- link screw5_left_link: mass 0 -> 0.01
- link screw5_right_link: mass 0 -> 0.01
- link screw6_left_link: mass 0 -> 0.01
- link screw6_right_link: mass 0 -> 0.01
- link screw7_left_link: mass 0 -> 0.01
- link screw7_right_link: mass 0 -> 0.01
- link screw8_left_link: mass 0 -> 0.01
- link screw8_right_link: mass 0 -> 0.01
- link screw9_left_link: mass 0 -> 0.01
- link screw9_right_link: mass 0 -> 0.01
- link screwA_link: mass 0 -> 0.01
- link screwB_link: mass 0 -> 0.01
- link screwC_link: mass 0 -> 0.01
- link screwD_link: mass 0 -> 0.01
- link stop_link: mass 0 -> 0.01
- link torso_link: mass 0 -> 0.01
