Commit message: urdf fixes for groovy and gazebo

File: bandit/bandit_urdf/defs/head.xacro (robot description, xacro)
@@ -1,7 +1,4 @@
 <?xml version="1.0"?>
-<robot xmlns:sensor="http://playerstage.sourceforge.net/gazebo/xmlschema/#sensor"
-       xmlns:controller="http://playerstage.sourceforge.net/gazebo/xmlschema/#controller"
-       xmlns:interface="http://playerstage.sourceforge.net/gazebo/xmlschema/#interface"
-       xmlns:xacro="http://ros.org/wiki/xacro">
+<robot xmlns:xacro="http://ros.org/wiki/xacro">
 	<!-- use the below line to specify path to meshes and materials -->
 	<property name="mesh_path" value="package://bandit_urdf/meshes/bandit_mesh"/>
@@ -67,5 +64,5 @@
         		<origin xyz="-.02 0 .01" rpy="${RCon*90} 0 ${RCon*90}"/>
         		<geometry name="head_tilt_visual_geom">
-        			<mesh filename="${mesh_path}/head_smallest.stl"/>
+        			<mesh filename="${mesh_path}/head_small.stl"/>
         		</geometry>
         		<material name="Head"/>
@@ -80,4 +77,5 @@
     	<!-- mouth_top_joint -->
       	<joint name="mouth_top_joint" type="revolute">
+            <origin xyz="0.07 0 -0.01" rpy="0 0 0"/>
         	<axis xyz="0 -1 0" />
         	<limit lower="-0.261799388" upper="0.261799388" effort="2.645" velocity="6" />
@@ -116,4 +114,5 @@
 		<!-- mouth_bottom_joint -->
 	  	<joint name="mouth_bottom_joint" type="revolute">
+            <origin xyz="0.07 0 -0.01" rpy="0 0 0"/>
 	    	<axis xyz="0 -1 0"/>
 	    	<limit lower="-0.261799388" upper="0.261799388" effort="2.645" velocity="6" />

File: bandit/bandit_urdf/defs/shoulder.xacro (robot description, xacro)
@@ -1,7 +1,4 @@
 <?xml version="1.0"?>
-<robot xmlns:sensor="http://playerstage.sourceforge.net/gazebo/xmlschema/#sensor"
-       xmlns:controller="http://playerstage.sourceforge.net/gazebo/xmlschema/#controller"
-       xmlns:interface="http://playerstage.sourceforge.net/gazebo/xmlschema/#interface"
-       xmlns:xacro="http://ros.org/wiki/xacro">
+<robot xmlns:xacro="http://ros.org/wiki/xacro">
 	<!-- use the below line to specify path to meshes and materials -->
 	<property name="mesh_path" value="package://bandit_urdf/meshes/bandit_mesh"/>

File: bandit/bandit_urdf/defs/torso.xacro (robot description, xacro)
@@ -1,7 +1,4 @@
 <?xml version="1.0"?>
-<robot xmlns:sensor="http://playerstage.sourceforge.net/gazebo/xmlschema/#sensor"
-       xmlns:controller="http://playerstage.sourceforge.net/gazebo/xmlschema/#controller"
-       xmlns:interface="http://playerstage.sourceforge.net/gazebo/xmlschema/#interface"
-       xmlns:xacro="http://ros.org/wiki/xacro">
+<robot  xmlns:xacro="http://www.ros.org/wiki/xacro">
 	<!-- use the below line to specify path to meshes and materials -->
 	<property name="mesh_path" value="package://bandit_urdf/meshes/bandit_mesh"/>
@@ -34,5 +31,5 @@
 		    <inertial>
 		        <mass value="0.01"/>
-		        <origin xyz="0 0 0"/>
+                <origin xyz="0 0 0"/>
 		        <inertia ixx="1" ixy="0" ixz="0" iyy="1" iyz="0" izz="1"/>
 		    </inertial>

File: bandit/bandit_urdf/urdf/bandit_defs.urdf (robot description, URDF)
Before this commit: robot bandit, 26 links, 25 joints
Links:
- added link world
- link head_tilt_link: geometry collision box size=0.147 0.156 0.16; visual mesh filename=package://bandit_urdf/meshes/bandit_mesh/head_small.stl
Joints:
- added joint fixed: type fixed, parent world, child torso_link
- joint head_tilt_joint: origin xyz=0 0 0.18135 rpy=0 0 0 -> xyz=0 0 0 rpy=0 0 0
- joint mouth_bottom_joint: origin xyz=0 0 0.18135 rpy=0 0 0 -> xyz=0.07 0 -0.01 rpy=0 0 0
- joint mouth_top_joint: origin xyz=0 0 0.18135 rpy=0 0 0 -> xyz=0.07 0 -0.01 rpy=0 0 0

File: bandit/bandit_urdf/urdf/bandit_defs.urdf.xacro (robot description, xacro)
@@ -1,25 +1,23 @@
 <?xml version="1.0"?>
-<robot xmlns:sensor="http://playerstage.sourceforge.net/gazebo/xmlschema/#sensor"
-       xmlns:controller="http://playerstage.sourceforge.net/gazebo/xmlschema/#controller"
-       xmlns:interface="http://playerstage.sourceforge.net/gazebo/xmlschema/#interface"
-       xmlns:xacro="http://playerstage.sourceforge.net/gazebo/xmlschema/#interface"
-             name="bandit">
+<robot name="bandit" xmlns:xacro="http://www.ros.org/wiki/xacro">
     <include filename="$(find bandit_urdf)/defs/common.xacro"/>
-  	<!-- uncomment the below line for the bandit_shirt materials -->
-  	<!--  <include filename="$(find bandit_urdf)/defs/shirt_materials.xacro"/>-->
-  	<!-- use the below line for the regular bandit materials -->
-    <include filename="$(find bandit_urdf)/defs/materials.xacro"/>
-    <include filename="$(find bandit_urdf)/defs/torso.xacro"/>
-    <include filename="$(find bandit_urdf)/defs/head.xacro"/>
-    <include filename="$(find bandit_urdf)/defs/shoulder.xacro"/>
-    <!-- use the below line for gazebo includes -->
-    <!--<include filename="$(find bandit_urdf)/urdf/gazebo.urdf.xacro"/>-->
-    <!-- use the below line for pr2 includes -->
-    <!--<xacro:pr2_base_v0 name="base"/>-->
-    <xacro:torso name="torso" parent="/robot/base_link">
+  <!-- Import Rviz colors -->
+    <xacro:include filename="$(find bandit_urdf)/defs/materials.xacro" />
+    <xacro:include filename="$(find bandit_urdf)/defs/torso.xacro"/>
+    <xacro:include filename="$(find bandit_urdf)/defs/head.xacro"/>
+    <xacro:include filename="$(find bandit_urdf)/defs/shoulder.xacro"/>
+  <!-- Import all Gazebo-customization elements, including Gazebo colors -->
+    <xacro:include filename="$(find bandit_urdf)/urdf/bandit.gazebo" />
+    <!-- Used for fixing robot to Gazebo 'base_link' -->
+    <link name="world"/>
+    <joint name="fixed" type="fixed">
+        <parent link="world"/>
+        <child link="torso_link"/>
+    </joint>
+    <xacro:torso name="torso" parent="world">
         <origin xyz="-0.00 0 ${body_height/2}" rpy="0 0 0"/>
     </xacro:torso>
-	<xacro:head name="head" parent="torso_link">
-        <origin xyz="0 0 ${body_height/2+neck_height/2+0.01}" rpy="0 0 0"/>
+    <xacro:head name="head" parent="torso_link">
+        <origin xyz="0 0 0" rpy="0 0 0"/>
     </xacro:head>
 	<xacro:shoulder side="left" parent="torso_link" reflect="1">

File: bandit/bandit_urdf/urdf/bandit_shirt_defs.urdf (robot description, URDF)
Before this commit: robot bandit, 109 links, 108 joints
Links:
- link head_tilt_link: geometry collision box size=0.147 0.156 0.16; visual mesh filename=package://bandit_urdf/meshes/bandit_mesh/head_small.stl
Joints:
- joint mouth_bottom_joint: origin xyz=0 0 0.18135 rpy=0 0 0 -> xyz=0.07 0 -0.01 rpy=0 0 0
- joint mouth_top_joint: origin xyz=0 0 0.18135 rpy=0 0 0 -> xyz=0.07 0 -0.01 rpy=0 0 0
